File: Hardware/ESP32_Thing_Plus.brd (EAGLE design)
At the start: 66 x 31.8 mm, 33 parts, among them J1 455-1750-1-ND, J2 USB Female Type C Connector, J3 AUDIO_JACK_TRRSSMD_RA, Q2 MBT3904DW1T1, U1 I2SMICMIC, U2 ESP-WROOM-32NARROW, U3 AP2112K-3.3V, U4 CP2102N

Commit message: updating mic and trrs circuits
Parts:
- removed U1: I2SMICMIC, Andy:I2CMIC
- added C4: 4.7uF, SparkFun-Capacitors:0603
- added C5: 100pF, SparkFun-Capacitors:0603
- added C6: 1.0uF, SparkFun-Capacitors:0603
- added C9: 0.1uF, SparkFun-Capacitors:0603
- added R10, R9: 10k, SparkFun-Resistors:0603
- added R11, R12: 100k, SparkFun-Resistors:0603
- added R13: 1k, SparkFun-Resistors:AXIAL-0.3
- added R14, R15: 1k, SparkFun-Resistors:0603
- added U$2: OPA344, SparkFun-IC-Amplifiers:SOT23-5
- added U$3: (no value), cec7b2_1ee547f747c2467bb1a21a2065860725_mv2#jpg (1):CEC7B2_1EE547F747C2467BB1A21A2065860725_MV2#JPG
- added U5: ADMP401, SparkFun-Sensors:ADMP401
- C2: value 180pF -> 0.1uF
- R5, R6, R7: value 47 -> 100k
- moved R5 46.4 mm to (16.5, 26.0), turned to 0 degrees
- moved C2 43.6 mm to (16.5, 22.2), turned to 0 degrees
- moved R7 30.6 mm to (16.5, 24.1), turned to 180 degrees
- moved R6 26.7 mm to (16.5, 20.3), turned to 0 degrees
- moved C3 25.5 mm to (16.5, 27.9), turned to 180 degrees
- moved R4 2.54 mm to (10.2, 12.7)
- moved J2 2.54 mm to (6.99, 11.6)
- moved R3 2.54 mm to (10.2, 10.2)
- moved C1 1.27 mm to (14.0, 8.26)
- moved C10 1.27 mm to (14.0, 10.2)
- moved C7 1.27 mm to (10.9, 4.45)
- moved R8 1.27 mm to (14.0, 1.27)
- moved U3 1.27 mm to (14.0, 5.08)
- moved U$1 1.27 mm to (17.8, 2.54)
Connections:
- removed net 25: R7.2, U1.1
- removed net 26: R6.2, U1.4
- removed net A2: U2.6
- removed net N$8: R7.1, U2.10
- new net MIC: C5.2, R11.2, U$2.1, U2.6
- new net N$11: C4.2, R13.P$1
- new net N$16: C6.1, R10.2, R9.1, U$2.3
- new net N$5: C4.1, U5.1
- new net N$9: C5.1, R11.1, R13.P$2, U$2.4
- new net RING1: C2.2, R6.2, R7.1, U2.11
- new net TIP: C3.1, R12.2, R5.2, U2.10
- net 12: no longer J3.RING1
- net 13: no longer J3.TIP
- net 3.3V: now also C9.1, R5.1, R7.2, R9.2, U$2.5, U5.5
- net 35: no longer R5.2
- net GND: now also C6.2, C9.2, R10.1, R12.1, R14.1, R15.1, R6.1, U$2.2, U5.2, U5.4, U5.6; no longer C2.2, C3.2, U1.3, U1.7, U1.8, U1.9
- net N$6: now also C3.2, J3.TIP, R15.2; no longer R5.1, U1.6
- net N$7: now also C2.1, J3.RING1, R14.2; no longer R6.1, U2.11
- net V_USB: no longer C2.1, C3.1, U1.2, U1.5
Routing:
- net 3.3V: track 77.8 -> 121.2 mm, vias 6 -> 9
- net 12: track 41.8 -> 0.00 mm
- net V_USB: track 130.1 -> 91.7 mm, vias 5 -> 3
- net TIP: track 0.00 -> 36.2 mm, vias 0 -> 2
- net 13: track 35.3 -> 0.00 mm
- net RING1: track 0.00 -> 33.4 mm
- net 26: track 25.3 -> 0.00 mm, vias 2 -> 0
- net 35: track 22.9 -> 0.00 mm
- net 25: track 16.1 -> 0.00 mm, vias 2 -> 0
- net N$9: track 0.00 -> 11.0 mm
- net N$7: track 3.40 -> 13.6 mm
- net MIC: track 0.00 -> 7.98 mm
- net N$11: track 0.00 -> 6.03 mm
- net N$16: track 0.00 -> 5.73 mm
- net N$6: track 2.09 -> 5.87 mm
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Other:
- board text added: "RST"
- board text added: "v11"
- board text removed: "v10"

Commit message: partially through layout
Parts:
- removed J1: 455-1750-1-ND, SparkFun-Connectors:1X03
- added D1, D10, D100, D101, D102, D103, D104, D105, D106, D107, D108, D109, D11, D110, D111, D112, D113, D114, D115, D116, D117, D118, D119, D12, D120, D121, D122, D123, D124, D125, D126, D127, D128, D129, D13, D130, D131, D132, D133, D134, D135, D136, D137, D138, D139, D14, D140, D141, D142, D143, D144, D145, D146, D147, D148, D149, D15, D150, D151, D152, D153, D154, D155, D156, D157, D158, D159, D16, D160, D161, D162, D163, D164, D165, D166, D167, D168, D169, D17, D170, D171, D172, D173, D174, D175, D176, D177, D178, D179, D18, D180, D181, D182, D183, D184, D185, D186, D187, D188, D189, D19, D190, D191, D192, D193, D194, D195, D196, D197, D198, D199, D2, D20, D200, D201, D202, D203, D204, D205, D206, D207, D208, D209, D21, D210, D211, D212, D213, D214, D215, D216, D217, D218, D219, D22, D220, D221, D222, D223, D224, D225, D226, D227, D228, D229, D23, D230, D231, D232, D233, D234, D235, D236, D237, D238, D239, D24, D240, D241, D242, D243, D244, D245, D246, D247, D248, D249, D25, D250, D251, D252, D253, D254, D255, D256, D257, D258, D259, D26, D260, D261, D262, D263, D27, D28, D29, D3, D30, D31, D32, D33, D34, D35, D36, D37, D38, D39, D4, D40, D41, D42, D43, D44, D45, D46, D47, D48, D49, D5, D50, D51, D52, D53, D54, D55, D56, D57, D58, D59, D6, D60, D61, D62, D63, D64, D65, D66, D67, D68, D69, D7, D70, D71, D72, D73, D74, D75, D76, D77, D78, D79, D8, D80, D81, D82, D83, D84, D85, D86, D87, D88, D89, D9, D90, D91, D92, D93, D94, D95, D96, D97, D98, D99: WS2812B, SparkFun-LED:WS2812B
- added FRAME2, FRAME3, FRAME4: FRAME-LEDGER, SparkFun-Aesthetics:CREATIVE_COMMONS
- added JP1, JP10, JP100, JP101, JP102, JP103, JP104, JP105, JP106, JP107, JP108, JP109, JP11, JP110, JP111, JP112, JP113, JP114, JP115, JP116, JP117, JP118, JP119, JP12, JP120, JP121, JP122, JP123, JP124, JP125, JP126, JP127, JP128, JP129, JP13, JP130, JP131, JP132, JP133, JP134, JP135, JP136, JP137, JP138, JP139, JP14, JP140, JP141, JP142, JP143, JP144, JP145, JP146, JP147, JP148, JP149, JP15, JP150, JP151, JP152, JP153, JP154, JP155, JP156, JP157, JP158, JP159, JP16, JP160, JP161, JP162, JP163, JP164, JP165, JP166, JP167, JP168, JP169, JP17, JP170, JP171, JP172, JP173, JP174, JP175, JP176, JP177, JP178, JP179, JP18, JP180, JP181, JP182, JP183, JP184, JP185, JP186, JP187, JP188, JP189, JP19, JP190, JP191, JP192, JP193, JP194, JP195, JP196, JP197, JP198, JP199, JP2, JP20, JP200, JP201, JP202, JP203, JP204, JP205, JP206, JP207, JP208, JP209, JP21, JP210, JP211, JP212, JP213, JP214, JP215, JP216, JP217, JP218, JP219, JP22, JP220, JP221, JP222, JP223, JP224, JP225, JP226, JP227, JP228, JP229, JP23, JP230, JP231, JP232, JP233, JP234, JP235, JP236, JP237, JP238, JP239, JP24, JP240, JP241, JP242, JP243, JP244, JP245, JP246, JP247, JP248, JP249, JP25, JP250, JP251, JP252, JP253, JP254, JP255, JP256, JP257, JP258, JP259, JP26, JP260, JP261, JP262, JP263, JP27, JP28, JP29, JP3, JP30, JP31, JP32, JP33, JP34, JP35, JP36, JP37, JP38, JP39, JP4, JP40, JP41, JP42, JP43, JP44, JP45, JP46, JP47, JP48, JP49, JP5, JP50, JP51, JP52, JP53, JP54, JP55, JP56, JP57, JP58, JP59, JP6, JP60, JP61, JP62, JP63, JP64, JP65, JP66, JP67, JP68, JP69, JP7, JP70, JP71, JP72, JP73, JP74, JP75, JP76, JP77, JP78, JP79, JP8, JP80, JP81, JP82, JP83, JP84, JP85, JP86, JP87, JP88, JP89, JP9, JP90, JP91, JP92, JP93, JP94, JP95, JP96, JP97, JP98, JP99: JUMPER-SMT_2_NO_NO-SILK, SparkFun-Jumpers:SMT-JUMPER_2_NO_NO-SILK
Connections:
- new net DIO0: D1.4, JP1.1, U2.13
- new net DIO1: D100.4, D101.2, D102.4, D99.2, JP100.1, JP101.2, JP102.1, JP99.2
- new net DIO10: D21.2, D22.4, JP21.2, JP22.1
- new net DIO100: D191.2, D192.4, JP191.2, JP192.1
- new net DIO101: D193.2, D194.4, JP193.2, JP194.1
- new net DIO102: D195.2, D196.4, JP195.2, JP196.1
- new net DIO103: D197.2, D198.4, JP197.2, JP198.1
- new net DIO104: D209.2, D210.4, JP209.2, JP210.1
- new net DIO105: D202.2, D203.4, JP202.2, JP203.1
- new net DIO106: D204.2, D205.4, JP204.2, JP205.1
- new net DIO107: D206.2, D207.4, JP206.2, JP207.1
- new net DIO108: D208.2, D209.4, JP208.2, JP209.1
- new net DIO109: D211.2, D212.4, JP211.2, JP212.1
- new net DIO11: D22.2, D23.4, JP22.2, JP23.1
- new net DIO110: D213.2, D214.4, JP213.2, JP214.1
- new net DIO111: D215.2, D216.4, JP215.2, JP216.1
- new net DIO112: D217.2, D218.4, JP217.2, JP218.1
- new net DIO113: D219.2, D220.4, JP219.2, JP220.1
- new net DIO114: D220.2, D221.4, JP220.2, JP221.1
- new net DIO115: D222.2, D223.4, JP222.2, JP223.1
- new net DIO116: D224.2, D225.4, JP224.2, JP225.1
- new net DIO117: D226.2, D227.4, JP226.2, JP227.1
- new net DIO118: D228.2, D229.4, JP228.2, JP229.1
- new net DIO119: D230.2, D231.4, JP230.2, JP231.1
- new net DIO12: D24.2, D25.4, JP24.2, JP25.1
- new net DIO120: D231.2, JP231.2
- new net DIO121: D232.4, JP232.1
- new net DIO122: D233.2, D234.4, JP233.2, JP234.1
- new net DIO123: D235.2, D236.4, JP235.2, JP236.1
- new net DIO124: D237.2, D238.4, JP237.2, JP238.1
- new net DIO125: D239.2, D240.4, JP239.2, JP240.1
- new net DIO126: D241.2, D242.4, JP241.2, JP242.1
- new net DIO128: D242.2, D243.4, JP242.2, JP243.1
- new net DIO129: D244.2, D245.4, JP244.2, JP245.1
- new net DIO13: D26.2, D27.4, JP26.2, JP27.1
- new net DIO130: D246.2, D247.4, JP246.2, JP247.1
- new net DIO131: D248.2, D249.4, JP248.2, JP249.1
- new net DIO132: D250.2, D251.4, JP250.2, JP251.1
- new net DIO133: D252.2, D253.4, JP252.2, JP253.1
- new net DIO134: D253.2, D254.4, JP253.2, JP254.1
- new net DIO135: D255.2, D256.4, JP255.2, JP256.1
- new net DIO136: D257.2, D258.4, JP257.2, JP258.1
- new net DIO137: D259.2, D260.4, JP259.2, JP260.1
- new net DIO138: D261.2, D262.4, JP261.2, JP262.1
- new net DIO139: D263.2, JP263.2
- new net DIO14: D28.2, D29.4, JP28.2, JP29.1
- new net DIO15: D30.2, D31.4, JP30.2, JP31.1
- new net DIO16: D32.2, D33.4, JP32.2, JP33.1
- new net DIO17: D33.2, D34.4, JP33.2, JP34.1
- new net DIO18: D35.2, D36.4, JP35.2, JP36.1
- new net DIO19: D37.2, D38.4, JP37.2, JP38.1
- new net DIO2: D198.2, D199.4, JP198.2, JP199.1
- new net DIO20: D39.2, D40.4, JP39.2, JP40.1
- new net DIO21: D41.2, D42.4, JP41.2, JP42.1
- new net DIO22: D43.2, D44.4, JP43.2, JP44.1
- new net DIO23: D44.2, D45.4, JP44.2, JP45.1
- new net DIO24: D46.2, D47.4, JP46.2, JP47.1
- new net DIO25: D48.2, D49.4, JP48.2, JP49.1
- new net DIO26: D50.2, D51.4, JP50.2, JP51.1
- new net DIO27: D52.2, D53.4, JP52.2, JP53.1
- new net DIO28: D54.2, D55.4, JP54.2, JP55.1
- new net DIO29: D55.2, D56.4, JP55.2, JP56.1
- new net DIO3: D6.2, D7.4, JP6.2, JP7.1
- new net DIO30: D57.2, D58.4, JP57.2, JP58.1
- new net DIO31: D59.2, D60.4, JP59.2, JP60.1
- new net DIO32: D61.2, D62.4, JP61.2, JP62.1
- new net DIO33: D63.2, D64.4, JP63.2, JP64.1
- new net DIO34: D65.2, D66.4, JP65.2, JP66.1
- new net DIO35: D66.2, D67.4, JP66.2, JP67.1
- new net DIO36: D68.2, D69.4, JP68.2, JP69.1
- new net DIO37: D70.2, D71.4, JP70.2, JP71.1
- new net DIO38: D72.2, D73.4, JP72.2, JP73.1
- new net DIO39: D74.2, D75.4, JP74.2, JP75.1
- new net DIO4: D8.2, D9.4, JP8.2, JP9.1
- new net DIO40: D76.2, D77.4, JP76.2, JP77.1
- new net DIO41: D77.2, D78.4, JP77.2, JP78.1
- new net DIO42: D79.2, D80.4, JP79.2, JP80.1
- new net DIO43: D81.2, D82.4, JP81.2, JP82.1
- new net DIO44: D83.2, D84.4, JP83.2, JP84.1
- new net DIO45: D85.2, D86.4, JP85.2, JP86.1
- new net DIO46: D87.2, D88.4, JP87.2, JP88.1
- new net DIO47: D88.2, D89.4, JP88.2, JP89.1
- new net DIO48: D90.2, D91.4, JP90.2, JP91.1
- new net DIO49: D92.2, D93.4, JP92.2, JP93.1
- new net DIO5: D10.2, D11.4, JP10.2, JP11.1
- new net DIO50: D94.2, D95.4, JP94.2, JP95.1
- new net DIO51: D96.2, D97.4, JP96.2, JP97.1
- new net DIO52: D98.2, D99.4, JP98.2, JP99.1
- new net DIO53: D103.2, D104.4, JP103.2, JP104.1
- new net DIO54: D105.2, D106.4, JP105.2, JP106.1
- new net DIO55: D107.2, D108.4, JP107.2, JP108.1
- new net DIO56: D109.2, D110.4, JP109.2, JP110.1
- new net DIO57: D112.2, D113.4, JP112.2, JP113.1
- new net DIO58: D114.2, D115.4, JP114.2, JP115.1
- new net DIO59: D116.2, D117.4, JP116.2, JP117.1
- new net DIO6: D13.2, D14.4, JP13.2, JP14.1
- new net DIO60: D118.2, D119.4, JP118.2, JP119.1
- new net DIO61: D120.2, D121.4, JP120.2, JP121.1
- new net DIO62: D121.2, D122.4, JP121.2, JP122.1
- new net DIO63: D123.2, D124.4, JP123.2, JP124.1
- new net DIO64: D125.2, D126.4, JP125.2, JP126.1
- new net DIO65: D127.2, D128.4, JP127.2, JP128.1
- new net DIO66: D129.2, D130.4, JP129.2, JP130.1
- new net DIO67: D131.2, D132.4, JP131.2, JP132.1
- new net DIO68: D132.2, D133.4, JP132.2, JP133.1
- new net DIO69: D134.2, D135.4, JP134.2, JP135.1
- new net DIO7: D15.2, D16.4, JP15.2, JP16.1
- new net DIO70: D136.2, D137.4, JP136.2, JP137.1
- new net DIO71: D138.2, D139.4, JP138.2, JP139.1
- new net DIO72: D140.2, D141.4, JP140.2, JP141.1
- new net DIO73: D142.2, D143.4, JP142.2, JP143.1
- new net DIO74: D143.2, D144.4, JP143.2, JP144.1
- new net DIO75: D145.2, D146.4, JP145.2, JP146.1
- new net DIO76: D147.2, D148.4, JP147.2, JP148.1
- new net DIO77: D149.2, D150.4, JP149.2, JP150.1
- new net DIO78: D151.2, D152.4, JP151.2, JP152.1
- new net DIO79: D153.2, D154.4, JP153.2, JP154.1
- new net DIO8: D17.2, D18.4, JP17.2, JP18.1
- new net DIO80: D154.2, D155.4, JP154.2, JP155.1
- new net DIO81: D156.2, D157.4, JP156.2, JP157.1
- new net DIO82: D158.2, D159.4, JP158.2, JP159.1
- new net DIO83: D160.2, D161.4, JP160.2, JP161.1
- new net DIO84: D162.2, D163.4, JP162.2, JP163.1
- new net DIO85: D164.2, D165.4, JP164.2, JP165.1
- new net DIO86: D165.2, D166.4, JP165.2, JP166.1
- new net DIO87: D167.2, D168.4, JP167.2, JP168.1
- new net DIO88: D169.2, D170.4, JP169.2, JP170.1
- new net DIO89: D171.2, D172.4, JP171.2, JP172.1
- new net DIO9: D19.2, D20.4, JP19.2, JP20.1
- new net DIO90: D173.2, D174.4, JP173.2, JP174.1
- new net DIO91: D175.2, D176.4, JP175.2, JP176.1
- new net DIO92: D176.2, D177.4, JP176.2, JP177.1
- new net DIO93: D178.2, D179.4, JP178.2, JP179.1
- new net DIO94: D180.2, D181.4, JP180.2, JP181.1
- new net DIO95: D182.2, D183.4, JP182.2, JP183.1
- new net DIO96: D184.2, D185.4, JP184.2, JP185.1
- new net DIO97: D186.2, D187.4, JP186.2, JP187.1
- new net DIO98: D187.2, D188.4, JP187.2, JP188.1
- new net DIO99: D189.2, D190.4, JP189.2, JP190.1
- new net N$100: D196.2, D197.4, JP196.2, JP197.1
- new net N$101: D194.2, D195.4, JP194.2, JP195.1
- new net N$102: D199.2, D200.4, JP199.2, JP200.1
- new net N$103: D203.2, D204.4, JP203.2, JP204.1
- new net N$104: D201.2, D202.4, JP201.2, JP202.1
- new net N$105: D207.2, D208.4, JP207.2, JP208.1
- new net N$106: D205.2, D206.4, JP205.2, JP206.1
- new net N$107: D210.2, D211.4, JP210.2, JP211.1
- new net N$108: D214.2, D215.4, JP214.2, JP215.1
- new net N$109: D212.2, D213.4, JP212.2, JP213.1
- new net N$110: D218.2, D219.4, JP218.2, JP219.1
- new net N$111: D216.2, D217.4, JP216.2, JP217.1
- new net N$112: D221.2, D222.4, JP221.2, JP222.1
- new net N$113: D225.2, D226.4, JP225.2, JP226.1
- new net N$114: D223.2, D224.4, JP223.2, JP224.1
- new net N$115: D229.2, D230.4, JP229.2, JP230.1
- new net N$116: D227.2, D228.4, JP227.2, JP228.1
- new net N$117: D232.2, D233.4, JP232.2, JP233.1
- new net N$118: D236.2, D237.4, JP236.2, JP237.1
- new net N$119: D234.2, D235.4, JP234.2, JP235.1
- new net N$120: D2.2, D3.4, JP2.2, JP3.1
- new net N$121: D4.2, D5.4, JP4.2, JP5.1
- new net N$122: D240.2, D241.4, JP240.2, JP241.1
- new net N$123: D238.2, D239.4, JP238.2, JP239.1
- new net N$124: D243.2, D244.4, JP243.2, JP244.1
- new net N$125: D247.2, D248.4, JP247.2, JP248.1
- new net N$126: D245.2, D246.4, JP245.2, JP246.1
- new net N$127: D251.2, D252.4, JP251.2, JP252.1
- new net N$128: D249.2, D250.4, JP249.2, JP250.1
- new net N$129: D254.2, D255.4, JP254.2, JP255.1
- new net N$13: D3.2, D4.4, JP3.2, JP4.1
- new net N$130: D258.2, D259.4, JP258.2, JP259.1
- new net N$131: D256.2, D257.4, JP256.2, JP257.1
- new net N$132: D262.2, D263.4, JP262.2, JP263.1
- new net N$133: D260.2, D261.4, JP260.2, JP261.1
- new net N$134: D110.2, D111.4, JP110.2, JP111.1
- new net N$135: D11.2, D12.4, JP11.2, JP12.1
- new net N$136: D200.2, D201.4, JP200.2, JP201.1
- new net N$14: D5.2, D6.4, JP5.2, JP6.1
- new net N$15: D10.4, D9.2, JP10.1, JP9.2
- new net N$17: D7.2, D8.4, JP7.2, JP8.1
- new net N$18: D16.2, D17.4, JP16.2, JP17.1
- new net N$19: D23.2, D24.4, JP23.2, JP24.1
- new net N$20: D14.2, D15.4, JP14.2, JP15.1
- new net N$21: D20.2, D21.4, JP20.2, JP21.1
- new net N$22: D18.2, D19.4, JP18.2, JP19.1
- new net N$23: D100.2, D101.4, JP100.2, JP101.1
- new net N$24: D27.2, D28.4, JP27.2, JP28.1
- new net N$25: D25.2, D26.4, JP25.2, JP26.1
- new net N$26: D31.2, D32.4, JP31.2, JP32.1
- new net N$27: D29.2, D30.4, JP29.2, JP30.1
- new net N$28: D104.2, D105.4, JP104.2, JP105.1
- new net N$29: D34.2, D35.4, JP34.2, JP35.1
- new net N$30: D38.2, D39.4, JP38.2, JP39.1
- new net N$31: D36.2, D37.4, JP36.2, JP37.1
- new net N$32: D42.2, D43.4, JP42.2, JP43.1
- new net N$33: D40.2, D41.4, JP40.2, JP41.1
- new net N$34: D45.2, D46.4, JP45.2, JP46.1
- new net N$35: D49.2, D50.4, JP49.2, JP50.1
- new net N$36: D47.2, D48.4, JP47.2, JP48.1
- new net N$37: D53.2, D54.4, JP53.2, JP54.1
- new net N$38: D51.2, D52.4, JP51.2, JP52.1
- new net N$39: D102.2, D103.4, JP102.2, JP103.1
- new net N$40: D56.2, D57.4, JP56.2, JP57.1
- new net N$41: D60.2, D61.4, JP60.2, JP61.1
- new net N$42: D58.2, D59.4, JP58.2, JP59.1
- new net N$43: D64.2, D65.4, JP64.2, JP65.1
- new net N$44: D62.2, D63.4, JP62.2, JP63.1
- new net N$45: D67.2, D68.4, JP67.2, JP68.1
- new net N$46: D71.2, D72.4, JP71.2, JP72.1
- new net N$47: D69.2, D70.4, JP69.2, JP70.1
- new net N$48: D75.2, D76.4, JP75.2, JP76.1
- new net N$49: D73.2, D74.4, JP73.2, JP74.1
- new net N$50: D78.2, D79.4, JP78.2, JP79.1
- new net N$51: D82.2, D83.4, JP82.2, JP83.1
- new net N$52: D80.2, D81.4, JP80.2, JP81.1
- new net N$53: D86.2, D87.4, JP86.2, JP87.1
- new net N$54: D84.2, D85.4, JP84.2, JP85.1
- new net N$55: D89.2, D90.4, JP89.2, JP90.1
- new net N$56: D93.2, D94.4, JP93.2, JP94.1
- new net N$57: D91.2, D92.4, JP91.2, JP92.1
- new net N$58: D97.2, D98.4, JP97.2, JP98.1
- new net N$59: D95.2, D96.4, JP95.2, JP96.1
- new net N$60: D108.2, D109.4, JP108.2, JP109.1
- new net N$61: D106.2, D107.4, JP106.2, JP107.1
- new net N$62: D111.2, D112.4, JP111.2, JP112.1
- new net N$63: D115.2, D116.4, JP115.2, JP116.1
- new net N$64: D113.2, D114.4, JP113.2, JP114.1
- new net N$65: D119.2, D120.4, JP119.2, JP120.1
- new net N$66: D117.2, D118.4, JP117.2, JP118.1
- new net N$67: D122.2, D123.4, JP122.2, JP123.1
- new net N$68: D126.2, D127.4, JP126.2, JP127.1
- new net N$69: D124.2, D125.4, JP124.2, JP125.1
- new net N$70: D130.2, D131.4, JP130.2, JP131.1
- new net N$71: D128.2, D129.4, JP128.2, JP129.1
- new net N$72: D133.2, D134.4, JP133.2, JP134.1
- new net N$73: D137.2, D138.4, JP137.2, JP138.1
- new net N$74: D135.2, D136.4, JP135.2, JP136.1
- new net N$75: D141.2, D142.4, JP141.2, JP142.1
- new net N$76: D139.2, D140.4, JP139.2, JP140.1
- new net N$77: D144.2, D145.4, JP144.2, JP145.1
- new net N$78: D148.2, D149.4, JP148.2, JP149.1
- new net N$79: D146.2, D147.4, JP146.2, JP147.1
- new net N$8: D12.2, D13.4, JP12.2, JP13.1
- new net N$80: D152.2, D153.4, JP152.2, JP153.1
- new net N$81: D150.2, D151.4, JP150.2, JP151.1
- new net N$82: D155.2, D156.4, JP155.2, JP156.1
- new net N$83: D159.2, D160.4, JP159.2, JP160.1
- new net N$84: D157.2, D158.4, JP157.2, JP158.1
- new net N$85: D163.2, D164.4, JP163.2, JP164.1
- new net N$86: D161.2, D162.4, JP161.2, JP162.1
- new net N$87: D166.2, D167.4, JP166.2, JP167.1
- new net N$88: D170.2, D171.4, JP170.2, JP171.1
- new net N$89: D168.2, D169.4, JP168.2, JP169.1
- new net N$90: D174.2, D175.4, JP174.2, JP175.1
- new net N$91: D172.2, D173.4, JP172.2, JP173.1
- new net N$92: D177.2, D178.4, JP177.2, JP178.1
- new net N$93: D181.2, D182.4, JP181.2, JP182.1
- new net N$94: D179.2, D180.4, JP179.2, JP180.1
- new net N$95: D185.2, D186.4, JP185.2, JP186.1
- new net N$96: D183.2, D184.4, JP183.2, JP184.1
- new net N$97: D188.2, D189.4, JP188.2, JP189.1
- new net N$98: D192.2, D193.4, JP192.2, JP193.1
- new net N$99: D190.2, D191.4, JP190.2, JP191.1
- net GND: now also D1.3, D10.3, D100.3, D101.3, D102.3, D103.3, D104.3, D105.3, D106.3, D107.3, D108.3, D109.3, D11.3, D110.3, D111.3, D112.3, D113.3, D114.3, D115.3, D116.3, D117.3, D118.3, D119.3, D12.3, D120.3, D121.3, D122.3, D123.3, D124.3, D125.3, D126.3, D127.3, D128.3, D129.3, D13.3, D130.3, D131.3, D132.3, D133.3, D134.3, D135.3, D136.3, D137.3, D138.3, D139.3, D14.3, D140.3, D141.3, D142.3, D143.3, D144.3, D145.3, D146.3, D147.3, D148.3, D149.3, D15.3, D150.3, D151.3, D152.3, D153.3, D154.3, D155.3, D156.3, D157.3, D158.3, D159.3, D16.3, D160.3, D161.3, D162.3, D163.3, D164.3, D165.3, D166.3, D167.3, D168.3, D169.3, D17.3, D170.3, D171.3, D172.3, D173.3, D174.3, D175.3, D176.3, D177.3, D178.3, D179.3, D18.3, D180.3, D181.3, D182.3, D183.3, D184.3, D185.3, D186.3, D187.3, D188.3, D189.3, D19.3, D190.3, D191.3, D192.3, D193.3, D194.3, D195.3, D196.3, D197.3, D198.3, D199.3, D2.3, D20.3, D200.3, D201.3, D202.3, D203.3, D204.3, D205.3, D206.3, D207.3, D208.3, D209.3, D21.3, D210.3, D211.3, D212.3, D213.3, D214.3, D215.3, D216.3, D217.3, D218.3, D219.3, D22.3, D220.3, D221.3, D222.3, D223.3, D224.3, D225.3, D226.3, D227.3, D228.3, D229.3, D23.3, D230.3, D231.3, D232.3, D233.3, D234.3, D235.3, D236.3, D237.3, D238.3, D239.3, D24.3, D240.3, D241.3, D242.3, D243.3, D244.3, D245.3, D246.3, D247.3, D248.3, D249.3, D25.3, D250.3, D251.3, D252.3, D253.3, D254.3, D255.3, D256.3, D257.3, D258.3, D259.3, D26.3, D260.3, D261.3, D262.3, D263.3, D27.3, D28.3, D29.3, D3.3, D30.3, D31.3, D32.3, D33.3, D34.3, D35.3, D36.3, D37.3, D38.3, D39.3, D4.3, D40.3, D41.3, D42.3, D43.3, D44.3, D45.3, D46.3, D47.3, D48.3, D49.3, D5.3, D50.3, D51.3, D52.3, D53.3, D54.3, D55.3, D56.3, D57.3, D58.3, D59.3, D6.3, D60.3, D61.3, D62.3, D63.3, D64.3, D65.3, D66.3, D67.3, D68.3, D69.3, D7.3, D70.3, D71.3, D72.3, D73.3, D74.3, D75.3, D76.3, D77.3, D78.3, D79.3, D8.3, D80.3, D81.3, D82.3, D83.3, D84.3, D85.3, D86.3, D87.3, D88.3, D89.3, D9.3, D90.3, D91.3, D92.3, D93.3, D94.3, D95.3, D96.3, D97.3, D98.3, D99.3; no longer J1.1
- net N$2: now also D1.2, D2.4, JP1.2, JP2.1; no longer J1.2, U2.13
- net V_USB: now also D1.1, D10.1, D100.1, D101.1, D102.1, D103.1, D104.1, D105.1, D106.1, D107.1, D108.1, D109.1, D11.1, D110.1, D111.1, D112.1, D113.1, D114.1, D115.1, D116.1, D117.1, D118.1, D119.1, D12.1, D120.1, D121.1, D122.1, D123.1, D124.1, D125.1, D126.1, D127.1, D128.1, D129.1, D13.1, D130.1, D131.1, D132.1, D133.1, D134.1, D135.1, D136.1, D137.1, D138.1, D139.1, D14.1, D140.1, D141.1, D142.1, D143.1, D144.1, D145.1, D146.1, D147.1, D148.1, D149.1, D15.1, D150.1, D151.1, D152.1, D153.1, D154.1, D155.1, D156.1, D157.1, D158.1, D159.1, D16.1, D160.1, D161.1, D162.1, D163.1, D164.1, D165.1, D166.1, D167.1, D168.1, D169.1, D17.1, D170.1, D171.1, D172.1, D173.1, D174.1, D175.1, D176.1, D177.1, D178.1, D179.1, D18.1, D180.1, D181.1, D182.1, D183.1, D184.1, D185.1, D186.1, D187.1, D188.1, D189.1, D19.1, D190.1, D191.1, D192.1, D193.1, D194.1, D195.1, D196.1, D197.1, D198.1, D199.1, D2.1, D20.1, D200.1, D201.1, D202.1, D203.1, D204.1, D205.1, D206.1, D207.1, D208.1, D209.1, D21.1, D210.1, D211.1, D212.1, D213.1, D214.1, D215.1, D216.1, D217.1, D218.1, D219.1, D22.1, D220.1, D221.1, D222.1, D223.1, D224.1, D225.1, D226.1, D227.1, D228.1, D229.1, D23.1, D230.1, D231.1, D232.1, D233.1, D234.1, D235.1, D236.1, D237.1, D238.1, D239.1, D24.1, D240.1, D241.1, D242.1, D243.1, D244.1, D245.1, D246.1, D247.1, D248.1, D249.1, D25.1, D250.1, D251.1, D252.1, D253.1, D254.1, D255.1, D256.1, D257.1, D258.1, D259.1, D26.1, D260.1, D261.1, D262.1, D263.1, D27.1, D28.1, D29.1, D3.1, D30.1, D31.1, D32.1, D33.1, D34.1, D35.1, D36.1, D37.1, D38.1, D39.1, D4.1, D40.1, D41.1, D42.1, D43.1, D44.1, D45.1, D46.1, D47.1, D48.1, D49.1, D5.1, D50.1, D51.1, D52.1, D53.1, D54.1, D55.1, D56.1, D57.1, D58.1, D59.1, D6.1, D60.1, D61.1, D62.1, D63.1, D64.1, D65.1, D66.1, D67.1, D68.1, D69.1, D7.1, D70.1, D71.1, D72.1, D73.1, D74.1, D75.1, D76.1, D77.1, D78.1, D79.1, D8.1, D80.1, D81.1, D82.1, D83.1, D84.1, D85.1, D86.1, D87.1, D88.1, D89.1, D9.1, D90.1, D91.1, D92.1, D93.1, D94.1, D95.1, D96.1, D97.1, D98.1, D99.1; no longer J1.3
Routing:
- net V_USB: track 91.7 -> 428.5 mm, vias 3 -> 250
- net DIO1: track 0.00 -> 33.7 mm
- net 3.3V: track 121.2 -> 153.4 mm
- net DIO115: track 0.00 -> 16.9 mm
- net N$65: track 0.00 -> 16.9 mm
- net N$56: track 0.00 -> 16.9 mm
- net N$48: track 0.00 -> 16.9 mm
- net N$31: track 0.00 -> 16.9 mm
- net N$20: track 0.00 -> 16.9 mm
- net N$135: track 0.00 -> 16.9 mm
- net DIO71: track 0.00 -> 16.9 mm
- net DIO60: track 0.00 -> 16.9 mm
- net DIO52: track 0.00 -> 16.9 mm
- net N$35: track 0.00 -> 16.9 mm
- net N$134: track 0.00 -> 16.9 mm
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- added copper zone on layer 16, net V_USB
- removed copper zone on layer 16, net GND
Other:
- board size 66 x 31.8 mm -> 316.5 x 197.8 mm
