File: Hardware/ESP32_Thing_Plus.brd (EAGLE design)
At the start: 316.5 x 197.8 mm, 570 parts, among them J2 USB Female Type C Connector, J3 AUDIO_JACK_TRRSSMD_RA, Q2 MBT3904DW1T1, U2 ESP-WROOM-32NARROW, U3 AP2112K-3.3V, U4 CP2102N, U5 ADMP401

Commit message: completing initial 13 in layout, ready for design review with jason
Connections:
- removed net DIO121: D232.4, JP232.1
- net DIO120: now also D232.4, JP232.1
Routing:
- net N$89: track 5.67 -> 319.1 mm, vias 0 -> 2
- net N$68: track 5.67 -> 319.1 mm, vias 0 -> 2
- net DIO99: track 5.67 -> 319.1 mm, vias 0 -> 2
- net DIO76: track 5.67 -> 319.1 mm, vias 0 -> 2
- net DIO54: track 5.67 -> 319.1 mm, vias 0 -> 2
- net N$54: track 5.67 -> 318.9 mm, vias 0 -> 2
- net DIO109: track 5.67 -> 304.1 mm, vias 0 -> 2
- net DIO120: track 2.83 -> 243.9 mm, vias 0 -> 2
- net N$125: track 5.67 -> 244.1 mm, vias 0 -> 2
- net V_USB: track 443.5 -> 533.5 mm, vias 263 -> 269
- net 3.3V: track 149.1 -> 146.1 mm
- net DIO121: track 2.83 -> 0.00 mm
- net DIO0: track 208.1 -> 205.7 mm
- added copper zone on layer 16, net GND
