File: Hardware/ESP32_Thing_Plus.sch (EAGLE design)
At the start: 573 parts, among them J2 USB Female Type C Connector, J3 AUDIO_JACK_TRRSSMD_RA, Q2 MBT3904DW1T1, U2 ESP-WROOM-32NARROW, U3 AP2112K-3.3V, U4 CP2102N, U5 ADMP401

Commit message: updating layout, fixing bad commit
Parts:
- removed D211, D263: WS2812B, SparkFun-LED:WS2812B
- removed JP211, JP263: JUMPER-SMT_2_NO_NO-SILK, SparkFun-Jumpers:JUMPER-SMT_2_NO_NO-SILK
- removed U$1: 47uF/6.3V, SparkFun-Capacitors:47UF
- added R16: 100, SparkFun-Resistors:100OHM-0603-1/4W-5%
- R8: value 100k -> 100K; device SparkFun-Resistors:100KOHM-0603-1/10W-1% -> SparkFun-Resistors:100KOHM-0402-1/16W-1%
Connections:
- removed net DIO139: D263.DO, JP263.2
- new net N$137: R16.2, U4.VBUS, U4.VREGIN
- net DIO1: no longer D101.DO, D102.DI, JP101.2, JP102.1
- net DIO109: now also D210.DO, JP210.2; no longer D211.DO, JP211.2
- net GND: no longer D211.VSS, D263.VSS, U$1.2
- net N$107: now also D101.DO, D102.DI, JP101.2, JP102.1; no longer D210.DO, D211.DI, JP210.2, JP211.1
- net N$132: no longer D263.DI, JP263.1
- net V_USB: now also R16.1; no longer D211.VDD, D263.VDD, U$1.1, U4.VBUS, U4.VREGIN

Commit message: completing initial 13 in layout, ready for design review with jason
Connections:
- removed net DIO121: D232.DI, JP232.1
- net DIO120: now also D232.DI, JP232.1
Changed lines of the file:
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@@
 <wire x1="20.32" y1="198.12" x2="419.1" y2="198.12" width="0.1524" layer="91"/>
 <wire x1="419.1" y1="198.12" x2="419.1" y2="208.28" width="0.1524" layer="91"/>
+<pinref part="D232" gate="G$1" pin="DI"/>
+<wire x1="27.94" y1="182.88" x2="20.32" y2="182.88" width="0.1524" layer="91"/>
+<wire x1="20.32" y1="182.88" x2="20.32" y2="175.26" width="0.1524" layer="91"/>
+<pinref part="JP232" gate="G$1" pin="1"/>
+<wire x1="20.32" y1="175.26" x2="35.56" y2="175.26" width="0.1524" layer="91"/>
+<wire x1="20.32" y1="198.12" x2="20.32" y2="182.88" width="0.1524" layer="91"/>
+<junction x="20.32" y="182.88"/>
 </segment>
 </net>
@@
 </segment>
 </net>
-<net name="DIO121" class="0">
-<segment>
-<pinref part="D232" gate="G$1" pin="DI"/>
-<wire x1="27.94" y1="182.88" x2="20.32" y2="182.88" width="0.1524" layer="91"/>
-<wire x1="20.32" y1="182.88" x2="20.32" y2="175.26" width="0.1524" layer="91"/>
-<pinref part="JP232" gate="G$1" pin="1"/>
-<wire x1="20.32" y1="175.26" x2="35.56" y2="175.26" width="0.1524" layer="91"/>
-<wire x1="20.32" y1="198.12" x2="20.32" y2="182.88" width="0.1524" layer="91"/>
-<junction x="20.32" y="182.88"/>
-</segment>
-</net>
