File: Hardware/BASE.brd (EAGLE design)
At the start: 326.5 x 197.8 mm, 569 parts, among them J2 USB Female Type C Connector, J3 AUDIO_JACK_TRRSSMD_RA, Q2 MBT3904DW1T1, U2 ESP-WROOM-32NARROW, U3 AP2112K-3.3V, U4 CP2102N, U5 ADMP401

Commit message: updating 13 inch, finish layout of 15 inch
Parts:
- R13: value 1k -> 2.2k; device SparkFun-Resistors:AXIAL-0.3 -> SparkFun-Resistors:0603
- moved J3 333.3 mm to (324.5, 30.1), turned to 180 degrees
- moved J2 322.3 mm to (319.0, 47.4), turned to 90 degrees
- moved R3 316.2 mm to (315.8, 48.8), turned to 0 degrees
- moved R4 315.7 mm to (315.8, 46.3), turned to 0 degrees
- moved R14 312.8 mm to (318.0, 35.5), turned to 180 degrees
- moved R6 312.4 mm to (320.0, 38.0), turned to 90 degrees
- moved C2 310.4 mm to (318.0, 38.0), turned to 90 degrees
- moved R15 310.0 mm to (315.0, 23.5), turned to 0 degrees
- moved R5 309.5 mm to (317.0, 21.0), turned to 270 degrees
- moved R7 308.3 mm to (316.0, 38.0), turned to 270 degrees
- moved C3 307.6 mm to (315.0, 21.0), turned to 90 degrees
- moved R12 305.7 mm to (313.0, 21.0), turned to 270 degrees
- moved U5 53.9 mm to (18.5, 17.4), turned to 270 degrees
- moved R10 47.9 mm to (25.5, 14.8), turned to 270 degrees
- moved R13 47.9 mm to (28.7, 11.5), turned to 0 degrees
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Connections:
- net N$11: now also R13.1; no longer R13.P$1
- net N$9: now also R13.2; no longer R13.P$2
Routing:
- net D-: track 31.8 -> 333.3 mm
- net D+: track 31.5 -> 331.8 mm
- net 3.3V: track 167.3 -> 402.2 mm, vias 10 -> 7
- net V_USB: track 553.2 -> 448.5 mm, vias 267 -> 269
- net TIP: track 48.1 -> 19.7 mm, vias 2 -> 0
- net MIC: track 32.4 -> 5.75 mm
- net RING1: track 45.2 -> 28.3 mm
- net DIO0: track 234.7 -> 218.1 mm
- net N$9: track 10.5 -> 6.68 mm
- net N$11: track 5.53 -> 8.15 mm
- net N$7: track 13.6 -> 11.3 mm
- net DIO109: track 304.1 -> 305.1 mm
- net GND: vias 18 -> 16
- net N$109: vias 0 -> 2
Other:
- outline, holes or cut-outs redrawn

Commit message: getting closer to final 15 inch layout
Parts:
- added D1, D21, D211, D263, D264: WS2812B, SparkFun-LED:WS2812B
- added JP1, JP21, JP211, JP263, JP264: JUMPER-SMT_2_NO_NO-SILK, SparkFun-Jumpers:SMT-JUMPER_2_NO_NO-SILK
- moved R11 6.39 mm to (24.7, 18.5), turned to 180 degrees
- moved C5 6.34 mm to (24.7, 16.6), turned to 180 degrees
- moved R5 6.27 mm to (311.8, 17.5), turned to 0 degrees
- moved C6 6.18 mm to (21.4, 13.3)
- moved R10 6.18 mm to (19.5, 13.3)
- moved R9 6.18 mm to (23.3, 13.3)
- moved S1 6.00 mm to (29.6, 6.35)
- moved S2 6.00 mm to (29.6, 2.54)
- moved C4 6.00 mm to (17.6, 17.4)
- moved FD4 6.00 mm to (10.5, 9.00)
- moved Q2 6.00 mm to (24.5, 4.45)
- moved R1 6.00 mm to (16.5, 1.79)
- moved R16 6.00 mm to (14.8, 4.00)
- moved R17 6.00 mm to (24.5, 1.91)
- moved R18 6.00 mm to (24.5, 6.99)
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Connections:
- removed net DIO120: D231.2, D232.4, JP231.2, JP232.1
- new net DIO121: D21.4, D231.2, JP21.1, JP231.2
- new net DIO127: D211.2, D263.4, JP211.2, JP263.1
- new net N$138: D263.2, D264.4, JP263.2, JP264.1
- new net N$140: D232.4, D264.2, JP232.1, JP264.2
- new net N$2: D21.2, D211.4, JP21.2, JP211.1
- new net N$21: D1.2, D212.4, JP1.2, JP212.1
- net DIO109: now also D1.4, JP1.1; no longer D212.4, JP212.1
- net GND: now also D1.3, D21.3, D211.3, D263.3, D264.3
- net V_USB: now also D1.1, D21.1, D211.1, D263.1, D264.1
Routing:
- net TIP: track 19.7 -> 290.9 mm
- net RING1: track 28.3 -> 293.8 mm
- net DIO120: track 243.9 -> 0.00 mm, vias 2 -> 0
- net DIO121: track 0.00 -> 242.1 mm, vias 0 -> 2
- net MIC: track 5.75 -> 30.0 mm
- net N$21: track 0.00 -> 16.8 mm
- net DIO109: track 305.1 -> 320.2 mm
- net V_USB: track 448.5 -> 441.6 mm
- net N$11: track 8.15 -> 13.2 mm
- net 3.3V: track 402.2 -> 406.7 mm, vias 7 -> 8
- net N$9: track 6.68 -> 9.78 mm
- net DIO0: track 218.1 -> 215.4 mm
- net D-: track 333.3 -> 335.4 mm
- net D+: track 331.8 -> 333.5 mm
- net N$6: track 6.14 -> 7.45 mm
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Other:
- outline, holes or cut-outs redrawn
