File: Hardware/BASE.sch (EAGLE design)
At the start: 568 parts, among them J2 USB Female Type C Connector, J3 AUDIO_JACK_TRRSSMD_RA, Q2 MBT3904DW1T1, U2 ESP-WROOM-32NARROW, U3 AP2112K-3.3V, U4 CP2102N, U5 ADMP401

Commit message: updating 13 inch, finish layout of 15 inch
Parts:
- R13: value 1k -> 2.2k; device SparkFun-Resistors:1KOHM-HORIZ-1/4W-5% -> SparkFun-Resistors:2.2KOHM-0603-1/10W-1%
- R16: device SparkFun-Resistors:100OHM-0603-1/4W-5% -> SparkFun-Resistors:100OHM-0603-1/10W-1%
Changed lines of the file:
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@@
 <?xml version="1.0" encoding="utf-8"?>
 <!DOCTYPE eagle SYSTEM "eagle.dtd">
-<eagle version="9.3.1">
+<eagle version="9.5.2">
 <drawing>
 <settings>
@@
 <part name="C6" library="SparkFun-Capacitors" deviceset="1.0UF" device="-0603-16V-10%" value="1.0uF"/>
 <part name="GND13" library="SparkFun-PowerSymbols" deviceset="GND" device=""/>
-<part name="R13" library="SparkFun-Resistors" deviceset="1KOHM" device="-HORIZ-1/4W-5%" value="1k"/>
+<part name="R13" library="SparkFun-Resistors" deviceset="2.2KOHM" device="-0603-1/10W-1%" value="2.2k"/>
 <part name="C9" library="SparkFun-Capacitors" deviceset="0.1UF" device="-0603-25V-5%" value="0.1uF"/>
 <part name="R11" library="SparkFun-Resistors" deviceset="100KOHM" device="-0603-1/10W-1%" value="100k"/>
@@
 <part name="JP261" library="SparkFun-Jumpers" deviceset="JUMPER-SMT_2_NO" device="_NO-SILK" value="JUMPER-SMT_2_NO_NO-SILK"/>
 <part name="JP262" library="SparkFun-Jumpers" deviceset="JUMPER-SMT_2_NO" device="_NO-SILK" value="JUMPER-SMT_2_NO_NO-SILK"/>
-<part name="R16" library="SparkFun-Resistors" deviceset="100OHM" device="-0603-1/4W-5%" value="100"/>
+<part name="R16" library="SparkFun-Resistors" deviceset="100OHM" device="-0603-1/10W-1%" value="100"/>
 <part name="H1" library="SparkFun-Hardware" deviceset="STAND-OFF" device=""/>
 <part name="H2" library="SparkFun-Hardware" deviceset="STAND-OFF" device=""/>

Commit message: getting closer to final 15 inch layout
Parts:
- added D1, D21, D211, D263, D264: WS2812B, SparkFun-LED:WS2812B
- added JP1, JP21, JP211, JP263, JP264: JUMPER-SMT_2_NO_NO-SILK, SparkFun-Jumpers:JUMPER-SMT_2_NO_NO-SILK
Connections:
- removed net DIO120: D231.DO, D232.DI, JP231.2, JP232.1
- new net DIO121: D21.DI, D231.DO, JP21.1, JP231.2
- new net DIO127: D211.DO, D263.DI, JP211.2, JP263.1
- new net N$138: D263.DO, D264.DI, JP263.2, JP264.1
- new net N$140: D232.DI, D264.DO, JP232.1, JP264.2
- new net N$2: D21.DO, D211.DI, JP21.2, JP211.1
- new net N$21: D1.DO, D212.DI, JP1.2, JP212.1
- net DIO109: now also D1.DI, JP1.1; no longer D212.DI, JP212.1
- net GND: now also D1.VSS, D21.VSS, D211.VSS, D263.VSS, D264.VSS
- net V_USB: now also D1.VDD, D21.VDD, D211.VDD, D263.VDD, D264.VDD
