File: Hardware/13NR.brd (EAGLE design)
At the start: 326.5 x 197.8 mm, 569 parts, among them J2 USB Female Type C Connector, J3 AUDIO_JACK_TRRSSMD_RA, Q2 MBT3904DW1T1, U2 ESP-WROOM-32NARROW, U3 AP2112K-3.3V, U4 CP2102N, U5 ADMP401

Commit message: updating 13NR, to move for mounting stuff
Parts:
- moved R8 15.3 mm to (16.0, 5.45)
- moved C8 15.1 mm to (12.1, 9.20)
- moved C1 15.1 mm to (16.0, 12.5)
- moved C7 15.1 mm to (16.0, 14.2)
- moved U3 15.1 mm to (16.0, 9.28)
- moved R9 4.00 mm to (73.2, 18.3)
- moved C4 4.00 mm to (70.6, 12.6)
- moved C5 4.00 mm to (69.4, 20.2)
- moved C6 4.00 mm to (73.2, 16.4)
- moved C9 4.00 mm to (73.2, 24.6)
- moved Q2 4.00 mm to (30.5, 8.45)
- moved R1 4.00 mm to (22.5, 5.79)
- moved R10 4.00 mm to (73.2, 14.5)
- moved R11 4.00 mm to (67.5, 20.2)
- moved R13 4.00 mm to (76.5, 17.7)
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Routing:
- net 3.3V: track 167.3 -> 150.2 mm
- net V_USB: track 553.2 -> 564.0 mm
- net TIP: track 48.1 -> 46.4 mm
- net RING1: track 45.2 -> 43.6 mm
- net DIO0: track 234.7 -> 233.1 mm
- net D+: track 31.5 -> 32.9 mm
- net GND: vias 18 -> 27
Other:
- outline, holes or cut-outs redrawn

Commit message: moving power to other side
Parts:
- removed D12, D252: WS2812B, SparkFun-LED:WS2812B
- removed JP12, JP252: JUMPER-SMT_2_NO_NO-SILK, SparkFun-Jumpers:SMT-JUMPER_2_NO_NO-SILK
- moved J3 335.7 mm to (326.3, 12.1), turned to 180 degrees
- moved J2 321.3 mm to (319.3, 28.4), turned to 90 degrees
- moved R3 315.1 mm to (316.1, 29.8), turned to 0 degrees
- moved R4 314.9 mm to (316.1, 27.3), turned to 0 degrees
- moved R15 298.2 mm to (302.3, 9.56), turned to 270 degrees
- moved R14 297.5 mm to (302.3, 15.3), turned to 270 degrees
- moved R12 293.5 mm to (299.8, 7.66), turned to 180 degrees
- moved C3 293.2 mm to (299.8, 9.56), turned to 0 degrees
- moved R5 292.9 mm to (299.8, 11.5), turned to 180 degrees
- moved R7 292.6 mm to (299.8, 13.4), turned to 0 degrees
- moved C2 292.4 mm to (299.8, 15.3), turned to 180 degrees
- moved R6 292.2 mm to (299.8, 17.2), turned to 180 degrees
- moved U$3 24.0 mm to (37.2, 27.5)
- moved C8 1.30 mm to (13.3, 9.55), turned to 90 degrees
Connections:
- removed net N$127: D251.2, D252.4, JP251.2, JP252.1
- removed net N$135: D11.2, D12.4, JP11.2, JP12.1
- net DIO133: now also D251.2, JP251.2; no longer D252.2, JP252.2
- net GND: no longer D12.3, D252.3
- net N$8: now also D11.2, JP11.2; no longer D12.2, JP12.2
- net V_USB: no longer D12.1, D252.1
Routing:
- net D-: track 32.1 -> 320.6 mm
- net D+: track 32.9 -> 320.0 mm
- net RING1: track 43.6 -> 268.0 mm
- net TIP: track 46.4 -> 268.8 mm, vias 2 -> 0
- net 3.3V: track 150.2 -> 363.4 mm, vias 10 -> 9
- net V_USB: track 564.0 -> 455.4 mm, vias 267 -> 265
- net N$127: track 23.6 -> 0.00 mm
- net DIO133: track 11.8 -> 33.6 mm
- net DIO0: track 233.1 -> 215.3 mm, vias 3 -> 2
- net N$6: track 5.87 -> 19.9 mm
- net N$135: track 13.1 -> 0.00 mm
- net N$8: track 20.6 -> 32.5 mm
- net N$7: track 13.6 -> 23.6 mm
- net MIC: track 32.4 -> 29.2 mm
Other:
- outline, holes or cut-outs redrawn

Commit message: strange gerber issue, counting a trace on dimension layer
Routing:
- net DIO0: track 215.3 -> 214.1 mm
- net N$8: track 32.5 -> 31.8 mm

Commit message: most of barebones backedn finished
Parts:
- moved J2 0.54 mm to (319.0, 28.0)
- moved J3 0.32 mm to (326.0, 12.0)
Routing:
- net D+: track 320.0 -> 315.8 mm
- net D-: track 320.6 -> 320.1 mm
Other:
- outline, holes or cut-outs redrawn

Commit message: updating 15TB outer dimensions, still need to re-place holes
Parts:
- added D1, D12, D21, D211, D252, D263, D264: WS2812B, SparkFun-LED:WS2812B
- added JP1, JP12, JP21, JP211, JP252, JP263, JP264: JUMPER-SMT_2_NO_NO-SILK, SparkFun-Jumpers:SMT-JUMPER_2_NO_NO-SILK
- R13: value 1k -> 2.2k; device SparkFun-Resistors:AXIAL-0.3 -> SparkFun-Resistors:0603
- moved U5 58.8 mm to (12.7, 17.5), turned to 270 degrees
- moved R10 53.7 mm to (19.5, 13.3), turned to 270 degrees
- moved C4 53.3 mm to (17.6, 17.4), turned to 270 degrees
- moved C6 51.9 mm to (21.4, 13.3), turned to 90 degrees
- moved R9 50.1 mm to (23.3, 13.3), turned to 90 degrees
- moved R13 49.9 mm to (27.0, 11.0), turned to 0 degrees
- moved U$2 46.9 mm to (27.0, 13.3), turned to 270 degrees
- moved C5 44.8 mm to (24.7, 16.6), turned to 180 degrees
- moved C9 44.5 mm to (30.1, 13.3), turned to 270 degrees
- moved R11 42.8 mm to (24.7, 18.5), turned to 180 degrees
- moved H2 41.2 mm to (181.6, 7.50)
- moved H1 41.2 mm to (134.9, 190.2)
- moved R7 29.5 mm to (316.0, 38.0), turned to 270 degrees
- moved C2 29.1 mm to (318.0, 38.0), turned to 90 degrees
- moved R6 29.0 mm to (320.0, 38.0), turned to 90 degrees
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Connections:
- removed net DIO120: D231.2, D232.4, JP231.2, JP232.1
- new net DIO121: D21.4, D231.2, JP21.1, JP231.2
- new net DIO127: D211.2, D263.4, JP211.2, JP263.1
- new net N$127: D251.2, D252.4, JP251.2, JP252.1
- new net N$135: D11.2, D12.4, JP11.2, JP12.1
- new net N$138: D263.2, D264.4, JP263.2, JP264.1
- new net N$140: D232.4, D264.2, JP232.1, JP264.2
- new net N$2: D21.2, D211.4, JP21.2, JP211.1
- new net N$21: D1.2, D212.4, JP1.2, JP212.1
- net DIO109: now also D1.4, JP1.1; no longer D212.4, JP212.1
- net DIO133: now also D252.2, JP252.2; no longer D251.2, JP251.2
- net GND: now also D1.3, D12.3, D21.3, D211.3, D252.3, D263.3, D264.3
- net N$11: now also R13.1; no longer R13.P$1
- net N$8: now also D12.2, JP12.2; no longer D11.2, JP11.2
- net N$9: now also R13.2; no longer R13.P$2
- net V_USB: now also D1.1, D12.1, D21.1, D211.1, D252.1, D263.1, D264.1
Routing:
- net DIO121: track 0.00 -> 321.3 mm, vias 0 -> 2
- net DIO120: track 243.9 -> 0.00 mm, vias 2 -> 0
- net 3.3V: track 363.4 -> 407.7 mm, vias 9 -> 8
- net DIO127: track 0.00 -> 31.8 mm, vias 0 -> 2
- net RING1: track 268.0 -> 293.8 mm
- net TIP: track 268.8 -> 290.9 mm
- net N$2: track 0.00 -> 18.0 mm, vias 0 -> 2
- net D+: track 315.8 -> 333.5 mm
- net N$135: track 0.00 -> 16.8 mm
- net N$127: track 0.00 -> 16.8 mm
- net N$21: track 0.00 -> 16.8 mm
- net N$140: track 0.00 -> 16.8 mm
- net N$138: track 0.00 -> 16.8 mm
- net DIO133: track 33.6 -> 16.8 mm
- net DIO109: track 304.1 -> 320.2 mm
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Other:
- outline, holes or cut-outs redrawn
- board text added: "13R"
- board text removed: "13NR"
- board text removed: "D"

Commit message: updating 13NR
Parts:
- removed D11, D12, D252, D253: WS2812B, SparkFun-LED:WS2812B
- removed JP11, JP12, JP252, JP253: JUMPER-SMT_2_NO_NO-SILK, SparkFun-Jumpers:SMT-JUMPER_2_NO_NO-SILK
- moved H2 41.2 mm to (140.4, 7.50)
- moved H1 41.2 mm to (176.1, 190.2)
- moved C2 6.00 mm to (318.0, 32.0)
- moved C3 6.00 mm to (313.5, 15.0)
- moved J2 6.00 mm to (319.0, 41.4)
- moved J3 6.00 mm to (324.5, 24.1)
- moved R12 6.00 mm to (313.5, 16.5)
- moved R14 6.00 mm to (318.0, 29.5)
- moved R15 6.00 mm to (313.5, 18.5)
- moved R3 6.00 mm to (315.8, 42.8)
- moved R4 6.00 mm to (315.8, 40.3)
- moved R5 6.00 mm to (311.8, 11.5)
- moved R6 6.00 mm to (320.0, 32.0)
- moved R7 6.00 mm to (316.0, 32.0)
Connections:
- removed net DIO133: D252.2, D253.4, JP252.2, JP253.1
- removed net DIO5: D10.2, D11.4, JP10.2, JP11.1
- removed net N$127: D251.2, D252.4, JP251.2, JP252.1
- removed net N$8: D12.2, D13.4, JP12.2, JP13.1
- net DIO134: now also D251.2, JP251.2; no longer D253.2, JP253.2
- net GND: no longer D11.3, D12.3, D252.3, D253.3
- net N$135: now also D10.2, D13.4, JP10.2, JP13.1; no longer D11.2, D12.4, JP11.2, JP12.1
- net V_USB: no longer D11.1, D12.1, D252.1, D253.1
Routing:
- net DIO134: track 16.8 -> 48.4 mm
- net N$135: track 16.8 -> 46.8 mm
- net DIO133: track 16.8 -> 0.00 mm
- net N$8: track 16.8 -> 0.00 mm
- net N$127: track 16.8 -> 0.00 mm
- net DIO5: track 16.8 -> 0.00 mm
- net RING1: track 293.8 -> 289.6 mm
- net V_USB: track 447.0 -> 443.3 mm, vias 273 -> 269
- net 3.3V: track 407.7 -> 410.2 mm
- net D-: track 335.4 -> 332.9 mm
- net D+: track 333.5 -> 331.0 mm
- net TIP: track 290.9 -> 292.6 mm
Other:
- outline, holes or cut-outs redrawn
- board text added: "13NR"
- board text removed: "13R"

Commit message: final touches, polishing, jumpers, CAM on all boards
Parts:
- added D11: WS2812B, SparkFun-LED:WS2812B
- added JP11, JP12, JP252, JP253, JP265, JP266, JP267, JP268, JP269, JP270, JP271, JP272, JP273: JUMPER-SMT_2_NO_NO-SILK, SparkFun-Jumpers:SMT-JUMPER_2_NO_NO-SILK
- moved R5 2.62 mm to (313.5, 13.5), turned to 180 degrees
Connections:
- removed net DIO10: D20.2, D22.4, JP20.2, JP22.1
- removed net DIO109: D1.4, D210.2, JP1.1, JP210.2
- removed net DIO121: D21.4, D231.2, JP21.1, JP231.2
- removed net DIO33: D63.2, D64.4, JP63.2, JP64.1
- removed net DIO54: D105.2, D106.4, JP105.2, JP106.1
- removed net DIO76: D147.2, D148.4, JP147.2, JP148.1
- removed net DIO99: D189.2, D190.4, JP189.2, JP190.1
- removed net N$32: D42.2, D43.4, JP42.2, JP43.1
- removed net N$54: D84.2, D85.4, JP84.2, JP85.1
- removed net N$68: D126.2, D127.4, JP126.2, JP127.1
- removed net N$89: D168.2, D169.4, JP168.2, JP169.1
- new net JUMPER0: D20.2, D22.4, JP11.2, JP20.2, JP22.1, JP252.1
- new net JUMPER1: D42.2, D43.4, JP252.2, JP253.1, JP42.2, JP43.1
- new net JUMPER10: D21.4, D231.2, JP21.1, JP231.2, JP272.2, JP273.1
- new net JUMPER11: D11.4, D247.2, JP12.1, JP247.2, JP273.2
- new net JUMPER2: D63.2, D64.4, JP253.2, JP265.1, JP63.2, JP64.1
- new net JUMPER3: D84.2, D85.4, JP265.2, JP266.1, JP84.2, JP85.1
- new net JUMPER4: D105.2, D106.4, JP105.2, JP106.1, JP266.2, JP267.1
- new net JUMPER5: D126.2, D127.4, JP126.2, JP127.1, JP267.2, JP268.1
- new net JUMPER6: D147.2, D148.4, JP147.2, JP148.1, JP268.2, JP269.1
- new net JUMPER7: D168.2, D169.4, JP168.2, JP169.1, JP269.2, JP270.1
- new net JUMPER8: D189.2, D190.4, JP189.2, JP190.1, JP270.2, JP271.1
- new net JUMPER9: D1.4, D210.2, JP1.1, JP210.2, JP271.2, JP272.1
- net DIO0: now also JP11.1
- net GND: now also D11.3
- net N$125: now also D11.2, JP12.2; no longer D247.2, JP247.2
- net V_USB: now also D11.1
Routing:
- net JUMPER10: track 0.00 -> 337.4 mm, vias 0 -> 4
- net JUMPER9: track 0.00 -> 332.2 mm, vias 0 -> 2
- net JUMPER6: track 0.00 -> 331.0 mm, vias 0 -> 2
- net JUMPER7: track 0.00 -> 331.0 mm, vias 0 -> 2
- net JUMPER8: track 0.00 -> 331.0 mm, vias 0 -> 2
- net JUMPER4: track 0.00 -> 331.0 mm, vias 0 -> 2
- net JUMPER5: track 0.00 -> 331.0 mm, vias 0 -> 2
- net JUMPER2: track 0.00 -> 330.8 mm, vias 0 -> 2
- net JUMPER1: track 0.00 -> 330.8 mm, vias 0 -> 2
- net JUMPER3: track 0.00 -> 330.7 mm, vias 0 -> 2
- net JUMPER0: track 0.00 -> 324.4 mm, vias 0 -> 2
- net DIO121: track 321.4 -> 0.00 mm, vias 2 -> 0
- net DIO109: track 320.2 -> 0.00 mm, vias 2 -> 0
- net N$89: track 319.1 -> 0.00 mm, vias 2 -> 0
- net N$68: track 319.1 -> 0.00 mm, vias 2 -> 0
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
Commit message: pushing final board changes
Parts:
- removed D21, D211, D263: WS2812B, SparkFun-LED:WS2812B
- removed JP21, JP211, JP263: JUMPER-SMT_2_NO_NO-SILK, SparkFun-Jumpers:SMT-JUMPER_2_NO_NO-SILK
- added U$1: (no value), unnamed#png (2):UNNAMED#PNG
- moved J2 18.5 mm to (320.0, 23.0)
- moved R3 18.5 mm to (316.4, 24.4)
- moved R4 18.4 mm to (316.3, 21.9)
- moved C3 17.1 mm to (315.5, 32.0), turned to 180 degrees
- moved R12 17.1 mm to (315.5, 33.5), turned to 0 degrees
- moved R5 17.1 mm to (315.5, 30.5), turned to 0 degrees
- moved J3 17.0 mm to (326.5, 41.0)
- moved R15 16.6 mm to (315.5, 35.0)
- moved R7 7.07 mm to (323.0, 33.0)
- moved R14 6.71 mm to (321.0, 35.5), turned to 0 degrees
- moved C7 5.02 mm to (5.97, 18.1), turned to 0 degrees
- moved U3 4.12 mm to (6.92, 22.0)
- moved C4 4.00 mm to (17.6, 21.4)
- moved C5 4.00 mm to (24.7, 20.6)
- moved FD4 4.00 mm to (10.5, 13.0)
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Connections:
- removed net DIO127: D211.2, D263.4, JP211.2, JP263.1
- removed net N$138: D263.2, D264.4, JP263.2, JP264.1
- removed net N$2: D21.2, D211.4, JP21.2, JP211.1
- net GND: no longer D21.3, D211.3, D263.3
- net JUMPER10: now also D264.4, JP264.1; no longer D21.4, JP21.1
- net V_USB: no longer D21.1, D211.1, D263.1
Routing:
- net DIO127: track 31.8 -> 0.00 mm, vias 2 -> 0
- net N$2: track 18.0 -> 0.00 mm, vias 2 -> 0
- net N$138: track 16.8 -> 0.00 mm
- net N$7: track 11.3 -> 5.22 mm
- net V_USB: track 445.8 -> 439.9 mm, vias 270 -> 268
- net D-: track 332.9 -> 327.4 mm, vias 0 -> 2
- net D+: track 331.0 -> 326.0 mm, vias 2 -> 4
- net RING1: track 289.6 -> 294.4 mm, vias 0 -> 2
- net TIP: track 290.6 -> 286.2 mm
- net JUMPER10: track 337.4 -> 333.4 mm, vias 4 -> 3
- net DIO0: track 223.0 -> 221.4 mm
- net EN: track 2.66 -> 1.72 mm
- net GND: track 78.2 -> 77.6 mm
- net 3.3V: vias 8 -> 9
Other:
- outline, holes or cut-outs redrawn
