File: Hardware/13NR.sch (EAGLE design)
At the start: 578 parts, among them J2 USB Female Type C Connector, J3 AUDIO_JACK_TRRSSMD_RA, Q2 MBT3904DW1T1, U2 ESP-WROOM-32NARROW, U3 AP2112K-3.3V, U4 CP2102N, U5 ADMP401

Commit message: updating 13NR
Parts:
- removed D11, D12, D252, D253: WS2812B, SparkFun-LED:WS2812B
- removed JP11, JP12, JP252, JP253: JUMPER-SMT_2_NO_NO-SILK, SparkFun-Jumpers:JUMPER-SMT_2_NO_NO-SILK
Connections:
- removed net DIO133: D252.DO, D253.DI, JP252.2, JP253.1
- removed net DIO5: D10.DO, D11.DI, JP10.2, JP11.1
- removed net N$127: D251.DO, D252.DI, JP251.2, JP252.1
- removed net N$8: D12.DO, D13.DI, JP12.2, JP13.1
- net DIO134: now also D251.DO, JP251.2; no longer D253.DO, JP253.2
- net GND: no longer D11.VSS, D12.VSS, D252.VSS, D253.VSS
- net N$135: now also D10.DO, D13.DI, JP10.2, JP13.1; no longer D11.DO, D12.DI, JP11.2, JP12.1
- net V_USB: no longer D11.VDD, D12.VDD, D252.VDD, D253.VDD

Commit message: final touches, polishing, jumpers, CAM on all boards
Parts:
- added D11: WS2812B, SparkFun-LED:WS2812B
- added JP11, JP12, JP252, JP253, JP265, JP266, JP267, JP268, JP269, JP270, JP271, JP272, JP273: JUMPER-SMT_2_NO_NO-SILK, SparkFun-Jumpers:JUMPER-SMT_2_NO_NO-SILK
Connections:
- removed net DIO10: D20.DO, D22.DI, JP20.2, JP22.1
- removed net DIO109: D1.DI, D210.DO, JP1.1, JP210.2
- removed net DIO121: D21.DI, D231.DO, JP21.1, JP231.2
- removed net DIO33: D63.DO, D64.DI, JP63.2, JP64.1
- removed net DIO54: D105.DO, D106.DI, JP105.2, JP106.1
- removed net DIO76: D147.DO, D148.DI, JP147.2, JP148.1
- removed net DIO99: D189.DO, D190.DI, JP189.2, JP190.1
- removed net N$32: D42.DO, D43.DI, JP42.2, JP43.1
- removed net N$54: D84.DO, D85.DI, JP84.2, JP85.1
- removed net N$68: D126.DO, D127.DI, JP126.2, JP127.1
- removed net N$89: D168.DO, D169.DI, JP168.2, JP169.1
- new net JUMPER0: D20.DO, D22.DI, JP11.2, JP20.2, JP22.1, JP252.1
- new net JUMPER1: D42.DO, D43.DI, JP252.2, JP253.1, JP42.2, JP43.1
- new net JUMPER10: D21.DI, D231.DO, JP21.1, JP231.2, JP272.2, JP273.1
- new net JUMPER11: D11.DI, D247.DO, JP12.1, JP247.2, JP273.2
- new net JUMPER2: D63.DO, D64.DI, JP253.2, JP265.1, JP63.2, JP64.1
- new net JUMPER3: D84.DO, D85.DI, JP265.2, JP266.1, JP84.2, JP85.1
- new net JUMPER4: D105.DO, D106.DI, JP105.2, JP106.1, JP266.2, JP267.1
- new net JUMPER5: D126.DO, D127.DI, JP126.2, JP127.1, JP267.2, JP268.1
- new net JUMPER6: D147.DO, D148.DI, JP147.2, JP148.1, JP268.2, JP269.1
- new net JUMPER7: D168.DO, D169.DI, JP168.2, JP169.1, JP269.2, JP270.1
- new net JUMPER8: D189.DO, D190.DI, JP189.2, JP190.1, JP270.2, JP271.1
- new net JUMPER9: D1.DI, D210.DO, JP1.1, JP210.2, JP271.2, JP272.1
- net DIO0: now also JP11.1
- net GND: now also D11.VSS
- net N$125: now also D11.DO, JP12.2; no longer D247.DO, JP247.2
- net V_USB: now also D11.VDD
Other:
- moved on the sheet: D248, D249, D250, D251, JP248, JP249, JP250, JP251

Commit message: pushing final board changes
Parts:
- removed D21, D211, D263: WS2812B, SparkFun-LED:WS2812B
- removed JP21, JP211, JP263: JUMPER-SMT_2_NO_NO-SILK, SparkFun-Jumpers:JUMPER-SMT_2_NO_NO-SILK
Connections:
- removed net DIO127: D211.DO, D263.DI, JP211.2, JP263.1
- removed net N$138: D263.DO, D264.DI, JP263.2, JP264.1
- removed net N$2: D21.DO, D211.DI, JP21.2, JP211.1
- net GND: no longer D21.VSS, D211.VSS, D263.VSS
- net JUMPER10: now also D264.DI, JP264.1; no longer D21.DI, JP21.1
- net V_USB: no longer D21.VDD, D211.VDD, D263.VDD
Changed lines of the file:
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@@
 <?xml version="1.0" encoding="utf-8"?>
 <!DOCTYPE eagle SYSTEM "eagle.dtd">
-<eagle version="9.5.2">
+<eagle version="9.6.0">
 <drawing>
 <settings>
@@
 <part name="GND4" library="SparkFun-PowerSymbols" deviceset="GND" device=""/>
 <part name="SUPPLY1" library="SparkFun-PowerSymbols" deviceset="V_USB" device=""/>
-<part name="SUPPLY30" library="SparkFun-PowerSymbols" deviceset="V_USB" device=""/>
-<part name="D21" library="SparkFun-LED" deviceset="WS2812B" device="" value="WS2812B"/>
-<part name="JP21" library="SparkFun-Jumpers" deviceset="JUMPER-SMT_2_NO" device="_NO-SILK" value="JUMPER-SMT_2_NO_NO-SILK"/>
-<part name="D211" library="SparkFun-LED" deviceset="WS2812B" device="" value="WS2812B"/>
-<part name="SUPPLY107" library="SparkFun-PowerSymbols" deviceset="V_USB" device=""/>
-<part name="GND8" library="SparkFun-PowerSymbols" deviceset="GND" device=""/>
-<part name="D263" library="SparkFun-LED" deviceset="WS2812B" device="" value="WS2812B"/>
-<part name="GND37" library="SparkFun-PowerSymbols" deviceset="GND" device=""/>
-<part name="SUPPLY221" library="SparkFun-PowerSymbols" deviceset="V_USB" device=""/>
-<part name="GND227" library="SparkFun-PowerSymbols" deviceset="GND" device=""/>
-<part name="JP211" library="SparkFun-Jumpers" deviceset="JUMPER-SMT_2_NO" device="_NO-SILK" value="JUMPER-SMT_2_NO_NO-SILK"/>
-<part name="JP263" library="SparkFun-Jumpers" deviceset="JUMPER-SMT_2_NO" device="_NO-SILK" value="JUMPER-SMT_2_NO_NO-SILK"/>
 <part name="D264" library="SparkFun-LED" deviceset="WS2812B" device="" value="WS2812B"/>
 <part name="SUPPLY273" library="SparkFun-PowerSymbols" deviceset="V_USB" device=""/>
@@
 <attribute name="VALUE" x="60.96" y="246.634" size="1.778" layer="96" align="bottom-center"/>
 </instance>
-<instance part="SUPPLY30" gate="G$1" x="-116.84" y="193.04" smashed="yes">
-<attribute name="VALUE" x="-116.84" y="195.834" size="1.778" layer="96" align="bottom-center"/>
-</instance>
-<instance part="D21" gate="G$1" x="-99.06" y="185.42" smashed="yes">
-<attribute name="NAME" x="-101.6" y="193.802" size="1.778" layer="95" font="vector" align="bottom-center"/>
-</instance>
-<instance part="JP21" gate="G$1" x="-101.6" y="175.26" smashed="yes">
-<attribute name="NAME" x="-104.14" y="177.8" size="1.778" layer="95" font="vector"/>
-</instance>
-<instance part="D211" gate="G$1" x="-63.5" y="185.42" smashed="yes">
-<attribute name="NAME" x="-66.04" y="193.802" size="1.778" layer="95" font="vector" align="bottom-center"/>
-</instance>
-<instance part="SUPPLY107" gate="G$1" x="-81.28" y="193.04" smashed="yes">
-<attribute name="VALUE" x="-81.28" y="195.834" size="1.778" layer="96" align="bottom-center"/>
-</instance>
-<instance part="GND8" gate="1" x="-83.82" y="177.8" smashed="yes">
-<attribute name="VALUE" x="-83.82" y="177.546" size="1.778" layer="96" align="top-center"/>
-</instance>
-<instance part="D263" gate="G$1" x="-27.94" y="185.42" smashed="yes">
-<attribute name="NAME" x="-30.48" y="193.802" size="1.778" layer="95" font="vector" align="bottom-center"/>
-</instance>
-<instance part="GND37" gate="1" x="-12.7" y="177.8" smashed="yes">
-<attribute name="VALUE" x="-12.7" y="177.546" size="1.778" layer="96" align="top-center"/>
-</instance>
-<instance part="SUPPLY221" gate="G$1" x="-45.72" y="193.04" smashed="yes">
-<attribute name="VALUE" x="-45.72" y="195.834" size="1.778" layer="96" align="bottom-center"/>
-</instance>
-<instance part="GND227" gate="1" x="-48.26" y="177.8" smashed="yes">
-<attribute name="VALUE" x="-48.26" y="177.546" size="1.778" layer="96" align="top-center"/>
-</instance>
-<instance part="JP211" gate="G$1" x="-66.04" y="175.26" smashed="yes">
-<attribute name="NAME" x="-68.58" y="177.8" size="1.778" layer="95" font="vector"/>
-</instance>
-<instance part="JP263" gate="G$1" x="-30.48" y="175.26" smashed="yes">
-<attribute name="NAME" x="-33.02" y="177.8" size="1.778" layer="95" font="vector"/>
-</instance>
 <instance part="D264" gate="G$1" x="7.62" y="185.42" smashed="yes">
 <attribute name="NAME" x="5.08" y="193.802" size="1.778" layer="95" font="vector" align="bottom-center"/>
@@
 </segment>
 <segment>
-<wire x1="-114.3" y1="190.5" x2="-116.84" y2="190.5" width="0.1524" layer="91"/>
-<wire x1="-116.84" y1="190.5" x2="-116.84" y2="193.04" width="0.1524" layer="91"/>
-<pinref part="SUPPLY30" gate="G$1" pin="V_USB"/>
-<pinref part="D21" gate="G$1" pin="VDD"/>
-</segment>
-<segment>
-<pinref part="D211" gate="G$1" pin="VDD"/>
-<wire x1="-78.74" y1="190.5" x2="-81.28" y2="190.5" width="0.1524" layer="91"/>
-<wire x1="-81.28" y1="190.5" x2="-81.28" y2="193.04" width="0.1524" layer="91"/>
-<pinref part="SUPPLY107" gate="G$1" pin="V_USB"/>
-</segment>
-<segment>
-<pinref part="D263" gate="G$1" pin="VDD"/>
-<wire x1="-43.18" y1="190.5" x2="-45.72" y2="190.5" width="0.1524" layer="91"/>
-<wire x1="-45.72" y1="190.5" x2="-45.72" y2="193.04" width="0.1524" layer="91"/>
-<pinref part="SUPPLY221" gate="G$1" pin="V_USB"/>
-</segment>
-<segment>
 <pinref part="D264" gate="G$1" pin="VDD"/>
 <wire x1="-7.62" y1="190.5" x2="-10.16" y2="190.5" width="0.1524" layer="91"/>
@@
 </segment>
 <segment>
-<pinref part="D21" gate="G$1" pin="VSS"/>
-<wire x1="-86.36" y1="190.5" x2="-83.82" y2="190.5" width="0.1524" layer="91"/>
-<wire x1="-83.82" y1="190.5" x2="-83.82" y2="180.34" width="0.1524" layer="91"/>
-<pinref part="GND8" gate="1" pin="GND"/>
-</segment>
-<segment>
-<pinref part="D263" gate="G$1" pin="VSS"/>
-<wire x1="-15.24" y1="190.5" x2="-12.7" y2="190.5" width="0.1524" layer="91"/>
-<wire x1="-12.7" y1="190.5" x2="-12.7" y2="180.34" width="0.1524" layer="91"/>
-<pinref part="GND37" gate="1" pin="GND"/>
-</segment>
-<segment>
-<pinref part="D211" gate="G$1" pin="VSS"/>
-<wire x1="-50.8" y1="190.5" x2="-48.26" y2="190.5" width="0.1524" layer="91"/>
-<wire x1="-48.26" y1="190.5" x2="-48.26" y2="180.34" width="0.1524" layer="91"/>
-<pinref part="GND227" gate="1" pin="GND"/>
-</segment>
-<segment>
 <pinref part="D264" gate="G$1" pin="VSS"/>
 <wire x1="20.32" y1="190.5" x2="22.86" y2="190.5" width="0.1524" layer="91"/>
@@
 <net name="JUMPER10" class="0">
 <segment>
-<pinref part="D21" gate="G$1" pin="DI"/>
-<wire x1="-114.3" y1="182.88" x2="-121.92" y2="182.88" width="0.1524" layer="91"/>
-<wire x1="-121.92" y1="182.88" x2="-121.92" y2="177.8" width="0.1524" layer="91"/>
-<pinref part="JP21" gate="G$1" pin="1"/>
-<wire x1="-121.92" y1="177.8" x2="-121.92" y2="175.26" width="0.1524" layer="91"/>
-<wire x1="-121.92" y1="175.26" x2="-106.68" y2="175.26" width="0.1524" layer="91"/>
-<wire x1="-121.92" y1="198.12" x2="-121.92" y2="182.88" width="0.1524" layer="91"/>
-<junction x="-121.92" y="182.88"/>
 <pinref part="D231" gate="G$1" pin="DO"/>
 <wire x1="411.48" y1="208.28" x2="416.56" y2="208.28" width="0.1524" layer="91"/>
@@
 <wire x1="416.56" y1="208.28" x2="416.56" y2="200.66" width="0.1524" layer="91"/>
 <junction x="416.56" y="208.28"/>
-<wire x1="-121.92" y1="198.12" x2="419.1" y2="198.12" width="0.1524" layer="91"/>
+<wire x1="-15.24" y1="198.12" x2="419.1" y2="198.12" width="0.1524" layer="91"/>
 <wire x1="419.1" y1="198.12" x2="419.1" y2="208.28" width="0.1524" layer="91"/>
-<wire x1="-121.92" y1="177.8" x2="-119.38" y2="177.8" width="0.1524" layer="91"/>
-<junction x="-121.92" y="177.8"/>
-<label x="-119.38" y="177.8" size="1.27" layer="95" xref="yes"/>
+<pinref part="D264" gate="G$1" pin="DI"/>
+<wire x1="-15.24" y1="182.88" x2="-7.62" y2="182.88" width="0.1524" layer="91"/>
+<pinref part="JP264" gate="G$1" pin="1"/>
+<wire x1="-15.24" y1="175.26" x2="0" y2="175.26" width="0.1524" layer="91"/>
+<wire x1="-15.24" y1="182.88" x2="-15.24" y2="175.26" width="0.1524" layer="91"/>
+<wire x1="-15.24" y1="198.12" x2="-15.24" y2="182.88" width="0.1524" layer="91"/>
+<junction x="-15.24" y="182.88"/>
 </segment>
 <segment>
@@
 </segment>
 </net>
-<net name="N$2" class="0">
-<segment>
-<pinref part="D21" gate="G$1" pin="DO"/>
-<pinref part="D211" gate="G$1" pin="DI"/>
-<wire x1="-86.36" y1="182.88" x2="-81.28" y2="182.88" width="0.1524" layer="91"/>
-<pinref part="JP21" gate="G$1" pin="2"/>
-<wire x1="-81.28" y1="182.88" x2="-78.74" y2="182.88" width="0.1524" layer="91"/>
-<wire x1="-96.52" y1="175.26" x2="-81.28" y2="175.26" width="0.1524" layer="91"/>
-<wire x1="-81.28" y1="175.26" x2="-81.28" y2="182.88" width="0.1524" layer="91"/>
-<junction x="-81.28" y="182.88"/>
-<pinref part="JP211" gate="G$1" pin="1"/>
-<wire x1="-81.28" y1="175.26" x2="-71.12" y2="175.26" width="0.1524" layer="91"/>
-<junction x="-81.28" y="175.26"/>
-</segment>
-</net>
-<net name="DIO127" class="0">
-<segment>
-<wire x1="-45.72" y1="175.26" x2="-35.56" y2="175.26" width="0.1524" layer="91"/>
-<pinref part="D211" gate="G$1" pin="DO"/>
-<pinref part="D263" gate="G$1" pin="DI"/>
-<wire x1="-50.8" y1="182.88" x2="-45.72" y2="182.88" width="0.1524" layer="91"/>
-<wire x1="-45.72" y1="182.88" x2="-43.18" y2="182.88" width="0.1524" layer="91"/>
-<wire x1="-45.72" y1="175.26" x2="-45.72" y2="182.88" width="0.1524" layer="91"/>
-<junction x="-45.72" y="182.88"/>
-<pinref part="JP263" gate="G$1" pin="1"/>
-<pinref part="JP211" gate="G$1" pin="2"/>
-<wire x1="-60.96" y1="175.26" x2="-45.72" y2="175.26" width="0.1524" layer="91"/>
-<junction x="-45.72" y="175.26"/>
-</segment>
-</net>
-<net name="N$138" class="0">
-<segment>
-<pinref part="D264" gate="G$1" pin="DI"/>
-<pinref part="D263" gate="G$1" pin="DO"/>
-<wire x1="-15.24" y1="182.88" x2="-10.16" y2="182.88" width="0.1524" layer="91"/>
-<wire x1="-10.16" y1="182.88" x2="-7.62" y2="182.88" width="0.1524" layer="91"/>
-<wire x1="-25.4" y1="175.26" x2="-10.16" y2="175.26" width="0.1524" layer="91"/>
-<pinref part="JP263" gate="G$1" pin="2"/>
-<pinref part="JP264" gate="G$1" pin="1"/>
-<wire x1="-10.16" y1="175.26" x2="0" y2="175.26" width="0.1524" layer="91"/>
-<wire x1="-10.16" y1="182.88" x2="-10.16" y2="175.26" width="0.1524" layer="91"/>
-<junction x="-10.16" y="182.88"/>
-<junction x="-10.16" y="175.26"/>
-</segment>
-</net>

Commit message: updating files
Parts:
- removed FD4: FIDUCIALUFIDUCIAL, SparkFun-Aesthetics:FIDUCIALUFIDUCIAL
Changed lines of the file:
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@@
 <part name="FD1" library="SparkFun-Aesthetics" deviceset="FIDUCIAL" device="UFIDUCIAL"/>
 <part name="FD2" library="SparkFun-Aesthetics" deviceset="FIDUCIAL" device="UFIDUCIAL"/>
-<part name="FD4" library="SparkFun-Aesthetics" deviceset="FIDUCIAL" device="UFIDUCIAL"/>
 <part name="S2" library="SparkFun-Switches" deviceset="MOMENTARY-SWITCH-SPST-2" device="-SMD-4.6X2.8MM" value="0"/>
 <part name="GND10" library="SparkFun-Aesthetics" deviceset="GND" device=""/>
@@
 <instance part="FD1" gate="G$1" x="429.26" y="33.02" smashed="yes"/>
 <instance part="FD2" gate="G$1" x="426.72" y="33.02" smashed="yes"/>
-<instance part="FD4" gate="G$1" x="429.26" y="30.48" smashed="yes"/>
 <instance part="S2" gate="G$1" x="294.64" y="177.8" smashed="yes">
 <attribute name="NAME" x="294.64" y="182.626" size="1.778" layer="95" font="vector" align="bottom-center"/>
