File: Hardware/13R.brd (EAGLE design)
At the start: 326.5 x 197.8 mm, 569 parts, among them J2 USB Female Type C Connector, J3 AUDIO_JACK_TRRSSMD_RA, Q2 MBT3904DW1T1, U2 ESP-WROOM-32NARROW, U3 AP2112K-3.3V, U4 CP2102N, U5 ADMP401

Commit message: final airwires on 13 inch retina, need to copy and move holes
Parts:
- added D1, D21, D211, D263, D264: WS2812B, SparkFun-LED:WS2812B
- added JP1, JP21, JP211, JP263, JP264: JUMPER-SMT_2_NO_NO-SILK, SparkFun-Jumpers:SMT-JUMPER_2_NO_NO-SILK
- R13: value 1k -> 2.2k; device SparkFun-Resistors:AXIAL-0.3 -> SparkFun-Resistors:0603
- moved J3 333.3 mm to (324.5, 30.1), turned to 180 degrees
- moved J2 322.3 mm to (319.0, 47.4), turned to 90 degrees
- moved R3 316.2 mm to (315.8, 48.8), turned to 0 degrees
- moved R4 315.7 mm to (315.8, 46.3), turned to 0 degrees
- moved R14 312.8 mm to (318.0, 35.5), turned to 180 degrees
- moved R6 312.4 mm to (320.0, 38.0), turned to 90 degrees
- moved C2 310.4 mm to (318.0, 38.0), turned to 90 degrees
- moved R15 308.5 mm to (313.5, 24.5), turned to 0 degrees
- moved R7 308.3 mm to (316.0, 38.0), turned to 270 degrees
- moved R12 306.1 mm to (313.5, 22.5), turned to 180 degrees
- moved C3 306.1 mm to (313.5, 21.0), turned to 0 degrees
- moved R5 304.5 mm to (311.8, 17.5)
- moved U5 59.6 mm to (12.7, 17.5), turned to 270 degrees
- moved C4 53.8 mm to (17.6, 17.4), turned to 270 degrees
- moved R10 53.8 mm to (19.5, 13.3), turned to 270 degrees
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Connections:
- removed net DIO120: D231.2, D232.4, JP231.2, JP232.1
- new net DIO121: D21.4, D231.2, JP21.1, JP231.2
- new net DIO127: D211.2, D263.4, JP211.2, JP263.1
- new net N$138: D263.2, D264.4, JP263.2, JP264.1
- new net N$140: D232.4, D264.2, JP232.1, JP264.2
- new net N$2: D21.2, D211.4, JP21.2, JP211.1
- new net N$21: D1.2, D212.4, JP1.2, JP212.1
- net DIO109: now also D1.4, JP1.1; no longer D212.4, JP212.1
- net GND: now also D1.3, D21.3, D211.3, D263.3, D264.3
- net N$11: now also R13.1; no longer R13.P$1
- net N$9: now also R13.2; no longer R13.P$2
- net V_USB: now also D1.1, D21.1, D211.1, D263.1, D264.1
Routing:
- net DIO121: track 0.00 -> 321.3 mm, vias 0 -> 2
- net D-: track 31.8 -> 335.4 mm
- net D+: track 31.5 -> 333.5 mm
- net RING1: track 45.2 -> 293.8 mm
- net DIO120: track 243.9 -> 0.00 mm, vias 2 -> 0
- net TIP: track 48.1 -> 290.9 mm, vias 2 -> 0
- net 3.3V: track 167.3 -> 407.7 mm, vias 10 -> 8
- net V_USB: track 553.2 -> 447.0 mm, vias 267 -> 273
- net DIO127: track 0.00 -> 31.8 mm, vias 0 -> 2
- net DIO0: track 234.7 -> 213.1 mm
- net N$2: track 0.00 -> 18.0 mm, vias 0 -> 2
- net N$21: track 0.00 -> 16.8 mm
- net N$140: track 0.00 -> 16.8 mm
- net N$138: track 0.00 -> 16.8 mm
- net DIO109: track 304.1 -> 320.2 mm
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Other:
- outline, holes or cut-outs redrawn
- board text removed: "D"

Commit message: updating 13NR
Parts:
- moved C2 12.5 mm to (307.0, 32.0)
- moved C3 12.5 mm to (302.5, 15.0)
- moved J2 12.5 mm to (308.0, 41.4)
- moved J3 12.5 mm to (313.5, 24.1)
- moved R12 12.5 mm to (302.5, 16.5)
- moved R14 12.5 mm to (307.0, 29.5)
- moved R15 12.5 mm to (302.5, 18.5)
- moved R3 12.5 mm to (304.8, 42.8)
- moved R4 12.5 mm to (304.8, 40.3)
- moved R5 12.5 mm to (300.8, 11.5)
- moved R6 12.5 mm to (309.0, 32.0)
- moved R7 12.5 mm to (305.0, 32.0)
- moved FD1 11.0 mm to (302.8, 195.0)
- moved H3 11.0 mm to (298.0, 7.50)
- moved H5 11.0 mm to (298.0, 190.2)
Routing:
- net V_USB: track 447.0 -> 572.3 mm
- net DIO33: track 318.9 -> 344.8 mm
- net N$125: track 244.1 -> 269.8 mm
- net DIO121: track 321.3 -> 346.9 mm
- net N$89: track 319.1 -> 344.8 mm
- net N$68: track 319.1 -> 344.8 mm
- net N$54: track 318.9 -> 344.5 mm
- net N$32: track 318.9 -> 344.6 mm
- net DIO99: track 319.1 -> 344.8 mm
- net DIO76: track 319.1 -> 344.8 mm
- net DIO54: track 319.1 -> 344.8 mm
- net DIO109: track 320.2 -> 345.9 mm
- net RING1: track 293.8 -> 278.6 mm
- net D-: track 335.4 -> 321.9 mm
- net D+: track 333.5 -> 320.0 mm
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Other:
- board size 326.5 x 197.8 mm -> 315.5 x 197.8 mm

Commit message: getting 4 boards polished
Other:
- board size 315.5 x 197.8 mm -> 315.5 x 197.1 mm
Changed lines of the file:
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@@
 <setting verticaltext="up"/>
 </settings>
-<grid distance="11" unitdist="mm" unit="mm" style="lines" multiple="1" display="yes" altdistance="0.05" altunitdist="mm" altunit="mm"/>
+<grid distance="2.5" unitdist="mm" unit="mm" style="lines" multiple="1" display="yes" altdistance="0.05" altunitdist="mm" altunit="mm"/>
 <layers>
 <layer number="1" name="Top" color="4" fill="1" visible="yes" active="yes"/>
@@
 <wire x1="315.5" y1="17" x2="315.5" y2="47" width="0.2032" layer="20"/>
 <wire x1="315.5" y1="47" x2="305.5" y2="47" width="0.2032" layer="20"/>
-<wire x1="305.5" y1="47" x2="305.5" y2="197.75" width="0.2032" layer="20"/>
-<wire x1="305.5" y1="197.75" x2="0" y2="197.75" width="0.2032" layer="20"/>
-<wire x1="0" y1="197.75" x2="0" y2="0" width="0.2032" layer="20"/>
+<wire x1="305.5" y1="47" x2="305.5" y2="197.125" width="0.2032" layer="20"/>
+<wire x1="305.5" y1="197.125" x2="0" y2="197.125" width="0.2032" layer="20"/>
+<wire x1="0" y1="197.125" x2="0" y2="0" width="0.2032" layer="20"/>
 <wire x1="0" y1="0" x2="53.563" y2="0" width="0.2032" layer="20"/>
 <wire x1="53.563" y1="0" x2="53.563" y2="19.32" width="0.2032" layer="20"/>
@@
 <polygon width="0.2032" layer="1">
 <vertex x="0" y="0"/>
-<vertex x="0" y="197.75"/>
-<vertex x="305.5" y="197.75"/>
+<vertex x="0" y="197.125"/>
+<vertex x="305.5" y="197.125"/>
 <vertex x="305.5" y="47"/>
 <vertex x="315.5" y="47"/>
@@
 <vertex x="301" y="0"/>
 <vertex x="315.5" y="0"/>
-<vertex x="315.5" y="197.75"/>
-<vertex x="301" y="197.75"/>
+<vertex x="315.5" y="197.125"/>
+<vertex x="301" y="197.125"/>
 </polygon>
 <via x="302.35" y="42.8" extent="1-16" drill="0.381"/>
@@
 <vertex x="60" y="0"/>
 <vertex x="300" y="0"/>
-<vertex x="300" y="197.75"/>
-<vertex x="0" y="197.75"/>
+<vertex x="300" y="197.125"/>
+<vertex x="0" y="197.125"/>
 <vertex x="0.17645625" y="21"/>
 <vertex x="60" y="21"/>

Commit message: polishing 13tb and 13r
Parts:
- removed D10, D105, D11, D12, D126, D147, D168, D189, D20, D210, D231, D247, D252, D253, D254, D42, D63, D84: WS2812B, SparkFun-LED:WS2812B
- removed JP10, JP105, JP11, JP12, JP126, JP147, JP168, JP189, JP20, JP210, JP231, JP247, JP252, JP253, JP254, JP42, JP63, JP84: JUMPER-SMT_2_NO_NO-SILK, SparkFun-Jumpers:SMT-JUMPER_2_NO_NO-SILK
- moved H2 46.8 mm to (134.9, 7.50)
- moved H1 35.8 mm to (170.6, 190.2)
- moved D248 12.2 mm to (70.2, 7.50)
- moved D249 12.2 mm to (85.2, 7.50)
- moved D250 12.2 mm to (100.2, 7.50)
- moved D251 12.2 mm to (115.2, 7.50)
- moved D255 12.2 mm to (176.5, 7.50)
- moved D256 12.2 mm to (190.2, 7.50)
- moved D257 12.2 mm to (205.2, 7.50)
- moved D258 12.2 mm to (220.2, 7.50)
- moved D259 12.2 mm to (235.2, 7.50)
- moved D260 12.2 mm to (250.2, 7.50)
- moved D261 12.2 mm to (265.2, 7.50)
- moved D262 12.2 mm to (280.2, 7.50)
- moved JP248 12.2 mm to (70.2, 7.50)
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Connections:
- removed net DIO10: D20.2, D22.4, JP20.2, JP22.1
- removed net DIO104: D209.2, D210.4, JP209.2, JP210.1
- removed net DIO121: D21.4, D231.2, JP21.1, JP231.2
- removed net DIO133: D252.2, D253.4, JP252.2, JP253.1
- removed net DIO5: D10.2, D11.4, JP10.2, JP11.1
- removed net N$125: D247.2, D248.4, JP247.2, JP248.1
- removed net N$127: D251.2, D252.4, JP251.2, JP252.1
- removed net N$129: D254.2, D255.4, JP254.2, JP255.1
- removed net N$135: D11.2, D12.4, JP11.2, JP12.1
- removed net N$15: D10.4, D9.2, JP10.1, JP9.2
- removed net N$28: D104.2, D105.4, JP104.2, JP105.1
- removed net N$32: D42.2, D43.4, JP42.2, JP43.1
- removed net N$44: D62.2, D63.4, JP62.2, JP63.1
- removed net N$54: D84.2, D85.4, JP84.2, JP85.1
- removed net N$68: D126.2, D127.4, JP126.2, JP127.1
- removed net N$79: D146.2, D147.4, JP146.2, JP147.1
- removed net N$89: D168.2, D169.4, JP168.2, JP169.1
- removed net N$97: D188.2, D189.4, JP188.2, JP189.1
- net DIO109: now also D209.2, JP209.2; no longer D210.2, JP210.2
- net DIO119: now also D21.4, JP21.1; no longer D231.4, JP231.1
- net DIO130: now also D248.4, JP248.1; no longer D247.4, JP247.1
- net DIO134: now also D251.2, D255.4, JP251.2, JP255.1; no longer D253.2, D254.4, JP253.2, JP254.1
- net DIO21: now also D43.4, JP43.1; no longer D42.4, JP42.1
- net DIO33: now also D62.2, JP62.2; no longer D63.2, JP63.2
- net DIO44: now also D85.4, JP85.1; no longer D84.4, JP84.1
- net DIO54: now also D104.2, JP104.2; no longer D105.2, JP105.2
- net DIO64: now also D127.4, JP127.1; no longer D126.4, JP126.1
- net DIO76: now also D146.2, JP146.2; no longer D147.2, JP147.2
- net DIO87: now also D169.4, JP169.1; no longer D168.4, JP168.1
- net DIO9: now also D22.4, JP22.1; no longer D20.4, JP20.1
- net DIO99: now also D188.2, JP188.2; no longer D189.2, JP189.2
- net GND: no longer D10.3, D105.3, D11.3, D12.3, D126.3, D147.3, D168.3, D189.3, D20.3, D210.3, D231.3, D247.3, D252.3, D253.3, D254.3, D42.3, D63.3, D84.3
- net N$8: now also D9.2, JP9.2; no longer D12.2, JP12.2
- net V_USB: no longer D10.1, D105.1, D11.1, D12.1, D126.1, D147.1, D168.1, D189.1, D20.1, D210.1, D231.1, D247.1, D252.1, D253.1, D254.1, D42.1, D63.1, D84.1
Routing:
- net DIO121: track 346.9 -> 0.00 mm, vias 2 -> 0
- net N$89: track 344.8 -> 0.00 mm, vias 2 -> 0
- net N$68: track 344.8 -> 0.00 mm, vias 2 -> 0
- net N$32: track 344.6 -> 0.00 mm, vias 2 -> 0
- net N$54: track 344.5 -> 0.00 mm, vias 2 -> 0
- net DIO10: track 312.5 -> 0.00 mm, vias 2 -> 0
- net DIO119: track 16.8 -> 305.8 mm, vias 0 -> 2
- net DIO64: track 16.8 -> 304.4 mm, vias 0 -> 2
- net DIO87: track 16.8 -> 304.4 mm, vias 0 -> 2
- net DIO44: track 16.8 -> 304.1 mm, vias 0 -> 2
- net DIO21: track 16.8 -> 304.0 mm, vias 0 -> 2
- net DIO9: track 16.8 -> 292.0 mm, vias 0 -> 2
- net N$125: track 269.8 -> 0.00 mm, vias 2 -> 0
- net DIO130: track 16.8 -> 244.4 mm, vias 0 -> 2
- net V_USB: track 572.3 -> 431.9 mm, vias 273 -> 256
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Other:
- outline, holes or cut-outs redrawn

Commit message: final touches, polishing, jumpers, CAM on all boards
Parts:
- added JP11, JP252, JP253, JP265, JP266, JP267, JP268, JP269, JP270, JP271, JP272, JP273: JUMPER-SMT_2_NO_NO-SILK, SparkFun-Jumpers:SMT-JUMPER_2_NO_NO-SILK
Connections:
- removed net DIO109: D1.4, D209.2, JP1.1, JP209.2
- removed net DIO119: D21.4, D230.2, JP21.1, JP230.2
- removed net DIO130: D246.2, D248.4, JP246.2, JP248.1
- removed net DIO21: D41.2, D43.4, JP41.2, JP43.1
- removed net DIO33: D62.2, D64.4, JP62.2, JP64.1
- removed net DIO44: D83.2, D85.4, JP83.2, JP85.1
- removed net DIO54: D104.2, D106.4, JP104.2, JP106.1
- removed net DIO64: D125.2, D127.4, JP125.2, JP127.1
- removed net DIO76: D146.2, D148.4, JP146.2, JP148.1
- removed net DIO87: D167.2, D169.4, JP167.2, JP169.1
- removed net DIO9: D19.2, D22.4, JP19.2, JP22.1
- removed net DIO99: D188.2, D190.4, JP188.2, JP190.1
- new net JUMPER0: D19.2, D22.4, JP11.2, JP19.2, JP22.1, JP252.1
- new net JUMPER1: D41.2, D43.4, JP252.2, JP253.1, JP41.2, JP43.1
- new net JUMPER10: D21.4, D230.2, JP21.1, JP230.2, JP272.2, JP273.1
- new net JUMPER11: D246.2, D248.4, JP246.2, JP248.1, JP273.2
- new net JUMPER2: D62.2, D64.4, JP253.2, JP265.1, JP62.2, JP64.1
- new net JUMPER3: D83.2, D85.4, JP265.2, JP266.1, JP83.2, JP85.1
- new net JUMPER4: D104.2, D106.4, JP104.2, JP106.1, JP266.2, JP267.1
- new net JUMPER5: D125.2, D127.4, JP125.2, JP127.1, JP267.2, JP268.1
- new net JUMPER6: D146.2, D148.4, JP146.2, JP148.1, JP268.2, JP269.1
- new net JUMPER7: D167.2, D169.4, JP167.2, JP169.1, JP269.2, JP270.1
- new net JUMPER8: D188.2, D190.4, JP188.2, JP190.1, JP270.2, JP271.1
- new net JUMPER9: D1.4, D209.2, JP1.1, JP209.2, JP271.2, JP272.1
- net DIO0: now also JP11.1
Routing:
- net JUMPER10: track 0.00 -> 327.1 mm, vias 0 -> 4
- net JUMPER9: track 0.00 -> 322.3 mm, vias 0 -> 2
- net JUMPER5: track 0.00 -> 321.2 mm, vias 0 -> 2
- net JUMPER7: track 0.00 -> 321.2 mm, vias 0 -> 2
- net JUMPER4: track 0.00 -> 321.2 mm, vias 0 -> 2
- net JUMPER6: track 0.00 -> 321.2 mm, vias 0 -> 2
- net JUMPER8: track 0.00 -> 321.2 mm, vias 0 -> 2
- net JUMPER3: track 0.00 -> 321.0 mm, vias 0 -> 2
- net JUMPER2: track 0.00 -> 320.9 mm, vias 0 -> 2
- net JUMPER1: track 0.00 -> 320.9 mm, vias 0 -> 2
- net JUMPER0: track 0.00 -> 308.9 mm, vias 0 -> 2
- net DIO119: track 305.8 -> 0.00 mm, vias 2 -> 0
- net DIO109: track 305.4 -> 0.00 mm, vias 2 -> 0
- net DIO64: track 304.4 -> 0.00 mm, vias 2 -> 0
- net DIO87: track 304.4 -> 0.00 mm, vias 2 -> 0
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
Commit message: pushing final board changes
Parts:
- removed D13, D14, D15, D16, D17, D18, D19, D2, D22, D3, D31, D32, D33, D4, D41, D5, D6, D7, D8, D9: WS2812B, SparkFun-LED:WS2812B
- removed JP11, JP13, JP14, JP15, JP16, JP17, JP18, JP19, JP2, JP22, JP3, JP31, JP32, JP33, JP4, JP41, JP5, JP6, JP7, JP8, JP9: JUMPER-SMT_2_NO_NO-SILK, SparkFun-Jumpers:SMT-JUMPER_2_NO_NO-SILK
- added U$1: (no value), unnamed#png (2):UNNAMED#PNG
- moved R5 18.7 mm to (303.5, 30.0), turned to 180 degrees
- moved R3 18.5 mm to (305.3, 24.3)
- moved R4 18.5 mm to (305.3, 21.8)
- moved J2 18.5 mm to (309.0, 23.0)
- moved J3 17.0 mm to (315.5, 41.0)
- moved C3 16.5 mm to (303.5, 31.5)
- moved R12 16.5 mm to (303.5, 33.0)
- moved R15 16.0 mm to (303.5, 34.5)
- moved C8 7.44 mm to (9.80, 21.9), turned to 270 degrees
- moved FD1 7.12 mm to (302.8, 187.9)
- moved H1 7.12 mm to (170.6, 183.1)
- moved H5 7.12 mm to (298.0, 183.1)
- moved H6 7.12 mm to (7.50, 183.1)
- moved C7 6.48 mm to (7.33, 16.9), turned to 180 degrees
- moved R8 6.17 mm to (5.10, 21.8), turned to 90 degrees
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Connections:
- removed net DIO11: D22.2, D23.4, JP22.2, JP23.1
- removed net DIO16: D32.2, D33.4, JP32.2, JP33.1
- removed net DIO17: D33.2, D34.4, JP33.2, JP34.1
- removed net DIO3: D6.2, D7.4, JP6.2, JP7.1
- removed net DIO4: D8.2, D9.4, JP8.2, JP9.1
- removed net DIO6: D13.2, D14.4, JP13.2, JP14.1
- removed net DIO7: D15.2, D16.4, JP15.2, JP16.1
- removed net DIO8: D17.2, D18.4, JP17.2, JP18.1
- removed net JUMPER0: D19.2, D22.4, JP11.2, JP19.2, JP22.1, JP252.1
- removed net N$120: D2.2, D3.4, JP2.2, JP3.1
- removed net N$121: D4.2, D5.4, JP4.2, JP5.1
- removed net N$13: D3.2, D4.4, JP3.2, JP4.1
- removed net N$14: D5.2, D6.4, JP5.2, JP6.1
- removed net N$17: D7.2, D8.4, JP7.2, JP8.1
- removed net N$18: D16.2, D17.4, JP16.2, JP17.1
- removed net N$20: D14.2, D15.4, JP14.2, JP15.1
- removed net N$22: D18.2, D19.4, JP18.2, JP19.1
- removed net N$26: D31.2, D32.4, JP31.2, JP32.1
- removed net N$33: D40.2, D41.4, JP40.2, JP41.1
- removed net N$8: D13.4, D9.2, JP13.1, JP9.2
- net DIO0: now also D23.4, JP23.1, JP252.1; no longer D2.4, JP11.1, JP2.1
- net DIO15: now also D34.4, JP34.1; no longer D31.4, JP31.1
- net GND: no longer D13.3, D14.3, D15.3, D16.3, D17.3, D18.3, D19.3, D2.3, D22.3, D3.3, D31.3, D32.3, D33.3, D4.3, D41.3, D5.3, D6.3, D7.3, D8.3, D9.3
- net JUMPER1: now also D40.2, JP40.2; no longer D41.2, JP41.2
- net V_USB: no longer D13.1, D14.1, D15.1, D16.1, D17.1, D18.1, D19.1, D2.1, D22.1, D3.1, D31.1, D32.1, D33.1, D4.1, D41.1, D5.1, D6.1, D7.1, D8.1, D9.1
Routing:
- net JUMPER0: track 308.9 -> 0.00 mm, vias 2 -> 0
- net N$8: track 61.8 -> 0.00 mm
- net DIO15: track 16.8 -> 61.8 mm
- net V_USB: track 431.9 -> 399.6 mm, vias 256 -> 235
- net N$26: track 16.8 -> 0.00 mm
- net N$20: track 16.8 -> 0.00 mm
- net N$18: track 16.8 -> 0.00 mm
- net DIO7: track 16.8 -> 0.00 mm
- net DIO6: track 16.8 -> 0.00 mm
- net DIO17: track 16.8 -> 0.00 mm
- net DIO16: track 16.8 -> 0.00 mm
- net DIO4: track 16.8 -> 0.00 mm
- net N$13: track 16.8 -> 0.00 mm
- net N$121: track 16.8 -> 0.00 mm
- net N$17: track 16.8 -> 0.00 mm
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Other:
- board size 315.5 x 197.1 mm -> 315.5 x 190 mm
- board text added: "v12"
- board text removed: "v11"

Commit message: updating files
Parts:
- removed FD2: FIDUCIALUFIDUCIAL, SparkFun-Aesthetics:FIDUCIAL-MICRO
Changed lines of the file:
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@@
 </element>
 <element name="FD1" library="SparkFun-Aesthetics" package="FIDUCIAL-MICRO" value="FIDUCIALUFIDUCIAL" x="302.75" y="187.875" smashed="yes"/>
-<element name="FD2" library="SparkFun-Aesthetics" package="FIDUCIAL-MICRO" value="FIDUCIALUFIDUCIAL" x="6.5" y="47.5" smashed="yes"/>
 <element name="FD4" library="SparkFun-Aesthetics" package="FIDUCIAL-MICRO" value="FIDUCIALUFIDUCIAL" x="10.5" y="9" smashed="yes" rot="R90"/>
 <element name="FRAME1" library="SparkFun-Aesthetics" package="CREATIVE_COMMONS" value="FRAME-LEDGER" x="7.62" y="-8.89" smashed="yes">
