File: Hardware/13R.sch (EAGLE design)
At the start: 578 parts, among them J2 USB Female Type C Connector, J3 AUDIO_JACK_TRRSSMD_RA, Q2 MBT3904DW1T1, U2 ESP-WROOM-32NARROW, U3 AP2112K-3.3V, U4 CP2102N, U5 ADMP401

Commit message: polishing 13tb and 13r
Parts:
- removed D10, D105, D11, D12, D126, D147, D168, D189, D20, D210, D231, D247, D252, D253, D254, D42, D63, D84: WS2812B, SparkFun-LED:WS2812B
- removed JP10, JP105, JP11, JP12, JP126, JP147, JP168, JP189, JP20, JP210, JP231, JP247, JP252, JP253, JP254, JP42, JP63, JP84: JUMPER-SMT_2_NO_NO-SILK, SparkFun-Jumpers:JUMPER-SMT_2_NO_NO-SILK
Connections:
- removed net DIO10: D20.DO, D22.DI, JP20.2, JP22.1
- removed net DIO104: D209.DO, D210.DI, JP209.2, JP210.1
- removed net DIO121: D21.DI, D231.DO, JP21.1, JP231.2
- removed net DIO133: D252.DO, D253.DI, JP252.2, JP253.1
- removed net DIO5: D10.DO, D11.DI, JP10.2, JP11.1
- removed net N$125: D247.DO, D248.DI, JP247.2, JP248.1
- removed net N$127: D251.DO, D252.DI, JP251.2, JP252.1
- removed net N$129: D254.DO, D255.DI, JP254.2, JP255.1
- removed net N$135: D11.DO, D12.DI, JP11.2, JP12.1
- removed net N$15: D10.DI, D9.DO, JP10.1, JP9.2
- removed net N$28: D104.DO, D105.DI, JP104.2, JP105.1
- removed net N$32: D42.DO, D43.DI, JP42.2, JP43.1
- removed net N$44: D62.DO, D63.DI, JP62.2, JP63.1
- removed net N$54: D84.DO, D85.DI, JP84.2, JP85.1
- removed net N$68: D126.DO, D127.DI, JP126.2, JP127.1
- removed net N$79: D146.DO, D147.DI, JP146.2, JP147.1
- removed net N$89: D168.DO, D169.DI, JP168.2, JP169.1
- removed net N$97: D188.DO, D189.DI, JP188.2, JP189.1
- net DIO109: now also D209.DO, JP209.2; no longer D210.DO, JP210.2
- net DIO119: now also D21.DI, JP21.1; no longer D231.DI, JP231.1
- net DIO130: now also D248.DI, JP248.1; no longer D247.DI, JP247.1
- net DIO134: now also D251.DO, D255.DI, JP251.2, JP255.1; no longer D253.DO, D254.DI, JP253.2, JP254.1
- net DIO21: now also D43.DI, JP43.1; no longer D42.DI, JP42.1
- net DIO33: now also D62.DO, JP62.2; no longer D63.DO, JP63.2
- net DIO44: now also D85.DI, JP85.1; no longer D84.DI, JP84.1
- net DIO54: now also D104.DO, JP104.2; no longer D105.DO, JP105.2
- net DIO64: now also D127.DI, JP127.1; no longer D126.DI, JP126.1
- net DIO76: now also D146.DO, JP146.2; no longer D147.DO, JP147.2
- net DIO87: now also D169.DI, JP169.1; no longer D168.DI, JP168.1
- net DIO9: now also D22.DI, JP22.1; no longer D20.DI, JP20.1
- net DIO99: now also D188.DO, JP188.2; no longer D189.DO, JP189.2
- net GND: no longer D10.VSS, D105.VSS, D11.VSS, D12.VSS, D126.VSS, D147.VSS, D168.VSS, D189.VSS, D20.VSS, D210.VSS, D231.VSS, D247.VSS, D252.VSS, D253.VSS, D254.VSS, D42.VSS, D63.VSS, D84.VSS
- net N$8: now also D9.DO, JP9.2; no longer D12.DO, JP12.2
- net V_USB: no longer D10.VDD, D105.VDD, D11.VDD, D12.VDD, D126.VDD, D147.VDD, D168.VDD, D189.VDD, D20.VDD, D210.VDD, D231.VDD, D247.VDD, D252.VDD, D253.VDD, D254.VDD, D42.VDD, D63.VDD, D84.VDD

Commit message: final touches, polishing, jumpers, CAM on all boards
Parts:
- added JP11, JP252, JP253, JP265, JP266, JP267, JP268, JP269, JP270, JP271, JP272, JP273: JUMPER-SMT_2_NO_NO-SILK, SparkFun-Jumpers:JUMPER-SMT_2_NO_NO-SILK
Connections:
- removed net DIO109: D1.DI, D209.DO, JP1.1, JP209.2
- removed net DIO119: D21.DI, D230.DO, JP21.1, JP230.2
- removed net DIO130: D246.DO, D248.DI, JP246.2, JP248.1
- removed net DIO21: D41.DO, D43.DI, JP41.2, JP43.1
- removed net DIO33: D62.DO, D64.DI, JP62.2, JP64.1
- removed net DIO44: D83.DO, D85.DI, JP83.2, JP85.1
- removed net DIO54: D104.DO, D106.DI, JP104.2, JP106.1
- removed net DIO64: D125.DO, D127.DI, JP125.2, JP127.1
- removed net DIO76: D146.DO, D148.DI, JP146.2, JP148.1
- removed net DIO87: D167.DO, D169.DI, JP167.2, JP169.1
- removed net DIO9: D19.DO, D22.DI, JP19.2, JP22.1
- removed net DIO99: D188.DO, D190.DI, JP188.2, JP190.1
- new net JUMPER0: D19.DO, D22.DI, JP11.2, JP19.2, JP22.1, JP252.1
- new net JUMPER1: D41.DO, D43.DI, JP252.2, JP253.1, JP41.2, JP43.1
- new net JUMPER10: D21.DI, D230.DO, JP21.1, JP230.2, JP272.2, JP273.1
- new net JUMPER11: D246.DO, D248.DI, JP246.2, JP248.1, JP273.2
- new net JUMPER2: D62.DO, D64.DI, JP253.2, JP265.1, JP62.2, JP64.1
- new net JUMPER3: D83.DO, D85.DI, JP265.2, JP266.1, JP83.2, JP85.1
- new net JUMPER4: D104.DO, D106.DI, JP104.2, JP106.1, JP266.2, JP267.1
- new net JUMPER5: D125.DO, D127.DI, JP125.2, JP127.1, JP267.2, JP268.1
- new net JUMPER6: D146.DO, D148.DI, JP146.2, JP148.1, JP268.2, JP269.1
- new net JUMPER7: D167.DO, D169.DI, JP167.2, JP169.1, JP269.2, JP270.1
- new net JUMPER8: D188.DO, D190.DI, JP188.2, JP190.1, JP270.2, JP271.1
- new net JUMPER9: D1.DI, D209.DO, JP1.1, JP209.2, JP271.2, JP272.1
- net DIO0: now also JP11.1

Commit message: pushing final board changes
Parts:
- removed D13, D14, D15, D16, D17, D18, D19, D2, D22, D3, D31, D32, D33, D4, D41, D5, D6, D7, D8, D9: WS2812B, SparkFun-LED:WS2812B
- removed JP11, JP13, JP14, JP15, JP16, JP17, JP18, JP19, JP2, JP22, JP3, JP31, JP32, JP33, JP4, JP41, JP5, JP6, JP7, JP8, JP9: JUMPER-SMT_2_NO_NO-SILK, SparkFun-Jumpers:JUMPER-SMT_2_NO_NO-SILK
Connections:
- removed net DIO11: D22.DO, D23.DI, JP22.2, JP23.1
- removed net DIO16: D32.DO, D33.DI, JP32.2, JP33.1
- removed net DIO17: D33.DO, D34.DI, JP33.2, JP34.1
- removed net DIO3: D6.DO, D7.DI, JP6.2, JP7.1
- removed net DIO4: D8.DO, D9.DI, JP8.2, JP9.1
- removed net DIO6: D13.DO, D14.DI, JP13.2, JP14.1
- removed net DIO7: D15.DO, D16.DI, JP15.2, JP16.1
- removed net DIO8: D17.DO, D18.DI, JP17.2, JP18.1
- removed net JUMPER0: D19.DO, D22.DI, JP11.2, JP19.2, JP22.1, JP252.1
- removed net N$120: D2.DO, D3.DI, JP2.2, JP3.1
- removed net N$121: D4.DO, D5.DI, JP4.2, JP5.1
- removed net N$13: D3.DO, D4.DI, JP3.2, JP4.1
- removed net N$14: D5.DO, D6.DI, JP5.2, JP6.1
- removed net N$17: D7.DO, D8.DI, JP7.2, JP8.1
- removed net N$18: D16.DO, D17.DI, JP16.2, JP17.1
- removed net N$20: D14.DO, D15.DI, JP14.2, JP15.1
- removed net N$22: D18.DO, D19.DI, JP18.2, JP19.1
- removed net N$26: D31.DO, D32.DI, JP31.2, JP32.1
- removed net N$33: D40.DO, D41.DI, JP40.2, JP41.1
- removed net N$8: D13.DI, D9.DO, JP13.1, JP9.2
- net DIO0: now also D23.DI, JP23.1, JP252.1; no longer D2.DI, JP11.1, JP2.1
- net DIO15: now also D34.DI, JP34.1; no longer D31.DI, JP31.1
- net GND: no longer D13.VSS, D14.VSS, D15.VSS, D16.VSS, D17.VSS, D18.VSS, D19.VSS, D2.VSS, D22.VSS, D3.VSS, D31.VSS, D32.VSS, D33.VSS, D4.VSS, D41.VSS, D5.VSS, D6.VSS, D7.VSS, D8.VSS, D9.VSS
- net JUMPER1: now also D40.DO, JP40.2; no longer D41.DO, JP41.2
- net V_USB: no longer D13.VDD, D14.VDD, D15.VDD, D16.VDD, D17.VDD, D18.VDD, D19.VDD, D2.VDD, D22.VDD, D3.VDD, D31.VDD, D32.VDD, D33.VDD, D4.VDD, D41.VDD, D5.VDD, D6.VDD, D7.VDD, D8.VDD, D9.VDD

Commit message: updating files
Parts:
- removed FD2: FIDUCIALUFIDUCIAL, SparkFun-Aesthetics:FIDUCIALUFIDUCIAL
Changed lines of the file:
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@@
 <part name="C1" library="SparkFun-Capacitors" deviceset="10UF" device="-0603-6.3V-20%" value="10uF"/>
 <part name="FD1" library="SparkFun-Aesthetics" deviceset="FIDUCIAL" device="UFIDUCIAL"/>
-<part name="FD2" library="SparkFun-Aesthetics" deviceset="FIDUCIAL" device="UFIDUCIAL"/>
 <part name="FD4" library="SparkFun-Aesthetics" deviceset="FIDUCIAL" device="UFIDUCIAL"/>
 <part name="S2" library="SparkFun-Switches" deviceset="MOMENTARY-SWITCH-SPST-2" device="-SMD-4.6X2.8MM" value="0"/>
@@
 </instance>
 <instance part="FD1" gate="G$1" x="429.26" y="33.02" smashed="yes"/>
-<instance part="FD2" gate="G$1" x="426.72" y="33.02" smashed="yes"/>
 <instance part="FD4" gate="G$1" x="429.26" y="30.48" smashed="yes"/>
 <instance part="S2" gate="G$1" x="294.64" y="177.8" smashed="yes">
