File: Hardware/13TB.brd (EAGLE design)
At the start: 326.5 x 197.8 mm, 569 parts, among them J2 USB Female Type C Connector, J3 AUDIO_JACK_TRRSSMD_RA, Q2 MBT3904DW1T1, U2 ESP-WROOM-32NARROW, U3 AP2112K-3.3V, U4 CP2102N, U5 ADMP401

Commit message: updating 15TB outer dimensions, still need to re-place holes
Parts:
- added D1, D21, D211, D263, D264: WS2812B, SparkFun-LED:WS2812B
- added JP1, JP21, JP211, JP263, JP264: JUMPER-SMT_2_NO_NO-SILK, SparkFun-Jumpers:SMT-JUMPER_2_NO_NO-SILK
- R13: value 1k -> 2.2k; device SparkFun-Resistors:AXIAL-0.3 -> SparkFun-Resistors:0603
- moved J3 333.3 mm to (324.5, 30.1), turned to 180 degrees
- moved J2 322.3 mm to (319.0, 47.4), turned to 90 degrees
- moved R3 316.2 mm to (315.8, 48.8), turned to 0 degrees
- moved R4 315.7 mm to (315.8, 46.3), turned to 0 degrees
- moved R14 312.8 mm to (318.0, 35.5), turned to 180 degrees
- moved R6 312.4 mm to (320.0, 38.0), turned to 90 degrees
- moved C2 310.4 mm to (318.0, 38.0), turned to 90 degrees
- moved R15 308.5 mm to (313.5, 24.5), turned to 0 degrees
- moved R7 308.3 mm to (316.0, 38.0), turned to 270 degrees
- moved R12 306.1 mm to (313.5, 22.5), turned to 180 degrees
- moved C3 306.1 mm to (313.5, 21.0), turned to 0 degrees
- moved R5 304.5 mm to (311.8, 17.5)
- moved U5 59.6 mm to (12.7, 17.5), turned to 270 degrees
- moved C4 53.8 mm to (17.6, 17.4), turned to 270 degrees
- moved R10 53.8 mm to (19.5, 13.3), turned to 270 degrees
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Connections:
- removed net DIO120: D231.2, D232.4, JP231.2, JP232.1
- new net DIO121: D21.4, D231.2, JP21.1, JP231.2
- new net DIO127: D211.2, D263.4, JP211.2, JP263.1
- new net N$138: D263.2, D264.4, JP263.2, JP264.1
- new net N$140: D232.4, D264.2, JP232.1, JP264.2
- new net N$2: D21.2, D211.4, JP21.2, JP211.1
- new net N$21: D1.2, D212.4, JP1.2, JP212.1
- net DIO109: now also D1.4, JP1.1; no longer D212.4, JP212.1
- net GND: now also D1.3, D21.3, D211.3, D263.3, D264.3
- net N$11: now also R13.1; no longer R13.P$1
- net N$9: now also R13.2; no longer R13.P$2
- net V_USB: now also D1.1, D21.1, D211.1, D263.1, D264.1
Routing:
- net DIO121: track 0.00 -> 321.3 mm, vias 0 -> 2
- net D-: track 31.8 -> 335.4 mm
- net D+: track 31.5 -> 333.5 mm
- net RING1: track 45.2 -> 293.8 mm
- net DIO120: track 243.9 -> 0.00 mm, vias 2 -> 0
- net TIP: track 48.1 -> 290.9 mm, vias 2 -> 0
- net 3.3V: track 167.3 -> 407.7 mm, vias 10 -> 8
- net V_USB: track 553.2 -> 447.0 mm, vias 267 -> 273
- net DIO127: track 0.00 -> 31.8 mm, vias 0 -> 2
- net DIO0: track 234.7 -> 213.1 mm
- net N$2: track 0.00 -> 18.0 mm, vias 0 -> 2
- net N$21: track 0.00 -> 16.8 mm
- net N$140: track 0.00 -> 16.8 mm
- net N$138: track 0.00 -> 16.8 mm
- net DIO109: track 304.1 -> 320.2 mm
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Other:
- outline, holes or cut-outs redrawn
- board text added: "13R"
- board text removed: "13TB"
- board text removed: "D"

Commit message: getting 4 boards polished
Parts:
- removed D10, D104, D105, D11, D12, D125, D126, D13, D14, D146, D147, D15, D16, D167, D168, D17, D18, D184, D185, D188, D189, D19, D20, D209, D210, D22, D230, D231, D246, D247, D262, D4, D40, D41, D42, D5, D6, D62, D63, D7, D8, D83, D84, D9: WS2812B, SparkFun-LED:WS2812B
- removed JP10, JP104, JP105, JP11, JP12, JP125, JP126, JP13, JP14, JP146, JP147, JP15, JP16, JP167, JP168, JP17, JP18, JP188, JP189, JP19, JP2, JP20, JP209, JP210, JP22, JP230, JP231, JP246, JP247, JP262, JP3, JP4, JP40, JP41, JP42, JP5, JP6, JP62, JP63, JP7, JP8, JP83, JP84, JP9: JUMPER-SMT_2_NO_NO-SILK, SparkFun-Jumpers:SMT-JUMPER_2_NO_NO-SILK
- moved D2 246.5 mm to (237.8, 67.5)
- moved D3 246.5 mm to (252.8, 67.5)
- moved C2 20.9 mm to (297.1, 38.0)
- moved C3 20.9 mm to (292.6, 21.0)
- moved H3 20.9 mm to (288.1, 7.50)
- moved J2 20.9 mm to (298.1, 47.4)
- moved J3 20.9 mm to (303.6, 30.1)
- moved R12 20.9 mm to (292.6, 22.5)
- moved R14 20.9 mm to (297.1, 35.5)
- moved R15 20.9 mm to (292.6, 24.5)
- moved R3 20.9 mm to (294.9, 48.8)
- moved R4 20.9 mm to (294.9, 46.3)
- moved R5 20.9 mm to (290.9, 17.5)
- moved R6 20.9 mm to (299.1, 38.0)
- moved R7 20.9 mm to (295.1, 38.0)
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Connections:
- removed net DIO10: D20.2, D22.4, JP20.2, JP22.1
- removed net DIO104: D209.2, D210.4, JP209.2, JP210.1
- removed net DIO108: D208.2, D209.4, JP208.2, JP209.1
- removed net DIO11: D22.2, D23.4, JP22.2, JP23.1
- removed net DIO119: D230.2, D231.4, JP230.2, JP231.1
- removed net DIO130: D246.2, D247.4, JP246.2, JP247.1
- removed net DIO21: D41.2, D42.4, JP41.2, JP42.1
- removed net DIO3: D6.2, D7.4, JP6.2, JP7.1
- removed net DIO33: D63.2, D64.4, JP63.2, JP64.1
- removed net DIO4: D8.2, D9.4, JP8.2, JP9.1
- removed net DIO44: D83.2, D84.4, JP83.2, JP84.1
- removed net DIO5: D10.2, D11.4, JP10.2, JP11.1
- removed net DIO53: D103.2, D104.4, JP103.2, JP104.1
- removed net DIO6: D13.2, D14.4, JP13.2, JP14.1
- removed net DIO64: D125.2, D126.4, JP125.2, JP126.1
- removed net DIO7: D15.2, D16.4, JP15.2, JP16.1
- removed net DIO75: D145.2, D146.4, JP145.2, JP146.1
- removed net DIO8: D17.2, D18.4, JP17.2, JP18.1
- removed net DIO87: D167.2, D168.4, JP167.2, JP168.1
- removed net DIO9: D19.2, D20.4, JP19.2, JP20.1
- removed net DIO99: D189.2, D190.4, JP189.2, JP190.1
- removed net N$115: D229.2, D230.4, JP229.2, JP230.1
- removed net N$120: D2.2, D3.4, JP2.2, JP3.1
- removed net N$121: D4.2, D5.4, JP4.2, JP5.1
- removed net N$126: D245.2, D246.4, JP245.2, JP246.1
- removed net N$13: D3.2, D4.4, JP3.2, JP4.1
- removed net N$132: D262.2, JP262.2
- removed net N$135: D11.2, D12.4, JP11.2, JP12.1
- removed net N$14: D5.2, D6.4, JP5.2, JP6.1
- removed net N$15: D10.4, D9.2, JP10.1, JP9.2
- removed net N$17: D7.2, D8.4, JP7.2, JP8.1
- removed net N$18: D16.2, D17.4, JP16.2, JP17.1
- removed net N$20: D14.2, D15.4, JP14.2, JP15.1
- removed net N$22: D18.2, D19.4, JP18.2, JP19.1
- removed net N$28: D104.2, D105.4, JP104.2, JP105.1
- removed net N$32: D42.2, D43.4, JP42.2, JP43.1
- removed net N$33: D40.2, D41.4, JP40.2, JP41.1
- removed net N$44: D62.2, D63.4, JP62.2, JP63.1
- removed net N$51: D82.2, D83.4, JP82.2, JP83.1
- removed net N$69: D124.2, D125.4, JP124.2, JP125.1
- removed net N$79: D146.2, D147.4, JP146.2, JP147.1
- removed net N$8: D12.2, D13.4, JP12.2, JP13.1
- removed net N$87: D166.2, D167.4, JP166.2, JP167.1
- removed net N$97: D188.2, D189.4, JP188.2, JP189.1
- net DIO0: now also D23.4, JP23.1; no longer D2.4, JP2.1
- net DIO109: now also D208.2, JP208.2; no longer D210.2, JP210.2
- net DIO121: now also D229.2, JP229.2; no longer D231.2, JP231.2
- net DIO138: no longer D262.4, JP262.1
- net DIO20: now also D43.4, JP43.1; no longer D40.4, JP40.1
- net DIO32: now also D64.4, JP64.1; no longer D62.4, JP62.1
- net DIO54: now also D103.2, JP103.2; no longer D105.2, JP105.2
- net DIO76: now also D145.2, JP145.2; no longer D147.2, JP147.2
- net DIO96: now also D2.2, D3.4; no longer D184.2, D185.4
- net DIO98: now also D190.4, JP190.1; no longer D188.4, JP188.1
- net GND: no longer D10.3, D104.3, D105.3, D11.3, D12.3, D125.3, D126.3, D13.3, D14.3, D146.3, D147.3, D15.3, D16.3, D167.3, D168.3, D17.3, D18.3, D184.3, D185.3, D188.3, D189.3, D19.3, D20.3, D209.3, D210.3, D22.3, D230.3, D231.3, D246.3, D247.3, D262.3, D4.3, D40.3, D41.3, D42.3, D5.3, D6.3, D62.3, D63.3, D7.3, D8.3, D83.3, D84.3, D9.3
- net N$125: now also D245.2, JP245.2; no longer D247.2, JP247.2
- net N$54: now also D82.2, JP82.2; no longer D84.2, JP84.2
- net N$68: now also D124.2, JP124.2; no longer D126.2, JP126.2
- net N$89: now also D166.2, JP166.2; no longer D168.2, JP168.2
- net N$95: now also D3.2; no longer D185.2
- net N$96: now also D2.4; no longer D184.4
- net V_USB: no longer D10.1, D104.1, D105.1, D11.1, D12.1, D125.1, D126.1, D13.1, D14.1, D146.1, D147.1, D15.1, D16.1, D167.1, D168.1, D17.1, D18.1, D184.1, D185.1, D188.1, D189.1, D19.1, D20.1, D209.1, D210.1, D22.1, D230.1, D231.1, D246.1, D247.1, D262.1, D4.1, D40.1, D41.1, D42.1, D5.1, D6.1, D62.1, D63.1, D7.1, D8.1, D83.1, D84.1, D9.1
Routing:
- net DIO99: track 319.1 -> 0.00 mm, vias 2 -> 0
- net N$32: track 318.9 -> 0.00 mm, vias 2 -> 0
- net DIO33: track 318.9 -> 0.00 mm, vias 2 -> 0
- net DIO10: track 312.5 -> 0.00 mm, vias 2 -> 0
- net DIO20: track 16.8 -> 321.2 mm, vias 0 -> 2
- net DIO98: track 16.8 -> 320.0 mm, vias 0 -> 2
- net DIO32: track 16.8 -> 319.6 mm, vias 0 -> 2
- net V_USB: track 447.0 -> 386.2 mm, vias 273 -> 229
- net D-: track 335.4 -> 308.9 mm
- net D+: track 333.5 -> 309.5 mm
- net RING1: track 293.8 -> 270.8 mm
- net TIP: track 290.9 -> 268.0 mm
- net DIO0: track 213.1 -> 194.3 mm
- net N$8: track 16.8 -> 0.00 mm
- net N$20: track 16.8 -> 0.00 mm
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Other:
- board size 326.5 x 197.8 mm -> 305.6 x 182.9 mm
- board text added: "13TB"
- board text removed: "13R"

Commit message: polishing 13tb and 13r
Parts:
- removed D251, D252, D253, D31, D32, D33: WS2812B, SparkFun-LED:WS2812B
- removed JP251, JP252, JP253, JP31, JP32, JP33: JUMPER-SMT_2_NO_NO-SILK, SparkFun-Jumpers:SMT-JUMPER_2_NO_NO-SILK
- moved H2 57.2 mm to (129.8, 7.75)
- moved D254 45.0 mm to (117.8, 7.50)
- moved D30 45.0 mm to (177.8, 172.5)
- moved JP254 45.0 mm to (117.8, 7.50)
- moved JP30 45.0 mm to (177.8, 172.5)
- moved H1 34.5 mm to (165.8, 175.2)
- moved H5 26.0 mm to (287.9, 175.2)
- moved H6 15.1 mm to (7.75, 175.2)
- moved FD4 8.86 mm to (2.00, 11.5)
- moved R13 7.83 mm to (27.7, 18.8)
- moved C4 7.15 mm to (24.7, 17.4)
- moved U5 6.15 mm to (18.9, 17.6)
- moved C5 3.35 mm to (27.7, 15.1)
- moved R11 3.35 mm to (27.7, 17.0)
- moved D255 1.25 mm to (177.8, 7.50)
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Connections:
- removed net DIO133: D252.2, D253.4, JP252.2, JP253.1
- removed net DIO134: D253.2, D254.4, JP253.2, JP254.1
- removed net DIO16: D32.2, D33.4, JP32.2, JP33.1
- removed net DIO17: D33.2, D34.4, JP33.2, JP34.1
- removed net N$127: D251.2, D252.4, JP251.2, JP252.1
- removed net N$26: D31.2, D32.4, JP31.2, JP32.1
- net DIO132: now also D254.4, JP254.1; no longer D251.4, JP251.1
- net DIO15: now also D34.4, JP34.1; no longer D31.4, JP31.1
- net GND: no longer D251.3, D252.3, D253.3, D31.3, D32.3, D33.3
- net V_USB: no longer D251.1, D252.1, D253.1, D31.1, D32.1, D33.1
Routing:
- net DIO20: track 321.2 -> 273.9 mm
- net N$27: track 16.8 -> 61.8 mm
- net N$129: track 21.3 -> 61.8 mm
- net DIO98: track 320.0 -> 289.0 mm
- net DIO109: track 321.0 -> 290.1 mm
- net DIO32: track 319.6 -> 288.8 mm
- net N$89: track 318.8 -> 289.0 mm
- net N$68: track 318.8 -> 289.0 mm
- net N$54: track 318.5 -> 288.8 mm
- net DIO76: track 318.8 -> 289.0 mm
- net DIO54: track 318.8 -> 289.0 mm
- net DIO121: track 320.7 -> 291.2 mm
- net N$125: track 257.4 -> 229.0 mm
- net DIO134: track 16.8 -> 0.00 mm
- net DIO133: track 16.8 -> 0.00 mm
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
Commit message: final touches, polishing, jumpers, CAM on all boards
Parts:
- added JP11, JP252, JP253, JP265, JP266, JP267, JP268, JP269, JP270, JP271, JP272: JUMPER-SMT_2_NO_NO-SILK, SparkFun-Jumpers:SMT-JUMPER_2_NO_NO-SILK
Connections:
- removed net DIO109: D1.4, D208.2, JP1.1, JP208.2
- removed net DIO121: D21.4, D229.2, JP21.1, JP229.2
- removed net DIO20: D39.2, D43.4, JP39.2, JP43.1
- removed net DIO32: D61.2, D64.4, JP61.2, JP64.1
- removed net DIO54: D103.2, D106.4, JP103.2, JP106.1
- removed net DIO76: D145.2, D148.4, JP145.2, JP148.1
- removed net DIO98: D187.2, D190.4, JP187.2, JP190.1
- removed net N$125: D245.2, D248.4, JP245.2, JP248.1
- removed net N$54: D82.2, D85.4, JP82.2, JP85.1
- removed net N$68: D124.2, D127.4, JP124.2, JP127.1
- removed net N$89: D166.2, D169.4, JP166.2, JP169.1
- new net JUMPER0: D39.2, D43.4, JP11.2, JP252.1, JP39.2, JP43.1
- new net JUMPER1: D61.2, D64.4, JP252.2, JP253.1, JP61.2, JP64.1
- new net JUMPER10: D245.2, D248.4, JP245.2, JP248.1, JP272.2
- new net JUMPER2: D82.2, D85.4, JP253.2, JP265.1, JP82.2, JP85.1
- new net JUMPER3: D103.2, D106.4, JP103.2, JP106.1, JP265.2, JP266.1
- new net JUMPER4: D124.2, D127.4, JP124.2, JP127.1, JP266.2, JP267.1
- new net JUMPER5: D145.2, D148.4, JP145.2, JP148.1, JP267.2, JP268.1
- new net JUMPER6: D166.2, D169.4, JP166.2, JP169.1, JP268.2, JP269.1
- new net JUMPER7: D187.2, D190.4, JP187.2, JP190.1, JP269.2, JP270.1
- new net JUMPER8: D1.4, D208.2, JP1.1, JP208.2, JP270.2, JP271.1
- new net JUMPER9: D21.4, D229.2, JP21.1, JP229.2, JP271.2, JP272.1
- net DIO0: now also JP11.1
Routing:
- net JUMPER9: track 0.00 -> 315.6 mm, vias 0 -> 4
- net JUMPER8: track 0.00 -> 309.5 mm, vias 0 -> 2
- net JUMPER7: track 0.00 -> 308.5 mm, vias 0 -> 2
- net JUMPER5: track 0.00 -> 308.5 mm, vias 0 -> 2
- net JUMPER4: track 0.00 -> 308.5 mm, vias 0 -> 2
- net JUMPER3: track 0.00 -> 308.5 mm, vias 0 -> 2
- net JUMPER6: track 0.00 -> 308.5 mm, vias 0 -> 2
- net JUMPER1: track 0.00 -> 308.2 mm, vias 0 -> 2
- net JUMPER2: track 0.00 -> 308.2 mm, vias 0 -> 2
- net JUMPER0: track 0.00 -> 293.3 mm, vias 0 -> 2
- net DIO121: track 291.2 -> 0.00 mm, vias 2 -> 0
- net DIO109: track 290.1 -> 0.00 mm, vias 2 -> 0
- net N$68: track 289.0 -> 0.00 mm, vias 2 -> 0
- net DIO98: track 289.0 -> 0.00 mm, vias 2 -> 0
- net DIO76: track 289.0 -> 0.00 mm, vias 2 -> 0
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
Commit message: pushing final board changes
Parts:
- removed D21, D211, D263: WS2812B, SparkFun-LED:WS2812B
- removed JP21, JP211, JP263: JUMPER-SMT_2_NO_NO-SILK, SparkFun-Jumpers:SMT-JUMPER_2_NO_NO-SILK
- added U$1: (no value), unnamed#png (2):UNNAMED#PNG
- moved R5 20.7 mm to (294.0, 38.0), turned to 180 degrees
- moved R4 18.6 mm to (295.5, 27.7)
- moved R3 18.6 mm to (295.6, 30.3)
- moved C3 18.6 mm to (294.0, 39.5)
- moved J2 18.5 mm to (299.1, 29.0)
- moved J3 17.0 mm to (305.5, 47.0)
- moved R15 16.6 mm to (294.0, 41.0)
- moved R12 14.1 mm to (294.0, 36.5)
- moved C7 9.93 mm to (10.0, 12.9), turned to 180 degrees
- moved C8 7.83 mm to (13.0, 18.0), turned to 270 degrees
- moved C1 7.62 mm to (10.0, 14.7), turned to 180 degrees
- moved R14 5.82 mm to (299.0, 41.0), turned to 0 degrees
- moved R8 5.02 mm to (10.2, 21.8), turned to 0 degrees
- moved U3 4.22 mm to (10.0, 17.9), turned to 180 degrees
- moved C4 4.00 mm to (24.7, 21.4)
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Connections:
- removed net DIO127: D211.2, D263.4, JP211.2, JP263.1
- removed net N$138: D263.2, D264.4, JP263.2, JP264.1
- removed net N$2: D21.2, D211.4, JP21.2, JP211.1
- net GND: no longer D21.3, D211.3, D263.3
- net JUMPER9: now also D264.4, JP264.1; no longer D21.4, JP21.1
- net V_USB: no longer D21.1, D211.1, D263.1
Routing:
- net DIO127: track 31.8 -> 0.00 mm, vias 2 -> 0
- net N$2: track 17.4 -> 0.00 mm, vias 2 -> 0
- net N$138: track 16.8 -> 0.00 mm
- net V_USB: track 386.3 -> 371.0 mm, vias 224 -> 220
- net RING1: track 272.0 -> 283.8 mm, vias 0 -> 2
- net D-: track 314.8 -> 304.4 mm
- net D+: track 312.9 -> 302.7 mm
- net 3.3V: track 377.3 -> 368.3 mm, vias 7 -> 6
- net N$7: track 11.3 -> 4.48 mm
- net TIP: track 268.9 -> 274.1 mm, vias 0 -> 2
- net DIO0: track 216.0 -> 212.0 mm
- net JUMPER9: track 315.6 -> 311.8 mm, vias 4 -> 3
- net N$6: track 7.45 -> 4.60 mm
- net JUMPER8: track 309.5 -> 307.9 mm
- net GND: vias 34 -> 33
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Other:
- outline, holes or cut-outs redrawn

Commit message: updating files
Parts:
- removed FD1: FIDUCIALUFIDUCIAL, SparkFun-Aesthetics:FIDUCIAL-MICRO
Changed lines of the file:
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@@
 <attribute name="VALUE" x="10.03" y="15.507" size="0.6096" layer="27" font="vector" ratio="20" rot="R180" align="top-center"/>
 </element>
-<element name="FD1" library="SparkFun-Aesthetics" package="FIDUCIAL-MICRO" value="FIDUCIALUFIDUCIAL" x="313.75" y="195" smashed="yes"/>
 <element name="FD2" library="SparkFun-Aesthetics" package="FIDUCIAL-MICRO" value="FIDUCIALUFIDUCIAL" x="9.055" y="42.5" smashed="yes"/>
 <element name="FD4" library="SparkFun-Aesthetics" package="FIDUCIAL-MICRO" value="FIDUCIALUFIDUCIAL" x="2" y="11.5" smashed="yes" rot="R90"/>
