File: Hardware/13TB.sch (EAGLE design)
At the start: 578 parts, among them J2 USB Female Type C Connector, J3 AUDIO_JACK_TRRSSMD_RA, Q2 MBT3904DW1T1, U2 ESP-WROOM-32NARROW, U3 AP2112K-3.3V, U4 CP2102N, U5 ADMP401

Commit message: getting 4 boards polished
Parts:
- removed D10, D104, D105, D11, D12, D125, D126, D13, D14, D146, D147, D15, D16, D167, D168, D17, D18, D184, D185, D188, D189, D19, D20, D209, D210, D22, D230, D231, D246, D247, D262, D4, D40, D41, D42, D5, D6, D62, D63, D7, D8, D83, D84, D9: WS2812B, SparkFun-LED:WS2812B
- removed JP10, JP104, JP105, JP11, JP12, JP125, JP126, JP13, JP14, JP146, JP147, JP15, JP16, JP167, JP168, JP17, JP18, JP188, JP189, JP19, JP2, JP20, JP209, JP210, JP22, JP230, JP231, JP246, JP247, JP262, JP3, JP4, JP40, JP41, JP42, JP5, JP6, JP62, JP63, JP7, JP8, JP83, JP84, JP9: JUMPER-SMT_2_NO_NO-SILK, SparkFun-Jumpers:JUMPER-SMT_2_NO_NO-SILK
Connections:
- removed net DIO10: D20.DO, D22.DI, JP20.2, JP22.1
- removed net DIO104: D209.DO, D210.DI, JP209.2, JP210.1
- removed net DIO108: D208.DO, D209.DI, JP208.2, JP209.1
- removed net DIO11: D22.DO, D23.DI, JP22.2, JP23.1
- removed net DIO119: D230.DO, D231.DI, JP230.2, JP231.1
- removed net DIO130: D246.DO, D247.DI, JP246.2, JP247.1
- removed net DIO21: D41.DO, D42.DI, JP41.2, JP42.1
- removed net DIO3: D6.DO, D7.DI, JP6.2, JP7.1
- removed net DIO33: D63.DO, D64.DI, JP63.2, JP64.1
- removed net DIO4: D8.DO, D9.DI, JP8.2, JP9.1
- removed net DIO44: D83.DO, D84.DI, JP83.2, JP84.1
- removed net DIO5: D10.DO, D11.DI, JP10.2, JP11.1
- removed net DIO53: D103.DO, D104.DI, JP103.2, JP104.1
- removed net DIO6: D13.DO, D14.DI, JP13.2, JP14.1
- removed net DIO64: D125.DO, D126.DI, JP125.2, JP126.1
- removed net DIO7: D15.DO, D16.DI, JP15.2, JP16.1
- removed net DIO75: D145.DO, D146.DI, JP145.2, JP146.1
- removed net DIO8: D17.DO, D18.DI, JP17.2, JP18.1
- removed net DIO87: D167.DO, D168.DI, JP167.2, JP168.1
- removed net DIO9: D19.DO, D20.DI, JP19.2, JP20.1
- removed net DIO99: D189.DO, D190.DI, JP189.2, JP190.1
- removed net N$115: D229.DO, D230.DI, JP229.2, JP230.1
- removed net N$120: D2.DO, D3.DI, JP2.2, JP3.1
- removed net N$121: D4.DO, D5.DI, JP4.2, JP5.1
- removed net N$126: D245.DO, D246.DI, JP245.2, JP246.1
- removed net N$13: D3.DO, D4.DI, JP3.2, JP4.1
- removed net N$132: D262.DO, JP262.2
- removed net N$135: D11.DO, D12.DI, JP11.2, JP12.1
- removed net N$14: D5.DO, D6.DI, JP5.2, JP6.1
- removed net N$15: D10.DI, D9.DO, JP10.1, JP9.2
- removed net N$17: D7.DO, D8.DI, JP7.2, JP8.1
- removed net N$18: D16.DO, D17.DI, JP16.2, JP17.1
- removed net N$20: D14.DO, D15.DI, JP14.2, JP15.1
- removed net N$22: D18.DO, D19.DI, JP18.2, JP19.1
- removed net N$28: D104.DO, D105.DI, JP104.2, JP105.1
- removed net N$32: D42.DO, D43.DI, JP42.2, JP43.1
- removed net N$33: D40.DO, D41.DI, JP40.2, JP41.1
- removed net N$44: D62.DO, D63.DI, JP62.2, JP63.1
- removed net N$51: D82.DO, D83.DI, JP82.2, JP83.1
- removed net N$69: D124.DO, D125.DI, JP124.2, JP125.1
- removed net N$79: D146.DO, D147.DI, JP146.2, JP147.1
- removed net N$8: D12.DO, D13.DI, JP12.2, JP13.1
- removed net N$87: D166.DO, D167.DI, JP166.2, JP167.1
- removed net N$97: D188.DO, D189.DI, JP188.2, JP189.1
- net DIO0: now also D23.DI, JP23.1; no longer D2.DI, JP2.1
- net DIO109: now also D208.DO, JP208.2; no longer D210.DO, JP210.2
- net DIO121: now also D229.DO, JP229.2; no longer D231.DO, JP231.2
- net DIO138: no longer D262.DI, JP262.1
- net DIO20: now also D43.DI, JP43.1; no longer D40.DI, JP40.1
- net DIO32: now also D64.DI, JP64.1; no longer D62.DI, JP62.1
- net DIO54: now also D103.DO, JP103.2; no longer D105.DO, JP105.2
- net DIO76: now also D145.DO, JP145.2; no longer D147.DO, JP147.2
- net DIO96: now also D2.DO, D3.DI; no longer D184.DO, D185.DI
- net DIO98: now also D190.DI, JP190.1; no longer D188.DI, JP188.1
- net GND: no longer D10.VSS, D104.VSS, D105.VSS, D11.VSS, D12.VSS, D125.VSS, D126.VSS, D13.VSS, D14.VSS, D146.VSS, D147.VSS, D15.VSS, D16.VSS, D167.VSS, D168.VSS, D17.VSS, D18.VSS, D184.VSS, D185.VSS, D188.VSS, D189.VSS, D19.VSS, D20.VSS, D209.VSS, D210.VSS, D22.VSS, D230.VSS, D231.VSS, D246.VSS, D247.VSS, D262.VSS, D4.VSS, D40.VSS, D41.VSS, D42.VSS, D5.VSS, D6.VSS, D62.VSS, D63.VSS, D7.VSS, D8.VSS, D83.VSS, D84.VSS, D9.VSS
- net N$125: now also D245.DO, JP245.2; no longer D247.DO, JP247.2
- net N$54: now also D82.DO, JP82.2; no longer D84.DO, JP84.2
- net N$68: now also D124.DO, JP124.2; no longer D126.DO, JP126.2
- net N$89: now also D166.DO, JP166.2; no longer D168.DO, JP168.2
- net N$95: now also D3.DO; no longer D185.DO
- net N$96: now also D2.DI; no longer D184.DI
- net V_USB: no longer D10.VDD, D104.VDD, D105.VDD, D11.VDD, D12.VDD, D125.VDD, D126.VDD, D13.VDD, D14.VDD, D146.VDD, D147.VDD, D15.VDD, D16.VDD, D167.VDD, D168.VDD, D17.VDD, D18.VDD, D184.VDD, D185.VDD, D188.VDD, D189.VDD, D19.VDD, D20.VDD, D209.VDD, D210.VDD, D22.VDD, D230.VDD, D231.VDD, D246.VDD, D247.VDD, D262.VDD, D4.VDD, D40.VDD, D41.VDD, D42.VDD, D5.VDD, D6.VDD, D62.VDD, D63.VDD, D7.VDD, D8.VDD, D83.VDD, D84.VDD, D9.VDD

Commit message: polishing 13tb and 13r
Parts:
- removed D251, D252, D253, D31, D32, D33: WS2812B, SparkFun-LED:WS2812B
- removed JP251, JP252, JP253, JP31, JP32, JP33: JUMPER-SMT_2_NO_NO-SILK, SparkFun-Jumpers:JUMPER-SMT_2_NO_NO-SILK
Connections:
- removed net DIO133: D252.DO, D253.DI, JP252.2, JP253.1
- removed net DIO134: D253.DO, D254.DI, JP253.2, JP254.1
- removed net DIO16: D32.DO, D33.DI, JP32.2, JP33.1
- removed net DIO17: D33.DO, D34.DI, JP33.2, JP34.1
- removed net N$127: D251.DO, D252.DI, JP251.2, JP252.1
- removed net N$26: D31.DO, D32.DI, JP31.2, JP32.1
- net DIO132: now also D254.DI, JP254.1; no longer D251.DI, JP251.1
- net DIO15: now also D34.DI, JP34.1; no longer D31.DI, JP31.1
- net GND: no longer D251.VSS, D252.VSS, D253.VSS, D31.VSS, D32.VSS, D33.VSS
- net V_USB: no longer D251.VDD, D252.VDD, D253.VDD, D31.VDD, D32.VDD, D33.VDD

Commit message: final touches, polishing, jumpers, CAM on all boards
Parts:
- added JP11, JP252, JP253, JP265, JP266, JP267, JP268, JP269, JP270, JP271, JP272: JUMPER-SMT_2_NO_NO-SILK, SparkFun-Jumpers:JUMPER-SMT_2_NO_NO-SILK
Connections:
- removed net DIO109: D1.DI, D208.DO, JP1.1, JP208.2
- removed net DIO121: D21.DI, D229.DO, JP21.1, JP229.2
- removed net DIO20: D39.DO, D43.DI, JP39.2, JP43.1
- removed net DIO32: D61.DO, D64.DI, JP61.2, JP64.1
- removed net DIO54: D103.DO, D106.DI, JP103.2, JP106.1
- removed net DIO76: D145.DO, D148.DI, JP145.2, JP148.1
- removed net DIO98: D187.DO, D190.DI, JP187.2, JP190.1
- removed net N$125: D245.DO, D248.DI, JP245.2, JP248.1
- removed net N$54: D82.DO, D85.DI, JP82.2, JP85.1
- removed net N$68: D124.DO, D127.DI, JP124.2, JP127.1
- removed net N$89: D166.DO, D169.DI, JP166.2, JP169.1
- new net JUMPER0: D39.DO, D43.DI, JP11.2, JP252.1, JP39.2, JP43.1
- new net JUMPER1: D61.DO, D64.DI, JP252.2, JP253.1, JP61.2, JP64.1
- new net JUMPER10: D245.DO, D248.DI, JP245.2, JP248.1, JP272.2
- new net JUMPER2: D82.DO, D85.DI, JP253.2, JP265.1, JP82.2, JP85.1
- new net JUMPER3: D103.DO, D106.DI, JP103.2, JP106.1, JP265.2, JP266.1
- new net JUMPER4: D124.DO, D127.DI, JP124.2, JP127.1, JP266.2, JP267.1
- new net JUMPER5: D145.DO, D148.DI, JP145.2, JP148.1, JP267.2, JP268.1
- new net JUMPER6: D166.DO, D169.DI, JP166.2, JP169.1, JP268.2, JP269.1
- new net JUMPER7: D187.DO, D190.DI, JP187.2, JP190.1, JP269.2, JP270.1
- new net JUMPER8: D1.DI, D208.DO, JP1.1, JP208.2, JP270.2, JP271.1
- new net JUMPER9: D21.DI, D229.DO, JP21.1, JP229.2, JP271.2, JP272.1
- net DIO0: now also JP11.1

Commit message: pushing final board changes
Parts:
- removed D21, D211, D263: WS2812B, SparkFun-LED:WS2812B
- removed JP21, JP211, JP263: JUMPER-SMT_2_NO_NO-SILK, SparkFun-Jumpers:JUMPER-SMT_2_NO_NO-SILK
Connections:
- removed net DIO127: D211.DO, D263.DI, JP211.2, JP263.1
- removed net N$138: D263.DO, D264.DI, JP263.2, JP264.1
- removed net N$2: D21.DO, D211.DI, JP21.2, JP211.1
- net GND: no longer D21.VSS, D211.VSS, D263.VSS
- net JUMPER9: now also D264.DI, JP264.1; no longer D21.DI, JP21.1
- net V_USB: no longer D21.VDD, D211.VDD, D263.VDD

Commit message: updating files
Parts:
- removed FD1: FIDUCIALUFIDUCIAL, SparkFun-Aesthetics:FIDUCIALUFIDUCIAL
Changed lines of the file:
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@@
 <part name="GND3" library="SparkFun-Aesthetics" deviceset="GND" device=""/>
 <part name="C1" library="SparkFun-Capacitors" deviceset="10UF" device="-0603-6.3V-20%" value="10uF"/>
-<part name="FD1" library="SparkFun-Aesthetics" deviceset="FIDUCIAL" device="UFIDUCIAL"/>
 <part name="FD2" library="SparkFun-Aesthetics" deviceset="FIDUCIAL" device="UFIDUCIAL"/>
 <part name="FD4" library="SparkFun-Aesthetics" deviceset="FIDUCIAL" device="UFIDUCIAL"/>
@@
 <attribute name="VALUE" x="110.744" y="231.521" size="1.778" layer="96" font="vector"/>
 </instance>
-<instance part="FD1" gate="G$1" x="429.26" y="33.02" smashed="yes"/>
 <instance part="FD2" gate="G$1" x="426.72" y="33.02" smashed="yes"/>
 <instance part="FD4" gate="G$1" x="429.26" y="30.48" smashed="yes"/>
