File: Hardware/15NR.brd (EAGLE design)
At the start: 360.5 x 217.5 mm, 669 parts, among them J2 USB Female Type C Connector, J3 AUDIO_JACK_TRRSSMD_RA, Q2 MBT3904DW1T1, U2 ESP-WROOM-32NARROW, U3 AP2112K-3.3V, U4 CP2102N, U5 ADMP401

Commit message: getting 4 boards polished
Parts:
- removed D11, D12, D13: WS2812B, SparkFun-LED:WS2812B
- removed JP11, JP12, JP13: JUMPER-SMT_2_NO_NO-SILK, SparkFun-Jumpers:SMT-JUMPER_2_NO_NO-SILK
- moved D256 51.1 mm to (208.2, 13.2)
- moved D257 51.1 mm to (223.2, 13.2)
- moved JP256 51.1 mm to (208.2, 13.2)
- moved JP257 51.1 mm to (223.2, 13.2)
- moved H1 38.6 mm to (196.0, 213.0)
- moved H2 33.0 mm to (160.5, 13.2)
- moved D1 8.13 mm to (313.2, 208.2)
- moved D10 8.13 mm to (148.2, 208.2)
- moved D100 8.13 mm to (238.2, 148.2)
- moved D101 8.13 mm to (253.2, 148.2)
- moved D102 8.13 mm to (268.2, 148.2)
- moved D103 8.13 mm to (283.2, 148.2)
- moved D104 8.13 mm to (298.2, 148.2)
- moved D105 8.13 mm to (313.2, 148.2)
- moved D106 8.13 mm to (13.2, 133.2)
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Connections:
- removed net DIO5: D10.2, D11.4, JP10.2, JP11.1
- removed net DIO6: D13.2, D14.4, JP13.2, JP14.1
- removed net N$135: D11.2, D12.4, JP11.2, JP12.1
- net GND: no longer D11.3, D12.3, D13.3
- net N$8: now also D10.2, D14.4, JP10.2, JP14.1; no longer D12.2, D13.4, JP12.2, JP13.1
- net V_USB: no longer D11.1, D12.1, D13.1
Routing:
- net DIO135: track 15.6 -> 62.9 mm
- net DIO136: track 63.6 -> 16.8 mm
- net N$8: track 16.8 -> 61.8 mm
- net N$135: track 16.8 -> 0.00 mm
- net DIO6: track 16.8 -> 0.00 mm
- net DIO5: track 16.8 -> 0.00 mm
- net DIO0: track 233.2 -> 246.2 mm
- net TIP: track 314.1 -> 323.7 mm
- net N$170: track 46.8 -> 38.2 mm
- net D-: track 379.6 -> 387.7 mm
- net V_USB: track 550.9 -> 558.7 mm, vias 317 -> 314
- net D+: track 377.7 -> 385.4 mm
- net RING1: track 316.9 -> 324.6 mm
- net 3.3V: track 435.5 -> 436.2 mm
Other:
- board size 360.5 x 217.5 mm -> 366.5 x 220.5 mm
- board text added: "15NR"
- board text removed: "15R"

Commit message: final touches, polishing, jumpers, CAM on all boards
Parts:
- added JP11, JP12, JP13, JP249, JP312, JP313, JP314, JP316, JP317, JP318, JP319, JP320, JP321: JUMPER-SMT_2_NO_NO-SILK, SparkFun-Jumpers:SMT-JUMPER_2_NO_NO-SILK
Connections:
- removed net DIO10: D211.2, D22.4, JP211.2, JP22.1
- removed net DIO109: D21.4, D210.2, JP1.1, JP210.2
- removed net DIO152: D248.4, D308.2, JP248.1, JP308.2
- removed net DIO99: D189.2, D190.4, JP189.2, JP190.1
- removed net N$128: D247.2, D250.4, JP247.2, JP250.1
- removed net N$139: D264.2, D43.4, JP264.2, JP43.1
- removed net N$140: D266.2, D64.4, JP266.2, JP64.1
- removed net N$144: D106.4, D270.2, JP106.1, JP270.2
- removed net N$147: D148.4, D274.2, JP148.1, JP274.2
- removed net N$172: D231.2, D309.4, JP231.2, JP309.1
- removed net N$54: D84.2, D85.4, JP84.2, JP85.1
- removed net N$68: D127.4, D272.2, JP127.1, JP272.2
- removed net N$89: D168.2, D169.4, JP168.2, JP169.1
- new net JUMPER0: D211.2, D22.4, JP11.2, JP12.1, JP211.2, JP22.1
- new net JUMPER1: D264.2, D43.4, JP12.2, JP13.1, JP264.2, JP43.1
- new net JUMPER10: D248.4, D308.2, JP248.1, JP308.2, JP319.2, JP320.1
- new net JUMPER11: D231.2, D309.4, JP231.2, JP309.1, JP320.2, JP321.1
- new net JUMPER12: D247.2, D250.4, JP247.2, JP250.1, JP321.2
- new net JUMPER2: D266.2, D64.4, JP13.2, JP249.1, JP266.2, JP64.1
- new net JUMPER3: D84.2, D85.4, JP249.2, JP312.1, JP84.2, JP85.1
- new net JUMPER4: D106.4, D270.2, JP106.1, JP270.2, JP312.2, JP313.1
- new net JUMPER5: D127.4, D272.2, JP127.1, JP272.2, JP313.2, JP314.1
- new net JUMPER6: D148.4, D274.2, JP148.1, JP274.2, JP314.2, JP316.1
- new net JUMPER7: D168.2, D169.4, JP168.2, JP169.1, JP316.2, JP317.1
- new net JUMPER8: D189.2, D190.4, JP189.2, JP190.1, JP317.2, JP318.1
- new net JUMPER9: D21.4, D210.2, JP1.1, JP210.2, JP318.2, JP319.1
- net DIO0: now also JP11.1
Routing:
- net JUMPER11: track 0.00 -> 380.4 mm, vias 0 -> 4
- net JUMPER9: track 0.00 -> 371.3 mm, vias 0 -> 2
- net JUMPER1: track 0.00 -> 370.1 mm, vias 0 -> 2
- net JUMPER2: track 0.00 -> 370.0 mm, vias 0 -> 2
- net JUMPER7: track 0.00 -> 369.0 mm, vias 0 -> 2
- net JUMPER8: track 0.00 -> 369.0 mm, vias 0 -> 2
- net JUMPER4: track 0.00 -> 368.9 mm, vias 0 -> 2
- net JUMPER3: track 0.00 -> 368.7 mm, vias 0 -> 2
- net JUMPER10: track 0.00 -> 368.2 mm, vias 0 -> 2
- net JUMPER6: track 0.00 -> 368.1 mm, vias 0 -> 2
- net JUMPER5: track 0.00 -> 367.7 mm, vias 0 -> 2
- net JUMPER0: track 0.00 -> 359.3 mm, vias 0 -> 2
- net DIO109: track 351.4 -> 0.00 mm, vias 2 -> 0
- net N$139: track 350.3 -> 0.00 mm, vias 2 -> 0
- net N$140: track 350.1 -> 0.00 mm, vias 2 -> 0
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
Commit message: pushing final board changes
Parts:
- added U$1: (no value), unnamed#png (2):UNNAMED#PNG
- moved C3 18.5 mm to (350.2, 44.6)
- moved R15 18.5 mm to (352.8, 44.6)
- moved R3 18.5 mm to (356.6, 30.3)
- moved R5 18.5 mm to (350.2, 46.5)
- moved C2 18.5 mm to (350.2, 50.3)
- moved R12 18.5 mm to (350.2, 42.7)
- moved R14 18.5 mm to (352.8, 50.3)
- moved R6 18.5 mm to (350.2, 52.2)
- moved R4 18.5 mm to (356.6, 27.8)
- moved R7 18.5 mm to (350.2, 48.4)
- moved J2 18.5 mm to (360.0, 29.0)
- moved J3 18.4 mm to (366.5, 47.0)
- moved H2 5.75 mm to (160.5, 7.50)
- moved C1 4.00 mm to (11.8, 22.8)
- moved C4 4.00 mm to (27.5, 19.0)
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Routing:
- net 3.3V: track 436.2 -> 458.1 mm
- net D-: track 387.7 -> 374.5 mm
- net D+: track 385.4 -> 373.4 mm
- net RING1: track 324.6 -> 332.8 mm, vias 0 -> 2
- net V_USB: track 567.2 -> 559.1 mm
- net TIP: track 323.7 -> 331.0 mm, vias 0 -> 2
- net N$170: track 38.2 -> 31.9 mm
- net DIO0: track 256.4 -> 253.3 mm
- net DIO135: track 62.9 -> 60.6 mm
- net JUMPER11: track 380.4 -> 378.3 mm
- net DIO110: vias 0 -> 2
Other:
- outline, holes or cut-outs redrawn

Commit message: updating files
Parts:
- removed FD1: FIDUCIALUFIDUCIAL, SparkFun-Aesthetics:FIDUCIAL-MICRO
Changed lines of the file:
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@@
 <attribute name="VALUE" x="10.988" y="22.8" size="0.6096" layer="27" font="vector" ratio="20" rot="R270" align="top-center"/>
 </element>
-<element name="FD1" library="SparkFun-Aesthetics" package="FIDUCIAL-MICRO" value="FIDUCIALUFIDUCIAL" x="313.75" y="210" smashed="yes"/>
 <element name="FD2" library="SparkFun-Aesthetics" package="FIDUCIAL-MICRO" value="FIDUCIALUFIDUCIAL" x="9.5" y="48.25" smashed="yes"/>
 <element name="FD4" library="SparkFun-Aesthetics" package="FIDUCIAL-MICRO" value="FIDUCIALUFIDUCIAL" x="1" y="2" smashed="yes"/>
