File: Hardware/15NR.sch (EAGLE design)
At the start: 668 parts, among them J2 USB Female Type C Connector, J3 AUDIO_JACK_TRRSSMD_RA, Q2 MBT3904DW1T1, U2 ESP-WROOM-32NARROW, U3 AP2112K-3.3V, U4 CP2102N, U5 ADMP401

Commit message: getting 4 boards polished
Parts:
- removed D11, D12, D13: WS2812B, SparkFun-LED:WS2812B
- removed JP11, JP12, JP13: JUMPER-SMT_2_NO_NO-SILK, SparkFun-Jumpers:JUMPER-SMT_2_NO_NO-SILK
Connections:
- removed net DIO5: D10.DO, D11.DI, JP10.2, JP11.1
- removed net DIO6: D13.DO, D14.DI, JP13.2, JP14.1
- removed net N$135: D11.DO, D12.DI, JP11.2, JP12.1
- net GND: no longer D11.VSS, D12.VSS, D13.VSS
- net N$8: now also D10.DO, D14.DI, JP10.2, JP14.1; no longer D12.DO, D13.DI, JP12.2, JP13.1
- net V_USB: no longer D11.VDD, D12.VDD, D13.VDD

Commit message: final touches, polishing, jumpers, CAM on all boards
Parts:
- added JP11, JP12, JP13, JP249, JP312, JP313, JP314, JP316, JP317, JP318, JP319, JP320, JP321: JUMPER-SMT_2_NO_NO-SILK, SparkFun-Jumpers:JUMPER-SMT_2_NO_NO-SILK
Connections:
- removed net DIO10: D211.DO, D22.DI, JP211.2, JP22.1
- removed net DIO109: D21.DI, D210.DO, JP1.1, JP210.2
- removed net DIO152: D248.DI, D308.DO, JP248.1, JP308.2
- removed net DIO99: D189.DO, D190.DI, JP189.2, JP190.1
- removed net N$128: D247.DO, D250.DI, JP247.2, JP250.1
- removed net N$139: D264.DO, D43.DI, JP264.2, JP43.1
- removed net N$140: D266.DO, D64.DI, JP266.2, JP64.1
- removed net N$144: D106.DI, D270.DO, JP106.1, JP270.2
- removed net N$147: D148.DI, D274.DO, JP148.1, JP274.2
- removed net N$172: D231.DO, D309.DI, JP231.2, JP309.1
- removed net N$54: D84.DO, D85.DI, JP84.2, JP85.1
- removed net N$68: D127.DI, D272.DO, JP127.1, JP272.2
- removed net N$89: D168.DO, D169.DI, JP168.2, JP169.1
- new net JUMPER0: D211.DO, D22.DI, JP11.2, JP12.1, JP211.2, JP22.1
- new net JUMPER1: D264.DO, D43.DI, JP12.2, JP13.1, JP264.2, JP43.1
- new net JUMPER10: D248.DI, D308.DO, JP248.1, JP308.2, JP319.2, JP320.1
- new net JUMPER11: D231.DO, D309.DI, JP231.2, JP309.1, JP320.2, JP321.1
- new net JUMPER12: D247.DO, D250.DI, JP247.2, JP250.1, JP321.2
- new net JUMPER2: D266.DO, D64.DI, JP13.2, JP249.1, JP266.2, JP64.1
- new net JUMPER3: D84.DO, D85.DI, JP249.2, JP312.1, JP84.2, JP85.1
- new net JUMPER4: D106.DI, D270.DO, JP106.1, JP270.2, JP312.2, JP313.1
- new net JUMPER5: D127.DI, D272.DO, JP127.1, JP272.2, JP313.2, JP314.1
- new net JUMPER6: D148.DI, D274.DO, JP148.1, JP274.2, JP314.2, JP316.1
- new net JUMPER7: D168.DO, D169.DI, JP168.2, JP169.1, JP316.2, JP317.1
- new net JUMPER8: D189.DO, D190.DI, JP189.2, JP190.1, JP317.2, JP318.1
- new net JUMPER9: D21.DI, D210.DO, JP1.1, JP210.2, JP318.2, JP319.1
- net DIO0: now also JP11.1

Commit message: updating files
Parts:
- removed FD1: FIDUCIALUFIDUCIAL, SparkFun-Aesthetics:FIDUCIALUFIDUCIAL
Changed lines of the file:
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@@
 <?xml version="1.0" encoding="utf-8"?>
 <!DOCTYPE eagle SYSTEM "eagle.dtd">
-<eagle version="9.5.2">
+<eagle version="9.6.0">
 <drawing>
 <settings>
@@
 <part name="GND3" library="SparkFun-Aesthetics" deviceset="GND" device=""/>
 <part name="C1" library="SparkFun-Capacitors" deviceset="10UF" device="-0603-6.3V-20%" value="10uF"/>
-<part name="FD1" library="SparkFun-Aesthetics" deviceset="FIDUCIAL" device="UFIDUCIAL"/>
 <part name="FD2" library="SparkFun-Aesthetics" deviceset="FIDUCIAL" device="UFIDUCIAL"/>
 <part name="FD4" library="SparkFun-Aesthetics" deviceset="FIDUCIAL" device="UFIDUCIAL"/>
@@
 <attribute name="VALUE" x="110.744" y="231.521" size="1.778" layer="96" font="vector"/>
 </instance>
-<instance part="FD1" gate="G$1" x="429.26" y="33.02" smashed="yes"/>
 <instance part="FD2" gate="G$1" x="426.72" y="33.02" smashed="yes"/>
 <instance part="FD4" gate="G$1" x="429.26" y="30.48" smashed="yes"/>
