File: Hardware/15R.brd (EAGLE design)
At the start: 360.5 x 217.5 mm, 669 parts, among them J2 USB Female Type C Connector, J3 AUDIO_JACK_TRRSSMD_RA, Q2 MBT3904DW1T1, U2 ESP-WROOM-32NARROW, U3 AP2112K-3.3V, U4 CP2102N, U5 ADMP401

Commit message: getting 4 boards polished
Parts:
- removed D11, D12, D13: WS2812B, SparkFun-LED:WS2812B
- removed JP11, JP12, JP13: JUMPER-SMT_2_NO_NO-SILK, SparkFun-Jumpers:SMT-JUMPER_2_NO_NO-SILK
- moved D256 47.0 mm to (204.4, 11.2)
- moved D257 47.0 mm to (219.4, 11.2)
- moved JP256 47.0 mm to (204.4, 11.2)
- moved JP257 47.0 mm to (219.4, 11.2)
- moved H1 35.5 mm to (193.0, 210.0)
- moved H2 35.5 mm to (157.5, 7.50)
- moved R12 12.8 mm to (344.8, 36.9), turned to 90 degrees
- moved C3 11.2 mm to (346.7, 36.9), turned to 270 degrees
- moved R6 11.0 mm to (354.3, 36.9), turned to 90 degrees
- moved R5 10.2 mm to (348.6, 36.9), turned to 90 degrees
- moved C2 10.0 mm to (352.4, 36.9), turned to 90 degrees
- moved R7 9.74 mm to (350.5, 36.9), turned to 270 degrees
- moved R15 8.32 mm to (346.7, 34.4), turned to 180 degrees
- moved R14 6.62 mm to (352.4, 34.4), turned to 180 degrees
- moved C7 4.47 mm to (7.45, 19.0)
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Connections:
- removed net DIO5: D10.2, D11.4, JP10.2, JP11.1
- removed net DIO6: D13.2, D14.4, JP13.2, JP14.1
- removed net N$135: D11.2, D12.4, JP11.2, JP12.1
- net GND: no longer D11.3, D12.3, D13.3
- net N$8: now also D10.2, D14.4, JP10.2, JP14.1; no longer D12.2, D13.4, JP12.2, JP13.1
- net V_USB: no longer D11.1, D12.1, D13.1
Routing:
- net DIO135: track 15.6 -> 62.9 mm
- net DIO136: track 63.6 -> 16.8 mm
- net N$8: track 16.8 -> 61.8 mm
- net N$135: track 16.8 -> 0.00 mm
- net DIO6: track 16.8 -> 0.00 mm
- net DIO5: track 16.8 -> 0.00 mm
- net RING1: track 316.9 -> 330.3 mm
- net 3.3V: track 435.5 -> 446.9 mm
- net N$6: track 5.87 -> 14.2 mm
- net TIP: track 314.1 -> 320.1 mm
- net DIO0: track 233.2 -> 237.7 mm
- net D-: track 379.6 -> 382.9 mm
- net D+: track 377.7 -> 380.8 mm
- net V_USB: track 550.9 -> 548.9 mm, vias 317 -> 314
- net N$170: track 46.8 -> 45.5 mm
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Other:
- outline, holes or cut-outs redrawn

Commit message: final touches, polishing, jumpers, CAM on all boards
Parts:
- added JP11, JP12, JP13, JP249, JP312, JP313, JP314, JP316, JP317, JP318, JP319, JP320, JP321: JUMPER-SMT_2_NO_NO-SILK, SparkFun-Jumpers:SMT-JUMPER_2_NO_NO-SILK
- moved FD2 3.00 mm to (2.62, 46.2)
Connections:
- removed net DIO10: D211.2, D22.4, JP211.2, JP22.1
- removed net DIO109: D21.4, D210.2, JP1.1, JP210.2
- removed net DIO152: D248.4, D308.2, JP248.1, JP308.2
- removed net DIO99: D189.2, D190.4, JP189.2, JP190.1
- removed net N$128: D247.2, D250.4, JP247.2, JP250.1
- removed net N$139: D264.2, D43.4, JP264.2, JP43.1
- removed net N$140: D266.2, D64.4, JP266.2, JP64.1
- removed net N$144: D106.4, D270.2, JP106.1, JP270.2
- removed net N$147: D148.4, D274.2, JP148.1, JP274.2
- removed net N$172: D231.2, D309.4, JP231.2, JP309.1
- removed net N$54: D84.2, D85.4, JP84.2, JP85.1
- removed net N$68: D127.4, D272.2, JP127.1, JP272.2
- removed net N$89: D168.2, D169.4, JP168.2, JP169.1
- new net JUMPER0: D211.2, D22.4, JP11.2, JP12.1, JP211.2, JP22.1
- new net JUMPER1: D264.2, D43.4, JP12.2, JP13.1, JP264.2, JP43.1
- new net JUMPER10: D248.4, D308.2, JP248.1, JP308.2, JP319.2, JP320.1
- new net JUMPER11: D231.2, D309.4, JP231.2, JP309.1, JP320.2, JP321.1
- new net JUMPER12: D247.2, D250.4, JP247.2, JP250.1, JP321.2
- new net JUMPER2: D266.2, D64.4, JP13.2, JP249.1, JP266.2, JP64.1
- new net JUMPER3: D84.2, D85.4, JP249.2, JP312.1, JP84.2, JP85.1
- new net JUMPER4: D106.4, D270.2, JP106.1, JP270.2, JP312.2, JP313.1
- new net JUMPER5: D127.4, D272.2, JP127.1, JP272.2, JP313.2, JP314.1
- new net JUMPER6: D148.4, D274.2, JP148.1, JP274.2, JP314.2, JP316.1
- new net JUMPER7: D168.2, D169.4, JP168.2, JP169.1, JP316.2, JP317.1
- new net JUMPER8: D189.2, D190.4, JP189.2, JP190.1, JP317.2, JP318.1
- new net JUMPER9: D21.4, D210.2, JP1.1, JP210.2, JP318.2, JP319.1
- net DIO0: now also JP11.1
Routing:
- net JUMPER11: track 0.00 -> 374.3 mm, vias 0 -> 3
- net JUMPER9: track 0.00 -> 367.4 mm, vias 0 -> 2
- net JUMPER1: track 0.00 -> 366.3 mm, vias 0 -> 2
- net JUMPER2: track 0.00 -> 366.1 mm, vias 0 -> 2
- net JUMPER7: track 0.00 -> 365.1 mm, vias 0 -> 2
- net JUMPER8: track 0.00 -> 365.1 mm, vias 0 -> 2
- net JUMPER4: track 0.00 -> 365.1 mm, vias 0 -> 2
- net JUMPER3: track 0.00 -> 364.9 mm, vias 0 -> 2
- net JUMPER10: track 0.00 -> 364.3 mm, vias 0 -> 2
- net JUMPER6: track 0.00 -> 364.2 mm, vias 0 -> 2
- net JUMPER5: track 0.00 -> 363.8 mm, vias 0 -> 2
- net JUMPER0: track 0.00 -> 355.4 mm, vias 0 -> 2
- net DIO109: track 351.4 -> 0.00 mm, vias 2 -> 0
- net N$139: track 350.3 -> 0.00 mm, vias 2 -> 0
- net N$140: track 350.1 -> 0.00 mm, vias 2 -> 0
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
Commit message: pushing final board changes
Parts:
- removed D309, D310, D311: WS2812B, SparkFun-LED:WS2812B
- removed JP309, JP310, JP311: JUMPER-SMT_2_NO_NO-SILK, SparkFun-Jumpers:SMT-JUMPER_2_NO_NO-SILK
- added U$1: (no value), unnamed#png (2):UNNAMED#PNG
- moved R4 18.8 mm to (350.0, 27.5)
- moved J2 18.5 mm to (354.0, 29.0)
- moved J3 18.4 mm to (360.5, 47.0)
- moved R3 18.3 mm to (350.0, 30.5)
- moved R12 10.6 mm to (355.2, 38.6), turned to 270 degrees
- moved R15 9.55 mm to (353.2, 41.4)
- moved R6 8.72 mm to (345.7, 38.6), turned to 270 degrees
- moved R14 8.26 mm to (347.6, 41.1), turned to 0 degrees
- moved C3 6.89 mm to (353.3, 38.6), turned to 90 degrees
- moved C2 5.04 mm to (347.6, 38.6), turned to 270 degrees
- moved C4 4.00 mm to (22.5, 19.0)
- moved C5 4.00 mm to (19.0, 19.0)
- moved C6 4.00 mm to (22.6, 21.7)
- moved C9 4.00 mm to (15.9, 21.7)
- moved Q2 4.00 mm to (23.5, 8.45)
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Connections:
- removed net DIO143: D309.2, D310.4, JP309.2, JP310.1
- removed net N$170: D310.2, D311.4, JP310.2, JP311.1
- removed net N$173: D311.2, D315.4, JP311.2, JP315.1
- net GND: no longer D309.3, D310.3, D311.3
- net JUMPER11: now also D315.4, JP315.1; no longer D309.4, JP309.1
- net V_USB: no longer D309.1, D310.1, D311.1
Routing:
- net N$170: track 45.5 -> 0.00 mm, vias 2 -> 0
- net V_USB: track 548.9 -> 518.6 mm, vias 314 -> 312
- net DIO143: track 17.5 -> 0.00 mm, vias 2 -> 0
- net N$173: track 16.8 -> 0.00 mm
- net D-: track 382.9 -> 368.4 mm
- net D+: track 380.8 -> 366.7 mm
- net RING1: track 330.3 -> 319.2 mm, vias 0 -> 2
- net N$6: track 14.2 -> 7.32 mm
- net TIP: track 320.1 -> 324.8 mm, vias 0 -> 2
- net JUMPER11: track 374.3 -> 378.8 mm
- net DIO0: track 247.4 -> 244.1 mm
- net 3.3V: track 446.9 -> 449.8 mm
- net N$7: track 12.5 -> 13.8 mm
- net N$4: track 2.22 -> 3.10 mm
- net N$3: track 2.32 -> 3.10 mm
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Other:
- outline, holes or cut-outs redrawn

Commit message: updating files
Parts:
- removed FD1: FIDUCIALUFIDUCIAL, SparkFun-Aesthetics:FIDUCIAL-MICRO
Changed lines of the file:
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@@
 <attribute name="VALUE" x="8.438" y="19" size="0.6096" layer="27" font="vector" ratio="20" rot="R270" align="top-center"/>
 </element>
-<element name="FD1" library="SparkFun-Aesthetics" package="FIDUCIAL-MICRO" value="FIDUCIALUFIDUCIAL" x="313.75" y="210" smashed="yes"/>
 <element name="FD2" library="SparkFun-Aesthetics" package="FIDUCIAL-MICRO" value="FIDUCIALUFIDUCIAL" x="2.625" y="46.25" smashed="yes"/>
 <element name="FD4" library="SparkFun-Aesthetics" package="FIDUCIAL-MICRO" value="FIDUCIALUFIDUCIAL" x="1" y="2" smashed="yes"/>
