File: Hardware/15TB.brd (EAGLE design)
At the start: 360.5 x 217.5 mm, 669 parts, among them J2 USB Female Type C Connector, J3 AUDIO_JACK_TRRSSMD_RA, Q2 MBT3904DW1T1, U2 ESP-WROOM-32NARROW, U3 AP2112K-3.3V, U4 CP2102N, U5 ADMP401

Commit message: updating 15TB outer dimensions, still need to re-place holes
Parts:
- moved H5 10.6 mm to (335.5, 202.5)
- moved H6 5.59 mm to (7.50, 204.4)
Other:
- board size 360.5 x 217.5 mm -> 351.6 x 211.9 mm
Changed lines of the file:
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@@
 <setting verticaltext="up"/>
 </settings>
-<grid distance="7.5" unitdist="mm" unit="mm" style="lines" multiple="1" display="yes" altdistance="0.05" altunitdist="mm" altunit="mm"/>
+<grid distance="7.5" unitdist="mm" unit="mm" style="lines" multiple="1" display="yes" altdistance="0.5" altunitdist="mm" altunit="mm"/>
 <layers>
 <layer number="1" name="Top" color="4" fill="1" visible="yes" active="yes"/>
@@
 <board>
 <plain>
-<wire x1="350.5" y1="0" x2="350.5" y2="23" width="0.2032" layer="20"/>
-<wire x1="350.5" y1="23" x2="360.5" y2="23" width="0.2032" layer="20"/>
-<wire x1="360.5" y1="23" x2="360.5" y2="53" width="0.2032" layer="20"/>
-<wire x1="360.5" y1="53" x2="350.5" y2="53" width="0.2032" layer="20"/>
-<wire x1="350.5" y1="53" x2="350.5" y2="217.5" width="0.2032" layer="20"/>
-<wire x1="350.5" y1="217.5" x2="0" y2="217.5" width="0.2032" layer="20"/>
-<wire x1="0" y1="217.5" x2="0" y2="0" width="0.2032" layer="20"/>
+<wire x1="341.61" y1="0" x2="341.61" y2="23" width="0.2032" layer="20"/>
+<wire x1="341.61" y1="23" x2="351.61" y2="23" width="0.2032" layer="20"/>
+<wire x1="351.61" y1="23" x2="351.61" y2="53" width="0.2032" layer="20"/>
+<wire x1="351.61" y1="53" x2="341.61" y2="53" width="0.2032" layer="20"/>
+<wire x1="341.61" y1="53" x2="341.61" y2="211.91" width="0.2032" layer="20"/>
+<wire x1="341.61" y1="211.91" x2="0" y2="211.91" width="0.2032" layer="20"/>
+<wire x1="0" y1="211.91" x2="0" y2="0" width="0.2032" layer="20"/>
 <wire x1="0" y1="0" x2="50.063" y2="0" width="0.2032" layer="20"/>
 <wire x1="50.063" y1="0" x2="50.063" y2="19.32" width="0.2032" layer="20"/>
 <wire x1="50.063" y1="19.32" x2="56.032" y2="19.32" width="0.2032" layer="20"/>
 <wire x1="56.032" y1="19.32" x2="56.032" y2="0" width="0.2032" layer="20"/>
-<wire x1="56.032" y1="0" x2="350.5" y2="0" width="0.2032" layer="20"/>
+<wire x1="56.032" y1="0" x2="341.61" y2="0" width="0.2032" layer="20"/>
 <text x="359.869" y="48.713" size="1.27" layer="16" font="vector" ratio="15" rot="SMR270">v11</text>
 <text x="359.055" y="38.991" size="1.27" layer="21" font="vector" ratio="15" rot="R270">15R</text>
@@
 <attribute name="VALUE" x="193" y="5.468" size="0.6096" layer="27" font="vector" ratio="20" align="top-center"/>
 </element>
-<element name="H5" library="SparkFun-Hardware" package="STAND-OFF" value="STAND-OFF" x="343" y="210" smashed="yes">
-<attribute name="NAME" x="343" y="212.032" size="0.6096" layer="25" font="vector" ratio="20" align="bottom-center"/>
-<attribute name="VALUE" x="343" y="207.968" size="0.6096" layer="27" font="vector" ratio="20" align="top-center"/>
-</element>
-<element name="H6" library="SparkFun-Hardware" package="STAND-OFF" value="STAND-OFF" x="7.5" y="210" smashed="yes">
-<attribute name="NAME" x="7.5" y="212.032" size="0.6096" layer="25" font="vector" ratio="20" align="bottom-center"/>
-<attribute name="VALUE" x="7.5" y="207.968" size="0.6096" layer="27" font="vector" ratio="20" align="top-center"/>
+<element name="H5" library="SparkFun-Hardware" package="STAND-OFF" value="STAND-OFF" x="335.5" y="202.5" smashed="yes">
+<attribute name="NAME" x="335.5" y="204.532" size="0.6096" layer="25" font="vector" ratio="20" align="bottom-center"/>
+<attribute name="VALUE" x="335.5" y="200.468" size="0.6096" layer="27" font="vector" ratio="20" align="top-center"/>
+</element>
+<element name="H6" library="SparkFun-Hardware" package="STAND-OFF" value="STAND-OFF" x="7.5" y="204.41" smashed="yes">
+<attribute name="NAME" x="7.5" y="206.442" size="0.6096" layer="25" font="vector" ratio="20" align="bottom-center"/>
+<attribute name="VALUE" x="7.5" y="202.378" size="0.6096" layer="27" font="vector" ratio="20" align="top-center"/>
 </element>
 <element name="C7" library="SparkFun-Capacitors" package="0603" value="1.0uF" x="3.75" y="16.5" smashed="yes" rot="R270">
@@
 <polygon width="0.2032" layer="1">
 <vertex x="0" y="0"/>
-<vertex x="0" y="217.5"/>
-<vertex x="350.5" y="217.5"/>
-<vertex x="350.5" y="53"/>
-<vertex x="360.5" y="53"/>
-<vertex x="360.5" y="23"/>
-<vertex x="350.5" y="23"/>
-<vertex x="350.5" y="0"/>
+<vertex x="0" y="211.91"/>
+<vertex x="341.61" y="211.91"/>
+<vertex x="341.61" y="53"/>
+<vertex x="351.61" y="53"/>
+<vertex x="351.61" y="23"/>
+<vertex x="341.61" y="23"/>
+<vertex x="341.61" y="0"/>
 </polygon>
 <wire x1="12.58" y1="7.1" x2="13.88" y2="7.1" width="0.3048" layer="1"/>
@@
 <contactref element="D261" pad="1"/>
 <polygon width="0.2032" layer="16">
-<vertex x="350.5" y="0"/>
-<vertex x="350.5" y="23"/>
-<vertex x="360.5" y="23"/>
-<vertex x="360.5" y="53"/>
-<vertex x="350.5" y="53"/>
-<vertex x="350.5" y="217.5"/>
-<vertex x="0" y="217.5"/>
+<vertex x="341.61" y="0"/>
+<vertex x="341.61" y="23"/>
+<vertex x="351.61" y="23"/>
+<vertex x="351.61" y="53"/>
+<vertex x="341.61" y="53"/>
+<vertex x="341.61" y="211.91"/>
+<vertex x="0" y="211.91"/>
 <vertex x="0" y="23.5"/>
 <vertex x="56.5" y="23.5"/>

Commit message: getting 4 boards polished
Parts:
- removed D11, D12, D13, D168, D189, D210, D211, D231, D247, D261, D264, D266, D270, D272, D274, D308, D84: WS2812B, SparkFun-LED:WS2812B
- removed JP11, JP12, JP13, JP168, JP189, JP210, JP211, JP231, JP247, JP261, JP264, JP266, JP270, JP272, JP274, JP308, JP84: JUMPER-SMT_2_NO_NO-SILK, SparkFun-Jumpers:SMT-JUMPER_2_NO_NO-SILK
- moved D256 50.8 mm to (208.3, 7.50)
- moved D257 50.8 mm to (223.3, 7.50)
- moved JP256 50.8 mm to (208.3, 7.50)
- moved JP257 50.8 mm to (223.3, 7.50)
- moved D255 49.6 mm to (193.3, 7.50)
- moved JP255 49.6 mm to (193.3, 7.50)
- moved H2 40.2 mm to (152.8, 7.75)
- moved H1 31.8 mm to (188.8, 204.2)
- moved H3 9.14 mm to (333.9, 7.50)
- moved C2 9.00 mm to (334.7, 31.8)
- moved C3 9.00 mm to (334.7, 26.1)
- moved J2 9.00 mm to (344.3, 47.4)
- moved J3 9.00 mm to (351.2, 28.6)
- moved R12 9.00 mm to (334.7, 24.2)
- moved R14 9.00 mm to (337.3, 31.8)
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Connections:
- removed net DIO104: D209.2, D210.4, JP209.2, JP210.1
- removed net DIO152: D248.4, D308.2, JP248.1, JP308.2
- removed net DIO5: D10.2, D11.4, JP10.2, JP11.1
- removed net DIO6: D13.2, D14.4, JP13.2, JP14.1
- removed net N$128: D247.2, D250.4, JP247.2, JP250.1
- removed net N$132: D261.2, JP261.2
- removed net N$135: D11.2, D12.4, JP11.2, JP12.1
- removed net N$139: D264.2, D43.4, JP264.2, JP43.1
- removed net N$140: D266.2, D64.4, JP266.2, JP64.1
- removed net N$144: D106.4, D270.2, JP106.1, JP270.2
- removed net N$147: D148.4, D274.2, JP148.1, JP274.2
- removed net N$172: D231.2, D309.4, JP231.2, JP309.1
- removed net N$21: D1.2, D211.4, JP21.2, JP211.1
- removed net N$54: D84.2, D85.4, JP84.2, JP85.1
- removed net N$68: D127.4, D272.2, JP127.1, JP272.2
- removed net N$89: D168.2, D169.4, JP168.2, JP169.1
- removed net N$97: D188.2, D189.4, JP188.2, JP189.1
- net DIO10: now also D1.2, JP21.2; no longer D211.2, JP211.2
- net DIO109: now also D209.2, JP209.2; no longer D210.2, JP210.2
- net DIO119: now also D309.4, JP309.1; no longer D231.4, JP231.1
- net DIO121: now also D43.4, JP43.1; no longer D264.4, JP264.1
- net DIO127: now also D64.4, JP64.1; no longer D266.4, JP266.1
- net DIO130: now also D250.4, JP250.1; no longer D247.4, JP247.1
- net DIO151: now also D248.4, JP248.1; no longer D308.4, JP308.1
- net DIO44: now also D106.4, JP106.1; no longer D270.4, JP270.1
- net DIO54: now also D127.4, JP127.1; no longer D272.4, JP272.1
- net DIO76: now also D148.4, JP148.1; no longer D274.4, JP274.1
- net DIO87: now also D169.4, JP169.1; no longer D168.4, JP168.1
- net DIO99: now also D188.2, JP188.2; no longer D189.2, JP189.2
- net GND: no longer D11.3, D12.3, D13.3, D168.3, D189.3, D210.3, D211.3, D231.3, D247.3, D261.3, D264.3, D266.3, D270.3, D272.3, D274.3, D308.3, D84.3
- net N$133: no longer D261.4, JP261.1
- net N$142: now also D85.4, JP85.1; no longer D84.4, JP84.1
- net N$8: now also D10.2, D14.4, JP10.2, JP14.1; no longer D12.2, D13.4, JP12.2, JP13.1
- net V_USB: no longer D11.1, D12.1, D13.1, D168.1, D189.1, D210.1, D211.1, D231.1, D247.1, D261.1, D264.1, D266.1, D270.1, D272.1, D274.1, D308.1, D84.1
Routing:
- net N$139: track 350.3 -> 0.00 mm, vias 2 -> 0
- net N$140: track 350.1 -> 0.00 mm, vias 2 -> 0
- net N$89: track 349.1 -> 0.00 mm, vias 2 -> 0
- net N$144: track 349.1 -> 0.00 mm, vias 2 -> 0
- net N$172: track 348.9 -> 0.00 mm, vias 2 -> 0
- net N$54: track 348.9 -> 0.00 mm, vias 2 -> 0
- net DIO152: track 348.3 -> 0.00 mm, vias 2 -> 0
- net N$147: track 348.2 -> 0.00 mm, vias 2 -> 0
- net N$68: track 347.8 -> 0.00 mm, vias 2 -> 0
- net DIO127: track 16.8 -> 335.3 mm, vias 0 -> 2
- net DIO121: track 16.8 -> 335.2 mm, vias 0 -> 2
- net DIO87: track 16.8 -> 334.0 mm, vias 0 -> 2
- net DIO44: track 16.8 -> 333.8 mm, vias 0 -> 2
- net DIO119: track 16.8 -> 333.8 mm, vias 0 -> 2
- net N$142: track 16.8 -> 333.8 mm, vias 0 -> 2
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Other:
- outline, holes or cut-outs redrawn
- board text added: "15TB"
- board text removed: "15R"

Commit message: final touches, polishing, jumpers, CAM on all boards
Parts:
- added JP11, JP12, JP13, JP249, JP312, JP313, JP314, JP316, JP317, JP318, JP319, JP320, JP321: JUMPER-SMT_2_NO_NO-SILK, SparkFun-Jumpers:SMT-JUMPER_2_NO_NO-SILK
Connections:
- removed net DIO10: D1.2, D22.4, JP21.2, JP22.1
- removed net DIO109: D209.2, D21.4, JP1.1, JP209.2
- removed net DIO119: D230.2, D309.4, JP230.2, JP309.1
- removed net DIO121: D263.2, D43.4, JP263.2, JP43.1
- removed net DIO127: D265.2, D64.4, JP265.2, JP64.1
- removed net DIO130: D246.2, D250.4, JP246.2, JP250.1
- removed net DIO151: D248.4, D307.2, JP248.1, JP307.2
- removed net DIO44: D106.4, D269.2, JP106.1, JP269.2
- removed net DIO54: D127.4, D271.2, JP127.1, JP271.2
- removed net DIO76: D148.4, D273.2, JP148.1, JP273.2
- removed net DIO87: D167.2, D169.4, JP167.2, JP169.1
- removed net DIO99: D188.2, D190.4, JP188.2, JP190.1
- removed net N$142: D268.2, D85.4, JP268.2, JP85.1
- new net JUMPER0: D1.2, D22.4, JP11.2, JP12.1, JP21.2, JP22.1
- new net JUMPER1: D263.2, D43.4, JP12.2, JP13.1, JP263.2, JP43.1
- new net JUMPER10: D248.4, D307.2, JP248.1, JP307.2, JP319.2, JP320.1
- new net JUMPER11: D230.2, D309.4, JP230.2, JP309.1, JP320.2, JP321.1
- new net JUMPER12: D246.2, D250.4, JP246.2, JP250.1, JP321.2
- new net JUMPER2: D265.2, D64.4, JP13.2, JP249.1, JP265.2, JP64.1
- new net JUMPER3: D268.2, D85.4, JP249.2, JP268.2, JP312.1, JP85.1
- new net JUMPER4: D106.4, D269.2, JP106.1, JP269.2, JP312.2, JP313.1
- new net JUMPER5: D127.4, D271.2, JP127.1, JP271.2, JP313.2, JP314.1
- new net JUMPER6: D148.4, D273.2, JP148.1, JP273.2, JP314.2, JP316.1
- new net JUMPER7: D167.2, D169.4, JP167.2, JP169.1, JP316.2, JP317.1
- new net JUMPER8: D188.2, D190.4, JP188.2, JP190.1, JP317.2, JP318.1
- new net JUMPER9: D209.2, D21.4, JP1.1, JP209.2, JP318.2, JP319.1
- net DIO0: now also JP11.1
Routing:
- net JUMPER11: track 0.00 -> 363.2 mm, vias 0 -> 3
- net JUMPER0: track 0.00 -> 359.1 mm, vias 0 -> 2
- net JUMPER9: track 0.00 -> 356.3 mm, vias 0 -> 2
- net JUMPER2: track 0.00 -> 355.3 mm, vias 0 -> 2
- net JUMPER1: track 0.00 -> 355.1 mm, vias 0 -> 2
- net JUMPER7: track 0.00 -> 354.0 mm, vias 0 -> 2
- net JUMPER8: track 0.00 -> 354.0 mm, vias 0 -> 2
- net JUMPER4: track 0.00 -> 353.8 mm, vias 0 -> 2
- net JUMPER3: track 0.00 -> 353.7 mm, vias 0 -> 2
- net JUMPER6: track 0.00 -> 353.2 mm, vias 0 -> 2
- net JUMPER10: track 0.00 -> 353.2 mm, vias 0 -> 2
- net JUMPER5: track 0.00 -> 353.1 mm, vias 0 -> 2
- net DIO10: track 339.1 -> 0.00 mm, vias 2 -> 0
- net DIO109: track 336.4 -> 0.00 mm, vias 2 -> 0
- net DIO127: track 335.3 -> 0.00 mm, vias 2 -> 0
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
Commit message: pushing final board changes
Parts:
- removed D309, D310, D311: WS2812B, SparkFun-LED:WS2812B
- removed JP309, JP310, JP311: JUMPER-SMT_2_NO_NO-SILK, SparkFun-Jumpers:SMT-JUMPER_2_NO_NO-SILK
- added U$1: (no value), unnamed#png (2):UNNAMED#PNG
- moved C3 18.5 mm to (335.2, 44.6)
- moved R15 18.5 mm to (337.8, 44.6)
- moved R5 18.5 mm to (335.2, 46.5)
- moved C2 18.5 mm to (335.2, 50.3)
- moved R12 18.5 mm to (335.2, 42.7)
- moved R14 18.5 mm to (337.8, 50.3)
- moved R6 18.5 mm to (335.2, 52.2)
- moved R7 18.5 mm to (335.2, 48.4)
- moved R3 18.5 mm to (341.1, 30.3)
- moved R4 18.5 mm to (341.1, 27.8)
- moved J2 18.5 mm to (345.1, 29.0)
- moved J3 18.4 mm to (351.6, 47.0)
- moved C4 4.00 mm to (28.5, 19.0)
- moved C5 4.00 mm to (25.0, 19.0)
- moved C6 4.00 mm to (28.6, 21.7)
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Connections:
- removed net DIO143: D309.2, D310.4, JP309.2, JP310.1
- removed net N$170: D310.2, D311.4, JP310.2, JP311.1
- removed net N$173: D311.2, D315.4, JP311.2, JP315.1
- net GND: no longer D309.3, D310.3, D311.3
- net JUMPER11: now also D315.4, JP315.1; no longer D309.4, JP309.1
- net V_USB: no longer D309.1, D310.1, D311.1
Routing:
- net V_USB: track 553.8 -> 517.0 mm, vias 300 -> 298
- net N$170: track 34.2 -> 0.00 mm, vias 2 -> 0
- net 3.3V: track 430.1 -> 450.4 mm
- net DIO143: track 17.5 -> 0.00 mm, vias 2 -> 0
- net N$173: track 16.8 -> 0.00 mm
- net D-: track 365.6 -> 350.1 mm
- net D+: track 364.0 -> 349.0 mm
- net RING1: track 301.0 -> 312.4 mm, vias 0 -> 2
- net TIP: track 297.8 -> 308.5 mm, vias 0 -> 2
- net JUMPER11: track 363.2 -> 372.2 mm
- net DIO0: track 253.8 -> 247.1 mm
- net N$3: track 2.32 -> 3.19 mm
- net N$4: track 2.22 -> 3.04 mm
Other:
- outline, holes or cut-outs redrawn

Commit message: updating files
Parts:
- removed FD2: FIDUCIALUFIDUCIAL, SparkFun-Aesthetics:FIDUCIAL-MICRO
Changed lines of the file:
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@@
 </element>
 <element name="FD1" library="SparkFun-Aesthetics" package="FIDUCIAL-MICRO" value="FIDUCIALUFIDUCIAL" x="313.75" y="210" smashed="yes"/>
-<element name="FD2" library="SparkFun-Aesthetics" package="FIDUCIAL-MICRO" value="FIDUCIALUFIDUCIAL" x="9.555" y="42.5" smashed="yes"/>
 <element name="FD4" library="SparkFun-Aesthetics" package="FIDUCIAL-MICRO" value="FIDUCIALUFIDUCIAL" x="1" y="2" smashed="yes"/>
 <element name="Q2" library="SparkFun-DiscreteSemi" package="SC70-6" value="MBT3904DW1T1" x="29.48" y="8.445" smashed="yes" rot="R180">
