File: Hardware/15TB.sch (EAGLE design)
At the start: 668 parts, among them J2 USB Female Type C Connector, J3 AUDIO_JACK_TRRSSMD_RA, Q2 MBT3904DW1T1, U2 ESP-WROOM-32NARROW, U3 AP2112K-3.3V, U4 CP2102N, U5 ADMP401

Commit message: getting 4 boards polished
Parts:
- removed D11, D12, D13, D168, D189, D210, D211, D231, D247, D261, D264, D266, D270, D272, D274, D308, D84: WS2812B, SparkFun-LED:WS2812B
- removed JP11, JP12, JP13, JP168, JP189, JP210, JP211, JP231, JP247, JP261, JP264, JP266, JP270, JP272, JP274, JP308, JP84: JUMPER-SMT_2_NO_NO-SILK, SparkFun-Jumpers:JUMPER-SMT_2_NO_NO-SILK
Connections:
- removed net DIO104: D209.DO, D210.DI, JP209.2, JP210.1
- removed net DIO152: D248.DI, D308.DO, JP248.1, JP308.2
- removed net DIO5: D10.DO, D11.DI, JP10.2, JP11.1
- removed net DIO6: D13.DO, D14.DI, JP13.2, JP14.1
- removed net N$128: D247.DO, D250.DI, JP247.2, JP250.1
- removed net N$132: D261.DO, JP261.2
- removed net N$135: D11.DO, D12.DI, JP11.2, JP12.1
- removed net N$139: D264.DO, D43.DI, JP264.2, JP43.1
- removed net N$140: D266.DO, D64.DI, JP266.2, JP64.1
- removed net N$144: D106.DI, D270.DO, JP106.1, JP270.2
- removed net N$147: D148.DI, D274.DO, JP148.1, JP274.2
- removed net N$172: D231.DO, D309.DI, JP231.2, JP309.1
- removed net N$21: D1.DO, D211.DI, JP21.2, JP211.1
- removed net N$54: D84.DO, D85.DI, JP84.2, JP85.1
- removed net N$68: D127.DI, D272.DO, JP127.1, JP272.2
- removed net N$89: D168.DO, D169.DI, JP168.2, JP169.1
- removed net N$97: D188.DO, D189.DI, JP188.2, JP189.1
- net DIO10: now also D1.DO, JP21.2; no longer D211.DO, JP211.2
- net DIO109: now also D209.DO, JP209.2; no longer D210.DO, JP210.2
- net DIO119: now also D309.DI, JP309.1; no longer D231.DI, JP231.1
- net DIO121: now also D43.DI, JP43.1; no longer D264.DI, JP264.1
- net DIO127: now also D64.DI, JP64.1; no longer D266.DI, JP266.1
- net DIO130: now also D250.DI, JP250.1; no longer D247.DI, JP247.1
- net DIO151: now also D248.DI, JP248.1; no longer D308.DI, JP308.1
- net DIO44: now also D106.DI, JP106.1; no longer D270.DI, JP270.1
- net DIO54: now also D127.DI, JP127.1; no longer D272.DI, JP272.1
- net DIO76: now also D148.DI, JP148.1; no longer D274.DI, JP274.1
- net DIO87: now also D169.DI, JP169.1; no longer D168.DI, JP168.1
- net DIO99: now also D188.DO, JP188.2; no longer D189.DO, JP189.2
- net GND: no longer D11.VSS, D12.VSS, D13.VSS, D168.VSS, D189.VSS, D210.VSS, D211.VSS, D231.VSS, D247.VSS, D261.VSS, D264.VSS, D266.VSS, D270.VSS, D272.VSS, D274.VSS, D308.VSS, D84.VSS
- net N$133: no longer D261.DI, JP261.1
- net N$142: now also D85.DI, JP85.1; no longer D84.DI, JP84.1
- net N$8: now also D10.DO, D14.DI, JP10.2, JP14.1; no longer D12.DO, D13.DI, JP12.2, JP13.1
- net V_USB: no longer D11.VDD, D12.VDD, D13.VDD, D168.VDD, D189.VDD, D210.VDD, D211.VDD, D231.VDD, D247.VDD, D261.VDD, D264.VDD, D266.VDD, D270.VDD, D272.VDD, D274.VDD, D308.VDD, D84.VDD

Commit message: final touches, polishing, jumpers, CAM on all boards
Parts:
- added JP11, JP12, JP13, JP249, JP312, JP313, JP314, JP316, JP317, JP318, JP319, JP320, JP321: JUMPER-SMT_2_NO_NO-SILK, SparkFun-Jumpers:JUMPER-SMT_2_NO_NO-SILK
Connections:
- removed net DIO10: D1.DO, D22.DI, JP21.2, JP22.1
- removed net DIO109: D209.DO, D21.DI, JP1.1, JP209.2
- removed net DIO119: D230.DO, D309.DI, JP230.2, JP309.1
- removed net DIO121: D263.DO, D43.DI, JP263.2, JP43.1
- removed net DIO127: D265.DO, D64.DI, JP265.2, JP64.1
- removed net DIO130: D246.DO, D250.DI, JP246.2, JP250.1
- removed net DIO151: D248.DI, D307.DO, JP248.1, JP307.2
- removed net DIO44: D106.DI, D269.DO, JP106.1, JP269.2
- removed net DIO54: D127.DI, D271.DO, JP127.1, JP271.2
- removed net DIO76: D148.DI, D273.DO, JP148.1, JP273.2
- removed net DIO87: D167.DO, D169.DI, JP167.2, JP169.1
- removed net DIO99: D188.DO, D190.DI, JP188.2, JP190.1
- removed net N$142: D268.DO, D85.DI, JP268.2, JP85.1
- new net JUMPER0: D1.DO, D22.DI, JP11.2, JP12.1, JP21.2, JP22.1
- new net JUMPER1: D263.DO, D43.DI, JP12.2, JP13.1, JP263.2, JP43.1
- new net JUMPER10: D248.DI, D307.DO, JP248.1, JP307.2, JP319.2, JP320.1
- new net JUMPER11: D230.DO, D309.DI, JP230.2, JP309.1, JP320.2, JP321.1
- new net JUMPER12: D246.DO, D250.DI, JP246.2, JP250.1, JP321.2
- new net JUMPER2: D265.DO, D64.DI, JP13.2, JP249.1, JP265.2, JP64.1
- new net JUMPER3: D268.DO, D85.DI, JP249.2, JP268.2, JP312.1, JP85.1
- new net JUMPER4: D106.DI, D269.DO, JP106.1, JP269.2, JP312.2, JP313.1
- new net JUMPER5: D127.DI, D271.DO, JP127.1, JP271.2, JP313.2, JP314.1
- new net JUMPER6: D148.DI, D273.DO, JP148.1, JP273.2, JP314.2, JP316.1
- new net JUMPER7: D167.DO, D169.DI, JP167.2, JP169.1, JP316.2, JP317.1
- new net JUMPER8: D188.DO, D190.DI, JP188.2, JP190.1, JP317.2, JP318.1
- new net JUMPER9: D209.DO, D21.DI, JP1.1, JP209.2, JP318.2, JP319.1
- net DIO0: now also JP11.1

Commit message: pushing final board changes
Parts:
- removed D309, D310, D311: WS2812B, SparkFun-LED:WS2812B
- removed JP309, JP310, JP311: JUMPER-SMT_2_NO_NO-SILK, SparkFun-Jumpers:JUMPER-SMT_2_NO_NO-SILK
Connections:
- removed net DIO143: D309.DO, D310.DI, JP309.2, JP310.1
- removed net N$170: D310.DO, D311.DI, JP310.2, JP311.1
- removed net N$173: D311.DO, D315.DI, JP311.2, JP315.1
- net GND: no longer D309.VSS, D310.VSS, D311.VSS
- net JUMPER11: now also D315.DI, JP315.1; no longer D309.DI, JP309.1
- net V_USB: no longer D309.VDD, D310.VDD, D311.VDD

Commit message: updating files
Parts:
- removed FD2: FIDUCIALUFIDUCIAL, SparkFun-Aesthetics:FIDUCIALUFIDUCIAL
Changed lines of the file:
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@@
 <part name="C1" library="SparkFun-Capacitors" deviceset="10UF" device="-0603-6.3V-20%" value="10uF"/>
 <part name="FD1" library="SparkFun-Aesthetics" deviceset="FIDUCIAL" device="UFIDUCIAL"/>
-<part name="FD2" library="SparkFun-Aesthetics" deviceset="FIDUCIAL" device="UFIDUCIAL"/>
 <part name="FD4" library="SparkFun-Aesthetics" deviceset="FIDUCIAL" device="UFIDUCIAL"/>
 <part name="S2" library="SparkFun-Switches" deviceset="MOMENTARY-SWITCH-SPST-2" device="-SMD-4.6X2.8MM" value="0"/>
@@
 </instance>
 <instance part="FD1" gate="G$1" x="429.26" y="33.02" smashed="yes"/>
-<instance part="FD2" gate="G$1" x="426.72" y="33.02" smashed="yes"/>
 <instance part="FD4" gate="G$1" x="429.26" y="30.48" smashed="yes"/>
 <instance part="S2" gate="G$1" x="294.64" y="177.8" smashed="yes">
